File: FPGA_DecCaps.sch (KiCad schematic (older format))
At the start: 15 parts

Commit message: La til hele Artix7-kretsen
Changed lines of the file:
@@
 $Descr A4 11693 8268
 encoding utf-8
-Sheet 2 2
+Sheet 2 3
 Title ""
 Date ""
@@
 Connection ~ 1700 3050
 Connection ~ 1300 3050
+Text HLabel 1300 3050 0    50   Input ~ 0
+FPGADecoupleVCC
+Text HLabel 1300 3550 0    50   Input ~ 0
+FPGADecoupleGND
 $EndSCHEMATC
