File: FPGADecCaps.sch (KiCad schematic (older format))
At the start: 15 parts

Commit message: Extra decouplers in FPGA-sheet
Parts:
- added C? (x2): 47u, symbol Device:C
- added C? (x4): 4.7u, symbol Device:C
- added C? (x6): 470n, symbol Device:C
- added C?: 100u, symbol Device:CP1
Connections:
- net labels added: +1V0, +1V8
- wire segments 30 -> 56
Other:
- moved on the sheet: C?

Commit message: Add capacitors to FPGA Decouplers to match datasheet for XC7A100T Split up the Vcco capacitors again into the banks as described in the datasheet. Copy a row of banks if we end up needing more io pins. The 100u capacitor can be used by up to 4 I/O banks. Add another if we end up exceeding that.
Parts:
- removed C?: 47u, symbol Device:C
- added C? (x4): 4.7u, symbol Device:C
- added C? (x7): 470n, symbol Device:C
- C? (x2): value 47u -> 100u
- C?: value 100u -> 330u
Connections:
- wire segments 56 -> 76
Other:
- note added: "Vccaux"
- note added: "Vccbram"
- note added: "Vccint"
- note added: "Vcco"
- moved on the sheet: C?

Commit message: Mye har skjedd
Parts:
- C12, C13, C14, C15, C16, C17, C18, C19, C20, C21, C22, C23, C24, C25, C26, C27, C28, C29, C30, C31, C32, C33, C34, C35, C36, C37, C38, C39, C40, C41, C42, C43, C44, C45, C46, C47, C48, C49: renamed from C?; footprint (none) -> Capacitor_THT:CP_Radial_D4.0mm_P1.50mm
Connections:
- net labels added: 1.0V, 1.8V, 3.3V
- net labels removed: +1V0, +1V8, +3.3V

Commit message: use power symbols for 1V0 1V8
Connections:
- net labels added: +1V0, +1V8, +3.3V
- net labels removed: 1.0V, 1.8V, 3.3V
Changed lines of the file:
@@
 Wire Wire Line
 	3800 6300 3800 6050
-Wire Wire Line
-	3800 5550 3800 5750
 $Comp
 L Device:C C14
@@
 Wire Wire Line
 	7700 5750 7000 5750
-Text Label 3800 1200 0    50   ~ 0
-1.0V
-Text Label 3800 2450 0    50   ~ 0
-1.0V
-Text Label 3800 3750 0    50   ~ 0
-1.8V
-Text Label 3800 5550 0    50   ~ 0
-3.3V
+$Comp
+L power:+1V0 #PWR?
+U 1 1 5D825A6C
+P 3800 2450
+F 0 "#PWR?" H 3800 2300 50  0001 C CNN
+F 1 "+1V0" H 3815 2623 50  0000 C CNN
+F 2 "" H 3800 2450 50  0001 C CNN
+F 3 "" H 3800 2450 50  0001 C CNN
+	1    3800 2450
+	1    0    0    -1
+$EndComp
+$Comp
+L power:+1V0 #PWR?
+U 1 1 5D828B0C
+P 3800 1200
+F 0 "#PWR?" H 3800 1050 50  0001 C CNN
+F 1 "+1V0" H 3815 1373 50  0000 C CNN
+F 2 "" H 3800 1200 50  0001 C CNN
+F 3 "" H 3800 1200 50  0001 C CNN
+	1    3800 1200
+	1    0    0    -1
+$EndComp
+$Comp
+L power:+1V8 #PWR?
+U 1 1 5D828EE9
+P 3800 3750
+F 0 "#PWR?" H 3800 3600 50  0001 C CNN
+F 1 "+1V8" H 3815 3923 50  0000 C CNN
+F 2 "" H 3800 3750 50  0001 C CNN
+F 3 "" H 3800 3750 50  0001 C CNN
+	1    3800 3750
+	1    0    0    -1
+$EndComp
+Wire Wire Line
+	3800 5550 3800 5750
+$Comp
+L power:+3.3V #PWR?
+U 1 1 5D829896
+P 3800 5550
+F 0 "#PWR?" H 3800 5400 50  0001 C CNN
+F 1 "+3.3V" H 3815 5723 50  0000 C CNN
+F 2 "" H 3800 5550 50  0001 C CNN
+F 3 "" H 3800 5550 50  0001 C CNN
+	1    3800 5550
+	1    0    0    -1
+$EndComp
 $EndSCHEMATC
