File: FPGADecCaps.sch (KiCad schematic (older format))
At the start: 38 parts

Commit message: Fixed FPGA decouplers so they deliver power. Removed Synthesizer-cache lib.
Connections:
- net labels added: +1V0, +1V8, +3.3V
- net labels removed: 1.0V, 1.8V, 3.3V
Changed lines of the file:
@@
 EESchema Schematic File Version 4
-LIBS:Synthesizer-cache
 EELAYER 30 0
 EELAYER END
@@
 	3800 4550 3800 4300
 Connection ~ 3800 4300
-Wire Wire Line
-	3800 3750 3800 4000
 $Comp
 L Device:C C18
@@
 Wire Wire Line
 	7700 5750 7000 5750
-Text Label 3800 1200 0    50   ~ 0
-1.0V
-Text Label 3800 2450 0    50   ~ 0
-1.0V
-Text Label 3800 3750 0    50   ~ 0
-1.8V
-Text Label 3800 5550 0    50   ~ 0
-3.3V
+$Comp
+L power:+1V0 #PWR?
+U 1 1 5D82295E
+P 3800 1200
+F 0 "#PWR?" H 3800 1050 50  0001 C CNN
+F 1 "+1V0" H 3815 1373 50  0000 C CNN
+F 2 "" H 3800 1200 50  0001 C CNN
+F 3 "" H 3800 1200 50  0001 C CNN
+	1    3800 1200
+	1    0    0    -1
+$EndComp
+$Comp
+L power:+1V0 #PWR?
+U 1 1 5D823042
+P 3800 2450
+F 0 "#PWR?" H 3800 2300 50  0001 C CNN
+F 1 "+1V0" H 3815 2623 50  0000 C CNN
+F 2 "" H 3800 2450 50  0001 C CNN
+F 3 "" H 3800 2450 50  0001 C CNN
+	1    3800 2450
+	1    0    0    -1
+$EndComp
+Wire Wire Line
+	3800 3750 3800 4000
+$Comp
+L power:+1V8 #PWR?
+U 1 1 5D824195
+P 3800 3750
+F 0 "#PWR?" H 3800 3600 50  0001 C CNN
+F 1 "+1V8" H 3815 3923 50  0000 C CNN
+F 2 "" H 3800 3750 50  0001 C CNN
+F 3 "" H 3800 3750 50  0001 C CNN
+	1    3800 3750
+	1    0    0    -1
+$EndComp
+$Comp
+L power:+3.3V #PWR?
+U 1 1 5D8259D3
+P 3800 5550
+F 0 "#PWR?" H 3800 5400 50  0001 C CNN
+F 1 "+3.3V" H 3815 5723 50  0000 C CNN
+F 2 "" H 3800 5550 50  0001 C CNN
+F 3 "" H 3800 5550 50  0001 C CNN
+	1    3800 5550
+	1    0    0    -1
+$EndComp
 $EndSCHEMATC

Commit message: Onsdags-commit
Parts:
- C12, C13, C14, C15, C16, C17, C18, C19, C20, C21, C22, C23, C24, C25, C26, C27, C28, C29, C30, C31, C32, C33, C34, C35, C36, C37, C38, C39, C40, C41, C42, C43, C44, C45, C46, C47, C48, C49: footprint Capacitor_SMD:C_0201_0603Metric -> Capacitor_SMD:C_0805_2012Metric

Commit message: Better footprints
Parts:
- C12, C13, C14, C15, C16, C17, C18, C19, C20, C21, C22, C23, C24, C25, C26, C27, C28, C29, C30, C31, C32, C33, C34, C35, C36, C37, C38, C39, C40, C41, C42, C43, C44, C45, C46, C47, C48, C49: footprint Capacitor_SMD:C_0805_2012Metric -> Capacitor_SMD:C_0805_2012Metric_Pad1.15x1.40mm_HandSolder

Commit message: Updated component footprints. The PCB is now an unholy mess.
Parts:
- C12, C13, C14, C15, C16, C17, C18, C19, C20, C21, C22, C23, C24, C25, C26, C27, C28, C29, C30, C31, C32, C33, C34, C35, C36, C37, C38, C39, C40, C41, C42, C43, C44, C45, C46, C47, C48, C49: footprint Capacitor_SMD:C_0805_2012Metric_Pad1.15x1.40mm_HandSolder -> Capacitor_SMD:C_1206_3216Metric_Pad1.42x1.75mm_HandSolder
