File: FPGADecCaps.sch (KiCad schematic (older format))
At the start: 38 parts

Commit message: Wire up 1V PSU. Use smaller footprints for small caps.
Parts:
- C18, C22, C23, C26, C29, C30, C32, C34, C35, C36, C37, C38, C40, C42, C43, C44, C45, C46, C47, C48, C49: footprint Capacitor_SMD:C_1206_3216Metric_Pad1.42x1.75mm_HandSolder -> Capacitor_SMD:C_0805_2012Metric_Pad1.15x1.40mm_HandSolder
Changed lines of the file:
@@
 F 0 "C43" H 8615 5946 50  0000 L CNN
 F 1 "470n" H 8615 5855 50  0000 L CNN
-F 2 "Capacitor_SMD:C_1206_3216Metric_Pad1.42x1.75mm_HandSolder" H 8538 5750 50  0001 C CNN
+F 2 "Capacitor_SMD:C_0805_2012Metric_Pad1.15x1.40mm_HandSolder" H 8538 5750 50  0001 C CNN
 F 3 "~" H 8500 5900 50  0001 C CNN
 	1    8500 5900
@@
 F 0 "C45" H 9015 5946 50  0000 L CNN
 F 1 "470n" H 9015 5855 50  0000 L CNN
-F 2 "Capacitor_SMD:C_1206_3216Metric_Pad1.42x1.75mm_HandSolder" H 8938 5750 50  0001 C CNN
+F 2 "Capacitor_SMD:C_0805_2012Metric_Pad1.15x1.40mm_HandSolder" H 8938 5750 50  0001 C CNN
 F 3 "~" H 8900 5900 50  0001 C CNN
 	1    8900 5900
@@
 F 0 "C47" H 9415 5946 50  0000 L CNN
 F 1 "470n" H 9415 5855 50  0000 L CNN
-F 2 "Capacitor_SMD:C_1206_3216Metric_Pad1.42x1.75mm_HandSolder" H 9338 5750 50  0001 C CNN
+F 2 "Capacitor_SMD:C_0805_2012Metric_Pad1.15x1.40mm_HandSolder" H 9338 5750 50  0001 C CNN
 F 3 "~" H 9300 5900 50  0001 C CNN
 	1    9300 5900
@@
 F 0 "C49" H 9815 5946 50  0000 L CNN
 F 1 "470n" H 9815 5855 50  0000 L CNN
-F 2 "Capacitor_SMD:C_1206_3216Metric_Pad1.42x1.75mm_HandSolder" H 9738 5750 50  0001 C CNN
+F 2 "Capacitor_SMD:C_0805_2012Metric_Pad1.15x1.40mm_HandSolder" H 9738 5750 50  0001 C CNN
 F 3 "~" H 9700 5900 50  0001 C CNN
 	1    9700 5900
@@
 F 0 "C30" H 5915 5946 50  0000 L CNN
 F 1 "470n" H 5915 5855 50  0000 L CNN
-F 2 "Capacitor_SMD:C_1206_3216Metric_Pad1.42x1.75mm_HandSolder" H 5838 5750 50  0001 C CNN
+F 2 "Capacitor_SMD:C_0805_2012Metric_Pad1.15x1.40mm_HandSolder" H 5838 5750 50  0001 C CNN
 F 3 "~" H 5800 5900 50  0001 C CNN
 	1    5800 5900
@@
 F 0 "C32" H 6315 5946 50  0000 L CNN
 F 1 "470n" H 6315 5855 50  0000 L CNN
-F 2 "Capacitor_SMD:C_1206_3216Metric_Pad1.42x1.75mm_HandSolder" H 6238 5750 50  0001 C CNN
+F 2 "Capacitor_SMD:C_0805_2012Metric_Pad1.15x1.40mm_HandSolder" H 6238 5750 50  0001 C CNN
 F 3 "~" H 6200 5900 50  0001 C CNN
 	1    6200 5900
@@
 F 0 "C34" H 6715 5946 50  0000 L CNN
 F 1 "470n" H 6715 5855 50  0000 L CNN
-F 2 "Capacitor_SMD:C_1206_3216Metric_Pad1.42x1.75mm_HandSolder" H 6638 5750 50  0001 C CNN
+F 2 "Capacitor_SMD:C_0805_2012Metric_Pad1.15x1.40mm_HandSolder" H 6638 5750 50  0001 C CNN
 F 3 "~" H 6600 5900 50  0001 C CNN
 	1    6600 5900
@@
 F 0 "C36" H 7115 5946 50  0000 L CNN
 F 1 "470n" H 7115 5855 50  0000 L CNN
-F 2 "Capacitor_SMD:C_1206_3216Metric_Pad1.42x1.75mm_HandSolder" H 7038 5750 50  0001 C CNN
+F 2 "Capacitor_SMD:C_0805_2012Metric_Pad1.15x1.40mm_HandSolder" H 7038 5750 50  0001 C CNN
 F 3 "~" H 7000 5900 50  0001 C CNN
 	1    7000 5900
@@
 F 0 "C23" H 5015 4196 50  0000 L CNN
 F 1 "470n" H 5015 4105 50  0000 L CNN
-F 2 "Capacitor_SMD:C_1206_3216Metric_Pad1.42x1.75mm_HandSolder" H 4938 4000 50  0001 C CNN
+F 2 "Capacitor_SMD:C_0805_2012Metric_Pad1.15x1.40mm_HandSolder" H 4938 4000 50  0001 C CNN
 F 3 "~" H 4900 4150 50  0001 C CNN
 	1    4900 4150
@@
 F 0 "C26" H 5415 4196 50  0000 L CNN
 F 1 "470n" H 5415 4105 50  0000 L CNN
-F 2 "Capacitor_SMD:C_1206_3216Metric_Pad1.42x1.75mm_HandSolder" H 5338 4000 50  0001 C CNN
+F 2 "Capacitor_SMD:C_0805_2012Metric_Pad1.15x1.40mm_HandSolder" H 5338 4000 50  0001 C CNN
 F 3 "~" H 5300 4150 50  0001 C CNN
 	1    5300 4150
@@
 F 0 "C29" H 5815 4196 50  0000 L CNN
 F 1 "470n" H 5815 4105 50  0000 L CNN
-F 2 "Capacitor_SMD:C_1206_3216Metric_Pad1.42x1.75mm_HandSolder" H 5738 4000 50  0001 C CNN
+F 2 "Capacitor_SMD:C_0805_2012Metric_Pad1.15x1.40mm_HandSolder" H 5738 4000 50  0001 C CNN
 F 3 "~" H 5700 4150 50  0001 C CNN
 	1    5700 4150
@@
 F 0 "C18" H 4365 2846 50  0000 L CNN
 F 1 "470n" H 4365 2755 50  0000 L CNN
-F 2 "Capacitor_SMD:C_1206_3216Metric_Pad1.42x1.75mm_HandSolder" H 4288 2650 50  0001 C CNN
+F 2 "Capacitor_SMD:C_0805_2012Metric_Pad1.15x1.40mm_HandSolder" H 4288 2650 50  0001 C CNN
 F 3 "~" H 4250 2800 50  0001 C CNN
 	1    4250 2800
@@
 F 0 "C35" H 6865 1546 50  0000 L CNN
 F 1 "470n" H 6865 1455 50  0000 L CNN
-F 2 "Capacitor_SMD:C_1206_3216Metric_Pad1.42x1.75mm_HandSolder" H 6788 1350 50  0001 C CNN
+F 2 "Capacitor_SMD:C_0805_2012Metric_Pad1.15x1.40mm_HandSolder" H 6788 1350 50  0001 C CNN
 F 3 "~" H 6750 1500 50  0001 C CNN
 	1    6750 1500
@@
 F 0 "C37" H 7265 1546 50  0000 L CNN
 F 1 "470n" H 7265 1455 50  0000 L CNN
-F 2 "Capacitor_SMD:C_1206_3216Metric_Pad1.42x1.75mm_HandSolder" H 7188 1350 50  0001 C CNN
+F 2 "Capacitor_SMD:C_0805_2012Metric_Pad1.15x1.40mm_HandSolder" H 7188 1350 50  0001 C CNN
 F 3 "~" H 7150 1500 50  0001 C CNN
 	1    7150 1500
@@
 F 0 "C48" H 9665 1546 50  0000 L CNN
 F 1 "470n" H 9665 1455 50  0000 L CNN
-F 2 "Capacitor_SMD:C_1206_3216Metric_Pad1.42x1.75mm_HandSolder" H 9588 1350 50  0001 C CNN
+F 2 "Capacitor_SMD:C_0805_2012Metric_Pad1.15x1.40mm_HandSolder" H 9588 1350 50  0001 C CNN
 F 3 "~" H 9550 1500 50  0001 C CNN
 	1    9550 1500
@@
 F 0 "C46" H 9265 1546 50  0000 L CNN
 F 1 "470n" H 9265 1455 50  0000 L CNN
-F 2 "Capacitor_SMD:C_1206_3216Metric_Pad1.42x1.75mm_HandSolder" H 9188 1350 50  0001 C CNN
+F 2 "Capacitor_SMD:C_0805_2012Metric_Pad1.15x1.40mm_HandSolder" H 9188 1350 50  0001 C CNN
 F 3 "~" H 9150 1500 50  0001 C CNN
 	1    9150 1500
@@
 F 0 "C44" H 8865 1546 50  0000 L CNN
 F 1 "470n" H 8865 1455 50  0000 L CNN
-F 2 "Capacitor_SMD:C_1206_3216Metric_Pad1.42x1.75mm_HandSolder" H 8788 1350 50  0001 C CNN
+F 2 "Capacitor_SMD:C_0805_2012Metric_Pad1.15x1.40mm_HandSolder" H 8788 1350 50  0001 C CNN
 F 3 "~" H 8750 1500 50  0001 C CNN
 	1    8750 1500
@@
 F 0 "C42" H 8465 1546 50  0000 L CNN
 F 1 "470n" H 8465 1455 50  0000 L CNN
-F 2 "Capacitor_SMD:C_1206_3216Metric_Pad1.42x1.75mm_HandSolder" H 8388 1350 50  0001 C CNN
+F 2 "Capacitor_SMD:C_0805_2012Metric_Pad1.15x1.40mm_HandSolder" H 8388 1350 50  0001 C CNN
 F 3 "~" H 8350 1500 50  0001 C CNN
 	1    8350 1500
@@
 F 0 "C40" H 8065 1546 50  0000 L CNN
 F 1 "470n" H 8065 1455 50  0000 L CNN
-F 2 "Capacitor_SMD:C_1206_3216Metric_Pad1.42x1.75mm_HandSolder" H 7988 1350 50  0001 C CNN
+F 2 "Capacitor_SMD:C_0805_2012Metric_Pad1.15x1.40mm_HandSolder" H 7988 1350 50  0001 C CNN
 F 3 "~" H 7950 1500 50  0001 C CNN
 	1    7950 1500
@@
 F 0 "C38" H 7665 1546 50  0000 L CNN
 F 1 "470n" H 7665 1455 50  0000 L CNN
-F 2 "Capacitor_SMD:C_1206_3216Metric_Pad1.42x1.75mm_HandSolder" H 7588 1350 50  0001 C CNN
+F 2 "Capacitor_SMD:C_0805_2012Metric_Pad1.15x1.40mm_HandSolder" H 7588 1350 50  0001 C CNN
 F 3 "~" H 7550 1500 50  0001 C CNN
 	1    7550 1500
@@
 F 0 "C22" H 4815 2846 50  0000 L CNN
 F 1 "470n" H 4815 2755 50  0000 L CNN
-F 2 "Capacitor_SMD:C_1206_3216Metric_Pad1.42x1.75mm_HandSolder" H 4738 2650 50  0001 C CNN
+F 2 "Capacitor_SMD:C_0805_2012Metric_Pad1.15x1.40mm_HandSolder" H 4738 2650 50  0001 C CNN
 F 3 "~" H 4700 2800 50  0001 C CNN
 	1    4700 2800

Commit message: Added in a bunch of footprints to the netlist; only missing buttons and some resistors, now.
Parts:
- C12: footprint Capacitor_SMD:C_1206_3216Metric_Pad1.42x1.75mm_HandSolder -> Capacitor_THT:CP_Radial_D10.0mm_P5.00mm
Changed lines of the file:
@@
 F 0 "C12" H 3915 1546 50  0000 L CNN
 F 1 "330u" H 3915 1455 50  0000 L CNN
-F 2 "Capacitor_SMD:C_1206_3216Metric_Pad1.42x1.75mm_HandSolder" H 3800 1500 50  0001 C CNN
+F 2 "Capacitor_THT:CP_Radial_D10.0mm_P5.00mm" H 3800 1500 50  0001 C CNN
 F 3 "~" H 3800 1500 50  0001 C CNN
 	1    3800 1500

Commit message: Revert "Added in a bunch of footprints to the netlist; only missing buttons and some resistors, now."
This reverts commit 26f31b12234d03a706d1f0abb84aa744ef749ada.
Parts:
- C12: footprint Capacitor_THT:CP_Radial_D10.0mm_P5.00mm -> Capacitor_SMD:C_1206_3216Metric_Pad1.42x1.75mm_HandSolder
Changed lines of the file:
@@
 F 0 "C12" H 3915 1546 50  0000 L CNN
 F 1 "330u" H 3915 1455 50  0000 L CNN
-F 2 "Capacitor_THT:CP_Radial_D10.0mm_P5.00mm" H 3800 1500 50  0001 C CNN
+F 2 "Capacitor_SMD:C_1206_3216Metric_Pad1.42x1.75mm_HandSolder" H 3800 1500 50  0001 C CNN
 F 3 "~" H 3800 1500 50  0001 C CNN
 	1    3800 1500
