File: Synthesizer.sch (KiCad schematic (older format))
At the start: 29 parts, among them J2 AudioJack3, SW1 SW_Push, SW10 SW_Push, SW11 SW_Push, SW12 SW_Push, SW13 SW_Push, SW2 SW_Push, SW3 SW_Push, SW4 SW_Push, SW5 SW_Push, SW6 SW_Push, SW7 SW_Push, SW8 SW_Push, SW9 SW_Push

Commit message: Added ESD protection to USB-A. Connected Soft-mute.
Parts:
- removed J?: USB_B, symbol Connector:USB_B
- added C1: 150u, symbol Device:C
- added C2: 0.1u, symbol Device:C
- added FB1, FB3: Ferrite_Bead, symbol Device:Ferrite_Bead
- added J3: USB_B_Micro, symbol Connector:USB_B_Micro
- added U1: TPD3S014, Package_TO_SOT_SMD:SOT-23-6, symbol Power_Protection:TPD3S014
- gave numbers to parts that had none: 1
Connections:
- net labels removed: +5V
- wire segments 80 -> 103
Changed lines of the file:
@@
 Wire Wire Line
 	9050 8200 9050 8400
-NoConn ~ 9150 8300
 Wire Wire Line
 	5350 13650 5350 14200
@@
 	-1   0    0    1
 $EndComp
+Wire Wire Line
+	6500 5300 8150 5300
+Wire Wire Line
+	6500 5400 8150 5400
+Wire Wire Line
+	6500 5500 8150 5500
+Wire Wire Line
+	8150 5600 6500 5600
+Wire Wire Line
+	6500 5150 8150 5150
+Wire Wire Line
+	8150 5050 6500 5050
+Wire Wire Line
+	11750 8200 12000 8200
+Wire Wire Line
+	11750 8100 12000 8100
+$Comp
+L power:GND #PWR04
+U 1 1 5D88FD38
+P 11900 8400
+F 0 "#PWR04" H 11900 8150 50  0001 C CNN
+F 1 "GND" H 11905 8227 50  0000 C CNN
+F 2 "" H 11900 8400 50  0001 C CNN
+F 3 "" H 11900 8400 50  0001 C CNN
+	1    11900 8400
+	1    0    0    -1
+$EndComp
+Wire Wire Line
+	12000 8300 11900 8300
+Wire Wire Line
+	11900 8300 11900 8400
+$Comp
+L power:GND #PWR05
+U 1 1 5D894417
+P 14350 5200
+F 0 "#PWR05" H 14350 4950 50  0001 C CNN
+F 1 "GND" H 14355 5027 50  0000 C CNN
+F 2 "" H 14350 5200 50  0001 C CNN
+F 3 "" H 14350 5200 50  0001 C CNN
+	1    14350 5200
+	1    0    0    -1
+$EndComp
+Wire Wire Line
+	14350 5050 14350 5200
+NoConn ~ 14650 4650
+NoConn ~ 14650 4750
+NoConn ~ 14250 5050
+Text Notes 5550 4850 0    50   ~ 0
+idk how to connect this
+Text Notes 14000 4100 0    50   ~ 0
+I think this makes sense?
+Wire Wire Line
+	14650 4450 15050 4450
+$Comp
+L Connector:USB_B_Micro J3
+U 1 1 5D8F0994
+P 14350 4650
+F 0 "J3" H 14407 5117 50  0000 C CNN
+F 1 "USB_B_Micro" H 14407 5026 50  0000 C CNN
+F 2 "" H 14500 4600 50  0001 C CNN
+F 3 "~" H 14500 4600 50  0001 C CNN
+	1    14350 4650
+	1    0    0    -1
+$EndComp
+$Comp
+L Power_Protection:TPD3S014 U1
+U 1 1 5D919E8B
+P 4300 4450
+F 0 "U1" H 4300 4725 50  0000 C CNN
+F 1 "TPD3S014" H 4300 4816 50  0000 C CNN
+F 2 "Package_TO_SOT_SMD:SOT-23-6" H 4300 4800 50  0001 C CNN
+F 3 "http://www.ti.com/lit/ds/symlink/tpd3s014.pdf" H 4100 4700 50  0001 C CNN
+	1    4300 4450
+	-1   0    0    1
+$EndComp
+Wire Wire Line
+	2800 5750 2800 5700
+Wire Wire Line
+	2800 5350 2800 5400
+$Comp
+L Device:Ferrite_Bead FB1
+U 1 1 5D913522
+P 2800 5550
+F 0 "FB1" H 2937 5596 50  0000 L CNN
+F 1 "Ferrite_Bead" H 2937 5505 50  0000 L CNN
+F 2 "" V 2730 5550 50  0001 C CNN
+F 3 "~" H 2800 5550 50  0001 C CNN
+	1    2800 5550
+	1    0    0    -1
+$EndComp
+$Comp
+L power:GND #PWR02
+U 1 1 5D8C6D8D
+P 2800 5750
+F 0 "#PWR02" H 2800 5500 50  0001 C CNN
+F 1 "GND" H 2805 5577 50  0000 C CNN
+F 2 "" H 2800 5750 50  0001 C CNN
+F 3 "" H 2800 5750 50  0001 C CNN
+	1    2800 5750
+	1    0    0    -1
+$EndComp
+Wire Wire Line
+	4950 4750 4750 4750
+Wire Wire Line
+	4800 4350 4700 4350
+$Comp
+L power:GND #PWR03
+U 1 1 5D937153
+P 4300 3900
+F 0 "#PWR03" H 4300 3650 50  0001 C CNN
+F 1 "GND" H 4305 3727 50  0000 C CNN
+F 2 "" H 4300 3900 50  0001 C CNN
+F 3 "" H 4300 3900 50  0001 C CNN
+	1    4300 3900
+	-1   0    0    1
+$EndComp
+Wire Wire Line
+	4950 5050 3850 5050
+Wire Wire Line
+	3900 4450 3850 4450
+Connection ~ 3850 5050
+Wire Wire Line
+	3850 5050 3100 5050
+Wire Wire Line
+	3850 4450 3850 5050
+Wire Wire Line
+	3100 4950 3800 4950
+Wire Wire Line
+	3900 4350 3800 4350
+Wire Wire Line
+	3800 4350 3800 4950
+Connection ~ 3800 4950
+Wire Wire Line
+	3800 4950 4950 4950
+$Comp
+L Device:C C1
+U 1 1 5D947DEC
+P 3700 4150
+F 0 "C1" H 3815 4196 50  0000 L CNN
+F 1 "150u" H 3815 4105 50  0000 L CNN
+F 2 "" H 3738 4000 50  0001 C CNN
+F 3 "~" H 3700 4150 50  0001 C CNN
+	1    3700 4150
+	1    0    0    -1
+$EndComp
+Wire Wire Line
+	3700 4750 3700 4550
+Wire Wire Line
+	3700 4550 3900 4550
+Wire Wire Line
+	3700 4550 3700 4300
+Connection ~ 3700 4550
+Wire Wire Line
+	4750 4750 4750 4550
+Wire Wire Line
+	4750 4550 4700 4550
+$Comp
+L Device:C C2
+U 1 1 5D9626CB
+P 4750 4150
+F 0 "C2" H 4865 4196 50  0000 L CNN
+F 1 "0.1u" H 4865 4105 50  0000 L CNN
+F 2 "" H 4788 4000 50  0001 C CNN
+F 3 "~" H 4750 4150 50  0001 C CNN
+	1    4750 4150
+	1    0    0    -1
+$EndComp
+Wire Wire Line
+	4750 4300 4750 4550
+Connection ~ 4750 4550
+Wire Wire Line
+	4750 4000 4300 4000
+Wire Wire Line
+	4300 4000 4300 3900
+Connection ~ 4300 4000
+Wire Wire Line
+	3700 4000 4300 4000
+Wire Wire Line
+	4300 4150 4300 4000
+Wire Wire Line
+	4950 4850 4800 4850
+Wire Wire Line
+	4800 4850 4800 4350
 $Sheet
 S 4950 4600 1550 1250
@@
 F10 "USB_D-" U L 4950 5050 50
 F11 "USB_D+" U L 4950 4950 50
+F12 "Overcurrent" I L 4950 4650 50
+F13 "Soft-mute" O R 6500 5800 50
 $EndSheet
 Wire Wire Line
-	6500 5300 8150 5300
-Wire Wire Line
-	6500 5400 8150 5400
-Wire Wire Line
-	6500 5500 8150 5500
-Wire Wire Line
-	8150 5600 6500 5600
-Wire Wire Line
-	6500 5150 8150 5150
-Wire Wire Line
-	8150 5050 6500 5050
-$Comp
-L Connector:USB_B J?
-U 1 1 5D8E7346
-P 14350 4650
-F 0 "J?" H 14407 5117 50  0000 C CNN
-F 1 "USB_B" H 14407 5026 50  0000 C CNN
-F 2 "" H 14500 4600 50  0001 C CNN
-F 3 " ~" H 14500 4600 50  0001 C CNN
-	1    14350 4650
-	1    0    0    -1
-$EndComp
-Wire Wire Line
-	11750 8200 12000 8200
-Wire Wire Line
-	11750 8100 12000 8100
-$Comp
-L power:GND #PWR?
-U 1 1 5D88FD38
-P 11900 8400
-F 0 "#PWR?" H 11900 8150 50  0001 C CNN
-F 1 "GND" H 11905 8227 50  0000 C CNN
-F 2 "" H 11900 8400 50  0001 C CNN
-F 3 "" H 11900 8400 50  0001 C CNN
-	1    11900 8400
-	1    0    0    -1
-$EndComp
-Wire Wire Line
-	12000 8300 11900 8300
-Wire Wire Line
-	11900 8300 11900 8400
-$Comp
-L power:GND #PWR?
-U 1 1 5D894417
-P 14350 5200
-F 0 "#PWR?" H 14350 4950 50  0001 C CNN
-F 1 "GND" H 14355 5027 50  0000 C CNN
-F 2 "" H 14350 5200 50  0001 C CNN
-F 3 "" H 14350 5200 50  0001 C CNN
-	1    14350 5200
-	1    0    0    -1
-$EndComp
-Wire Wire Line
-	14350 5050 14350 5200
-Wire Wire Line
-	14650 4450 14800 4450
-NoConn ~ 14650 4650
-NoConn ~ 14650 4750
-NoConn ~ 14250 5050
-Text Notes 14000 4100 0    50   ~ 0
-I think this makes sense?
-$Comp
-L Connector:USB_A J?
+	6500 5800 6650 5800
+Wire Wire Line
+	6650 5800 6650 8300
+Wire Wire Line
+	6650 8300 9150 8300
+$Comp
+L Device:Ferrite_Bead FB3
+U 1 1 5D98E4B3
+P 3350 4750
+F 0 "FB3" V 3076 4750 50  0000 C CNN
+F 1 "Ferrite_Bead" V 3167 4750 50  0000 C CNN
+F 2 "" V 3280 4750 50  0001 C CNN
+F 3 "~" H 3350 4750 50  0001 C CNN
+	1    3350 4750
+	0    1    1    0
+$EndComp
+Wire Wire Line
+	3700 4750 3500 4750
+Wire Wire Line
+	3200 4750 3100 4750
+$Comp
+L Connector:USB_A J1
 U 1 1 5D8BD3E6
-P 3950 4950
-F 0 "J?" H 4007 5417 50  0000 C CNN
-F 1 "USB_A" H 4007 5326 50  0000 C CNN
-F 2 "" H 4100 4900 50  0001 C CNN
-F 3 " ~" H 4100 4900 50  0001 C CNN
-	1    3950 4950
-	1    0    0    -1
-$EndComp
-$Comp
-L power:+5V #PWR?
-U 1 1 5D8C2B59
-P 14800 4300
-F 0 "#PWR?" H 14800 4150 50  0001 C CNN
-F 1 "+5V" H 14815 4473 50  0000 C CNN
-F 2 "" H 14800 4300 50  0001 C CNN
-F 3 "" H 14800 4300 50  0001 C CNN
-	1    14800 4300
-	1    0    0    -1
-$EndComp
-Wire Wire Line
-	14800 4300 14800 4450
-Connection ~ 14800 4450
-Wire Wire Line
-	14800 4450 15050 4450
-$Comp
-L power:GND #PWR?
-U 1 1 5D8C6D8D
-P 3950 5550
-F 0 "#PWR?" H 3950 5300 50  0001 C CNN
-F 1 "GND" H 3955 5377 50  0000 C CNN
-F 2 "" H 3950 5550 50  0001 C CNN
-F 3 "" H 3950 5550 50  0001 C CNN
-	1    3950 5550
-	1    0    0    -1
-$EndComp
-Wire Wire Line
-	3950 5350 3950 5550
-Wire Wire Line
-	4250 4750 4950 4750
-Wire Wire Line
-	4250 4950 4950 4950
-Wire Wire Line
-	4950 5050 4250 5050
-Text Notes 5550 4850 0    50   ~ 0
-idk how to connect this
+P 2800 4950
+F 0 "J1" H 2857 5417 50  0000 C CNN
+F 1 "USB_A" H 2857 5326 50  0000 C CNN
+F 2 "" H 2950 4900 50  0001 C CNN
+F 3 " ~" H 2950 4900 50  0001 C CNN
+	1    2800 4950
+	1    0    0    -1
+$EndComp
+NoConn ~ 2700 5350
 $EndSCHEMATC
