File: Synthesizer.sch (KiCad schematic (older format))
At the start: 34 parts, among them J1 USB_A, J2 AudioJack3, J3 USB_B_Micro, SW1 SW_Push, SW10 SW_Push, SW11 SW_Push, SW12 SW_Push, SW13 SW_Push, SW2 SW_Push, SW3 SW_Push, SW4 SW_Push, SW5 SW_Push, SW6 SW_Push, SW7 SW_Push, SW8 SW_Push, SW9 SW_Push, U1 TPD3S014

Commit message: Added power source for USB-A.
Connections:
- net labels added: +5V
- wire segments 103 -> 105
- no-connect marks 4 -> 5
Other:
- note added: "TODO: Add a switch here for Overcurrent"
Changed lines of the file:
@@
 	0    1    1    0
 $EndComp
-$Comp
-L power:PWR_FLAG #FLG0101
-U 1 1 5E0BB0C2
-P 4900 2200
-F 0 "#FLG0101" H 4900 2275 50  0001 C CNN
-F 1 "PWR_FLAG" H 4900 2373 50  0000 C CNN
-F 2 "" H 4900 2200 50  0001 C CNN
-F 3 "~" H 4900 2200 50  0001 C CNN
-	1    4900 2200
-	1    0    0    -1
-$EndComp
-$Comp
-L power:GND #PWR0120
-U 1 1 5E0BBA07
-P 4900 2400
-F 0 "#PWR0120" H 4900 2150 50  0001 C CNN
-F 1 "GND" H 4905 2227 50  0000 C CNN
-F 2 "" H 4900 2400 50  0001 C CNN
-F 3 "" H 4900 2400 50  0001 C CNN
-	1    4900 2400
-	1    0    0    -1
-$EndComp
-Wire Wire Line
-	4900 2200 4900 2400
 Wire Wire Line
 	17400 4400 17200 4400
@@
 $EndComp
 Wire Wire Line
-	6500 5300 8150 5300
-Wire Wire Line
-	6500 5400 8150 5400
-Wire Wire Line
-	6500 5500 8150 5500
-Wire Wire Line
-	8150 5600 6500 5600
-Wire Wire Line
-	6500 5150 8150 5150
-Wire Wire Line
-	8150 5050 6500 5050
+	6900 5300 8150 5300
+Wire Wire Line
+	6900 5400 8150 5400
+Wire Wire Line
+	6900 5500 8150 5500
+Wire Wire Line
+	8150 5600 6900 5600
+Wire Wire Line
+	6900 5150 8150 5150
+Wire Wire Line
+	8150 5050 6900 5050
 Wire Wire Line
 	11750 8200 12000 8200
@@
 NoConn ~ 14650 4750
 NoConn ~ 14250 5050
-Text Notes 5550 4850 0    50   ~ 0
+Text Notes 5950 4800 0    50   ~ 0
 idk how to connect this
 Text Notes 14000 4100 0    50   ~ 0
@@
 $EndComp
 Wire Wire Line
-	4950 4750 4750 4750
+	5350 4750 4900 4750
 Wire Wire Line
 	4800 4350 4700 4350
@@
 $EndComp
 Wire Wire Line
-	4950 5050 3850 5050
+	5350 5050 3850 5050
 Wire Wire Line
 	3900 4450 3850 4450
@@
 Connection ~ 3800 4950
 Wire Wire Line
-	3800 4950 4950 4950
+	3800 4950 5350 4950
 $Comp
 L Device:C C1
@@
 	4300 4150 4300 4000
 Wire Wire Line
-	4950 4850 4800 4850
+	5350 4850 4800 4850
 Wire Wire Line
 	4800 4850 4800 4350
 $Sheet
-S 4950 4600 1550 1250
+S 5350 4600 1550 1250
 U 5D8502F2
 F0 "EFM32" 50
 F1 "EFM32.sch" 50
-F2 "SPI_MISO" I R 6500 5400 50
-F3 "SPI_CLK" O R 6500 5500 50
-F4 "SPI_CS" O R 6500 5600 50
-F5 "SPI_MOSI" O R 6500 5300 50
-F6 "FPGA_Ready" I R 6500 5050 50
-F7 "FPGA_Reset" O R 6500 5150 50
-F8 "USB_VBUS" I L 4950 4750 50
-F9 "USB_VBUSEN" I L 4950 4850 50
-F10 "USB_D-" U L 4950 5050 50
-F11 "USB_D+" U L 4950 4950 50
-F12 "Overcurrent" I L 4950 4650 50
-F13 "Soft-mute" O R 6500 5800 50
+F2 "SPI_MISO" I R 6900 5400 50
+F3 "SPI_CLK" O R 6900 5500 50
+F4 "SPI_CS" O R 6900 5600 50
+F5 "SPI_MOSI" O R 6900 5300 50
+F6 "FPGA_Ready" I R 6900 5050 50
+F7 "FPGA_Reset" O R 6900 5150 50
+F8 "USB_VBUS" I L 5350 4750 50
+F9 "USB_VBUSEN" I L 5350 4850 50
+F10 "USB_D-" U L 5350 5050 50
+F11 "USB_D+" U L 5350 4950 50
+F12 "Overcurrent" I L 5350 4650 50
+F13 "Soft-mute" O R 6900 5800 50
 $EndSheet
 Wire Wire Line
-	6500 5800 6650 5800
-Wire Wire Line
-	6650 5800 6650 8300
-Wire Wire Line
-	6650 8300 9150 8300
+	6900 5800 7200 5800
+Wire Wire Line
+	7200 5800 7200 8300
+Wire Wire Line
+	7200 8300 9150 8300
 $Comp
 L Device:Ferrite_Bead FB3
@@
 $EndComp
 NoConn ~ 2700 5350
+Wire Wire Line
+	4900 2200 4900 2400
+$Comp
+L power:GND #PWR0120
+U 1 1 5E0BBA07
+P 4900 2400
+F 0 "#PWR0120" H 4900 2150 50  0001 C CNN
+F 1 "GND" H 4905 2227 50  0000 C CNN
+F 2 "" H 4900 2400 50  0001 C CNN
+F 3 "" H 4900 2400 50  0001 C CNN
+	1    4900 2400
+	1    0    0    -1
+$EndComp
+$Comp
+L power:PWR_FLAG #FLG0101
+U 1 1 5E0BB0C2
+P 4900 2200
+F 0 "#FLG0101" H 4900 2275 50  0001 C CNN
+F 1 "PWR_FLAG" H 4900 2373 50  0000 C CNN
+F 2 "" H 4900 2200 50  0001 C CNN
+F 3 "~" H 4900 2200 50  0001 C CNN
+	1    4900 2200
+	1    0    0    -1
+$EndComp
+$Comp
+L power:+5V #PWR046
+U 1 1 5D9D4DF6
+P 4900 4500
+F 0 "#PWR046" H 4900 4350 50  0001 C CNN
+F 1 "+5V" H 4915 4673 50  0000 C CNN
+F 2 "" H 4900 4500 50  0001 C CNN
+F 3 "" H 4900 4500 50  0001 C CNN
+	1    4900 4500
+	1    0    0    -1
+$EndComp
+Wire Wire Line
+	4900 4500 4900 4750
+Connection ~ 4900 4750
+Wire Wire Line
+	4900 4750 4750 4750
+Text Notes 4950 4500 0    50   ~ 0
+TODO: Add a switch here for Overcurrent
+NoConn ~ 14650 4850
 $EndSCHEMATC

Commit message: Added forgotten USB-B power source, powered bank 14 of FPGA.
Connections:
- wire segments 105 -> 107
Changed lines of the file:
@@
 I think this makes sense?
 Wire Wire Line
-	14650 4450 15050 4450
+	14650 4450 14800 4450
 $Comp
 L Connector:USB_B_Micro J3
@@
 TODO: Add a switch here for Overcurrent
 NoConn ~ 14650 4850
+$Comp
+L power:+5V #PWR047
+U 1 1 5DA5CFE7
+P 14800 4350
+F 0 "#PWR047" H 14800 4200 50  0001 C CNN
+F 1 "+5V" H 14815 4523 50  0000 C CNN
+F 2 "" H 14800 4350 50  0001 C CNN
+F 3 "" H 14800 4350 50  0001 C CNN
+	1    14800 4350
+	1    0    0    -1
+$EndComp
+Wire Wire Line
+	14800 4450 14800 4350
+Connection ~ 14800 4450
+Wire Wire Line
+	14800 4450 15050 4450
 $EndSCHEMATC

Commit message: add placeholder footprints, clean up ratsnest a bit
Parts:
- C1, C2: footprint (none) -> Capacitor_SMD:C_0805_2012Metric_Pad1.15x1.40mm_HandSolder
- FB1, FB3: footprint (none) -> Inductor_SMD:L_0805_2012Metric_Pad1.15x1.40mm_HandSolder
- J1: footprint (none) -> Connector_USB:USB_A_CNCTech_1001-011-01101_Horizontal
- J3: footprint (none) -> Connector_USB:USB_Micro-B_GCT_USB3076-30-A
Changed lines of the file:
@@
 EESchema Schematic File Version 4
+LIBS:Synthesizer-cache
 EELAYER 30 0
 EELAYER END
@@
 F 0 "J3" H 14407 5117 50  0000 C CNN
 F 1 "USB_B_Micro" H 14407 5026 50  0000 C CNN
-F 2 "" H 14500 4600 50  0001 C CNN
+F 2 "Connector_USB:USB_Micro-B_GCT_USB3076-30-A" H 14500 4600 50  0001 C CNN
 F 3 "~" H 14500 4600 50  0001 C CNN
 	1    14350 4650
@@
 F 0 "FB1" H 2937 5596 50  0000 L CNN
 F 1 "Ferrite_Bead" H 2937 5505 50  0000 L CNN
-F 2 "" V 2730 5550 50  0001 C CNN
+F 2 "Inductor_SMD:L_0805_2012Metric_Pad1.15x1.40mm_HandSolder" V 2730 5550 50  0001 C CNN
 F 3 "~" H 2800 5550 50  0001 C CNN
 	1    2800 5550
@@
 F 0 "C1" H 3815 4196 50  0000 L CNN
 F 1 "150u" H 3815 4105 50  0000 L CNN
-F 2 "" H 3738 4000 50  0001 C CNN
+F 2 "Capacitor_SMD:C_0805_2012Metric_Pad1.15x1.40mm_HandSolder" H 3738 4000 50  0001 C CNN
 F 3 "~" H 3700 4150 50  0001 C CNN
 	1    3700 4150
@@
 F 0 "C2" H 4865 4196 50  0000 L CNN
 F 1 "0.1u" H 4865 4105 50  0000 L CNN
-F 2 "" H 4788 4000 50  0001 C CNN
+F 2 "Capacitor_SMD:C_0805_2012Metric_Pad1.15x1.40mm_HandSolder" H 4788 4000 50  0001 C CNN
 F 3 "~" H 4750 4150 50  0001 C CNN
 	1    4750 4150
@@
 F 0 "FB3" V 3076 4750 50  0000 C CNN
 F 1 "Ferrite_Bead" V 3167 4750 50  0000 C CNN
-F 2 "" V 3280 4750 50  0001 C CNN
+F 2 "Inductor_SMD:L_0805_2012Metric_Pad1.15x1.40mm_HandSolder" V 3280 4750 50  0001 C CNN
 F 3 "~" H 3350 4750 50  0001 C CNN
 	1    3350 4750
@@
 F 0 "J1" H 2857 5417 50  0000 C CNN
 F 1 "USB_A" H 2857 5326 50  0000 C CNN
-F 2 "" H 2950 4900 50  0001 C CNN
+F 2 "Connector_USB:USB_A_CNCTech_1001-011-01101_Horizontal" H 2950 4900 50  0001 C CNN
 F 3 " ~" H 2950 4900 50  0001 C CNN
 	1    2800 4950

Commit message: Connect buttons and move MCU->FPGA done/program_b pins
Parts:
- added R? (x3): R, Resistor_SMD:R_0805_2012Metric_Pad1.15x1.40mm_HandSolder, symbol Device:R
- added SW? (x3): SW_Push, Button_Switch_SMD:SW_Push_1P1T_NO_6x6mm_H9.5mm, symbol Switch:SW_Push
- renumbered SW13 to SW14
Connections:
- net labels added: Button0, Button14, Button15
- wire segments 107 -> 129

Commit message: Added NPN transistor on USB and wired shield. Added LEDs, debug pins.
Parts:
- added D1, D2, D3, D4: LED, symbol Device:LED
- added FB4: Ferrite_Bead, Inductor_SMD:L_0805_2012Metric_Pad1.15x1.40mm_HandSolder, symbol Device:Ferrite_Bead
- added Q1: Q_NPN_BCE, symbol Device:Q_NPN_BCE
- gave numbers to parts that had none: 6
Connections:
- wire segments 129 -> 153
- no-connect marks 5 -> 4
Other:
- note added: "Do we need to wire shield here\nwhen we don't use data pins?"
- note added: "huge TODO on this transistor, i have no idea what im doing"
- note added: "transistor needs 5V VC and 3.3V VB, i think?"
- note removed: "TODO: Add a switch here for Overcurrent"
- note removed: "idk how to connect this"

Commit message: Give footprints to LEDs
Parts:
- D1, D2, D3, D4: footprint (none) -> LED_THT:LED_D3.0mm
Changed lines of the file:
@@
 F 0 "D1" H 7300 5750 50  0000 C CNN
 F 1 "LED" H 7150 5750 50  0000 C CNN
-F 2 "" H 7150 5850 50  0001 C CNN
+F 2 "LED_THT:LED_D3.0mm" H 7150 5850 50  0001 C CNN
 F 3 "~" H 7150 5850 50  0001 C CNN
 	1    7150 5850
@@
 F 0 "D2" H 7200 6050 50  0000 C CNN
 F 1 "LED" H 7050 6050 50  0000 C CNN
-F 2 "" H 7150 5950 50  0001 C CNN
+F 2 "LED_THT:LED_D3.0mm" H 7150 5950 50  0001 C CNN
 F 3 "~" H 7150 5950 50  0001 C CNN
 	1    7150 5950
@@
 F 0 "D4" H 10700 5100 50  0000 C CNN
 F 1 "LED" H 10700 5200 50  0000 C CNN
-F 2 "" H 10700 5000 50  0001 C CNN
+F 2 "LED_THT:LED_D3.0mm" H 10700 5000 50  0001 C CNN
 F 3 "~" H 10700 5000 50  0001 C CNN
 	1    10700 5000
@@
 F 0 "D3" H 10693 4645 50  0000 C CNN
 F 1 "LED" H 10693 4736 50  0000 C CNN
-F 2 "" H 10700 4900 50  0001 C CNN
+F 2 "LED_THT:LED_D3.0mm" H 10700 4900 50  0001 C CNN
 F 3 "~" H 10700 4900 50  0001 C CNN
 	1    10700 4900

Commit message: Fix USB connections and various cleanup
Parts:
- removed Q1: Q_NPN_BCE, symbol Device:Q_NPN_BCE
- added R33, R34: 33, Resistor_SMD:R_0805_2012Metric_Pad1.15x1.40mm_HandSolder, symbol Device:R
Connections:
- wire segments 153 -> 155
- no-connect marks 4 -> 3
Other:
- note removed: "Do we need to wire shield here\nwhen we don't use data pins?"
- note removed: "huge TODO on this transistor, i have no idea what im doing"
- note removed: "transistor needs 5V VC and 3.3V VB, i think?"
