File: Synthesizer.sch (KiCad schematic (older format))
At the start: 51 parts, among them J1 USB_A, J2 AudioJack3, J3 USB_B_Micro, SW1 SW_Push, SW10 SW_Push, SW11 SW_Push, SW12 SW_Push, SW13 SW_Push, SW14 SW_Push, SW15 SW_Push, SW16 SW_Push, SW2 SW_Push, SW3 SW_Push, SW4 SW_Push, SW5 SW_Push, SW6 SW_Push, SW7 SW_Push, SW8 SW_Push, SW9 SW_Push, U1 TPD3S014

Commit message: Updated component footprints. The PCB is now an unholy mess.
Parts:
- C1, C2: footprint Capacitor_SMD:C_0805_2012Metric_Pad1.15x1.40mm_HandSolder -> Capacitor_SMD:C_1206_3216Metric_Pad1.42x1.75mm_HandSolder
- FB1, FB3, FB4: footprint Inductor_SMD:L_0805_2012Metric_Pad1.15x1.40mm_HandSolder -> footprints:FerriteBead_74279215
- R18, R19, R20, R21, R22, R23, R24, R25, R26, R27, R28, R29, R32, R33, R34, R35, R36, R37: footprint Resistor_SMD:R_0805_2012Metric_Pad1.15x1.40mm_HandSolder -> Resistor_SMD:R_1206_3216Metric_Pad1.42x1.75mm_HandSolder
- R38, R39, R40, R41: footprint (none) -> Resistor_SMD:R_1206_3216Metric_Pad1.42x1.75mm_HandSolder
Changed lines of the file:
@@
 F 0 "R18" H 1580 8404 50  0000 R CNN
 F 1 "R" H 1580 8495 50  0000 R CNN
-F 2 "Resistor_SMD:R_0805_2012Metric_Pad1.15x1.40mm_HandSolder" V 1580 8450 50  0001 C CNN
+F 2 "Resistor_SMD:R_1206_3216Metric_Pad1.42x1.75mm_HandSolder" V 1580 8450 50  0001 C CNN
 F 3 "~" H 1650 8450 50  0001 C CNN
 	1    1650 8450
@@
 F 0 "R27" H 1580 13354 50  0000 R CNN
 F 1 "R" H 1580 13445 50  0000 R CNN
-F 2 "Resistor_SMD:R_0805_2012Metric_Pad1.15x1.40mm_HandSolder" V 1580 13400 50  0001 C CNN
+F 2 "Resistor_SMD:R_1206_3216Metric_Pad1.42x1.75mm_HandSolder" V 1580 13400 50  0001 C CNN
 F 3 "~" H 1650 13400 50  0001 C CNN
 	1    1650 13400
@@
 F 0 "R26" H 1580 12804 50  0000 R CNN
 F 1 "R" H 1580 12895 50  0000 R CNN
-F 2 "Resistor_SMD:R_0805_2012Metric_Pad1.15x1.40mm_HandSolder" V 1580 12850 50  0001 C CNN
+F 2 "Resistor_SMD:R_1206_3216Metric_Pad1.42x1.75mm_HandSolder" V 1580 12850 50  0001 C CNN
 F 3 "~" H 1650 12850 50  0001 C CNN
 	1    1650 12850
@@
 F 0 "R25" H 1580 12254 50  0000 R CNN
 F 1 "R" H 1580 12345 50  0000 R CNN
-F 2 "Resistor_SMD:R_0805_2012Metric_Pad1.15x1.40mm_HandSolder" V 1580 12300 50  0001 C CNN
+F 2 "Resistor_SMD:R_1206_3216Metric_Pad1.42x1.75mm_HandSolder" V 1580 12300 50  0001 C CNN
 F 3 "~" H 1650 12300 50  0001 C CNN
 	1    1650 12300
@@
 F 0 "R24" H 1580 11704 50  0000 R CNN
 F 1 "R" H 1580 11795 50  0000 R CNN
-F 2 "Resistor_SMD:R_0805_2012Metric_Pad1.15x1.40mm_HandSolder" V 1580 11750 50  0001 C CNN
+F 2 "Resistor_SMD:R_1206_3216Metric_Pad1.42x1.75mm_HandSolder" V 1580 11750 50  0001 C CNN
 F 3 "~" H 1650 11750 50  0001 C CNN
 	1    1650 11750
@@
 F 0 "R23" H 1580 11154 50  0000 R CNN
 F 1 "R" H 1580 11245 50  0000 R CNN
-F 2 "Resistor_SMD:R_0805_2012Metric_Pad1.15x1.40mm_HandSolder" V 1580 11200 50  0001 C CNN
+F 2 "Resistor_SMD:R_1206_3216Metric_Pad1.42x1.75mm_HandSolder" V 1580 11200 50  0001 C CNN
 F 3 "~" H 1650 11200 50  0001 C CNN
 	1    1650 11200
@@
 F 0 "R22" H 1580 10604 50  0000 R CNN
 F 1 "R" H 1580 10695 50  0000 R CNN
-F 2 "Resistor_SMD:R_0805_2012Metric_Pad1.15x1.40mm_HandSolder" V 1580 10650 50  0001 C CNN
+F 2 "Resistor_SMD:R_1206_3216Metric_Pad1.42x1.75mm_HandSolder" V 1580 10650 50  0001 C CNN
 F 3 "~" H 1650 10650 50  0001 C CNN
 	1    1650 10650
@@
 F 0 "R21" H 1580 10054 50  0000 R CNN
 F 1 "R" H 1580 10145 50  0000 R CNN
-F 2 "Resistor_SMD:R_0805_2012Metric_Pad1.15x1.40mm_HandSolder" V 1580 10100 50  0001 C CNN
+F 2 "Resistor_SMD:R_1206_3216Metric_Pad1.42x1.75mm_HandSolder" V 1580 10100 50  0001 C CNN
 F 3 "~" H 1650 10100 50  0001 C CNN
 	1    1650 10100
@@
 F 0 "R20" H 1580 9504 50  0000 R CNN
 F 1 "R" H 1580 9595 50  0000 R CNN
-F 2 "Resistor_SMD:R_0805_2012Metric_Pad1.15x1.40mm_HandSolder" V 1580 9550 50  0001 C CNN
+F 2 "Resistor_SMD:R_1206_3216Metric_Pad1.42x1.75mm_HandSolder" V 1580 9550 50  0001 C CNN
 F 3 "~" H 1650 9550 50  0001 C CNN
 	1    1650 9550
@@
 F 0 "R19" H 1580 8954 50  0000 R CNN
 F 1 "R" H 1580 9045 50  0000 R CNN
-F 2 "Resistor_SMD:R_0805_2012Metric_Pad1.15x1.40mm_HandSolder" V 1580 9000 50  0001 C CNN
+F 2 "Resistor_SMD:R_1206_3216Metric_Pad1.42x1.75mm_HandSolder" V 1580 9000 50  0001 C CNN
 F 3 "~" H 1650 9000 50  0001 C CNN
 	1    1650 9000
@@
 F 0 "R28" H 1580 13904 50  0000 R CNN
 F 1 "R" H 1580 13995 50  0000 R CNN
-F 2 "Resistor_SMD:R_0805_2012Metric_Pad1.15x1.40mm_HandSolder" V 1580 13950 50  0001 C CNN
+F 2 "Resistor_SMD:R_1206_3216Metric_Pad1.42x1.75mm_HandSolder" V 1580 13950 50  0001 C CNN
 F 3 "~" H 1650 13950 50  0001 C CNN
 	1    1650 13950
@@
 F 0 "R32" H 3130 13904 50  0000 R CNN
 F 1 "R" H 3130 13995 50  0000 R CNN
-F 2 "Resistor_SMD:R_0805_2012Metric_Pad1.15x1.40mm_HandSolder" V 3130 13950 50  0001 C CNN
+F 2 "Resistor_SMD:R_1206_3216Metric_Pad1.42x1.75mm_HandSolder" V 3130 13950 50  0001 C CNN
 F 3 "~" H 3200 13950 50  0001 C CNN
 	1    3200 13950
@@
 F 0 "C2" H 4865 4196 50  0000 L CNN
 F 1 "0.1u" H 4865 4105 50  0000 L CNN
-F 2 "Capacitor_SMD:C_0805_2012Metric_Pad1.15x1.40mm_HandSolder" H 4788 4000 50  0001 C CNN
+F 2 "Capacitor_SMD:C_1206_3216Metric_Pad1.42x1.75mm_HandSolder" H 4788 4000 50  0001 C CNN
 F 3 "~" H 4750 4150 50  0001 C CNN
 	1    4750 4150
@@
 F 0 "FB3" V 3226 4750 50  0000 C CNN
 F 1 "Ferrite_Bead" V 3317 4750 50  0000 C CNN
-F 2 "Inductor_SMD:L_0805_2012Metric_Pad1.15x1.40mm_HandSolder" V 3430 4750 50  0001 C CNN
+F 2 "footprints:FerriteBead_74279215" V 3430 4750 50  0001 C CNN
 F 3 "~" H 3500 4750 50  0001 C CNN
 	1    3500 4750
@@
 F 0 "R35" H 1580 7854 50  0000 R CNN
 F 1 "R" H 1580 7945 50  0000 R CNN
-F 2 "Resistor_SMD:R_0805_2012Metric_Pad1.15x1.40mm_HandSolder" V 1580 7900 50  0001 C CNN
+F 2 "Resistor_SMD:R_1206_3216Metric_Pad1.42x1.75mm_HandSolder" V 1580 7900 50  0001 C CNN
 F 3 "~" H 1650 7900 50  0001 C CNN
 	1    1650 7900
@@
 F 0 "R36" H 3130 13354 50  0000 R CNN
 F 1 "R" H 3130 13445 50  0000 R CNN
-F 2 "Resistor_SMD:R_0805_2012Metric_Pad1.15x1.40mm_HandSolder" V 3130 13400 50  0001 C CNN
+F 2 "Resistor_SMD:R_1206_3216Metric_Pad1.42x1.75mm_HandSolder" V 3130 13400 50  0001 C CNN
 F 3 "~" H 3200 13400 50  0001 C CNN
 	1    3200 13400
@@
 F 0 "R37" H 3130 14504 50  0000 R CNN
 F 1 "R" H 3130 14595 50  0000 R CNN
-F 2 "Resistor_SMD:R_0805_2012Metric_Pad1.15x1.40mm_HandSolder" V 3130 14550 50  0001 C CNN
+F 2 "Resistor_SMD:R_1206_3216Metric_Pad1.42x1.75mm_HandSolder" V 3130 14550 50  0001 C CNN
 F 3 "~" H 3200 14550 50  0001 C CNN
 	1    3200 14550
@@
 F 0 "R29" H 1580 14454 50  0000 R CNN
 F 1 "R" H 1580 14545 50  0000 R CNN
-F 2 "Resistor_SMD:R_0805_2012Metric_Pad1.15x1.40mm_HandSolder" V 1580 14500 50  0001 C CNN
+F 2 "Resistor_SMD:R_1206_3216Metric_Pad1.42x1.75mm_HandSolder" V 1580 14500 50  0001 C CNN
 F 3 "~" H 1650 14500 50  0001 C CNN
 	1    1650 14500
@@
 F 0 "FB1" H 3087 5696 50  0000 L CNN
 F 1 "Ferrite_Bead" H 3087 5605 50  0000 L CNN
-F 2 "Inductor_SMD:L_0805_2012Metric_Pad1.15x1.40mm_HandSolder" V 2880 5650 50  0001 C CNN
+F 2 "footprints:FerriteBead_74279215" V 2880 5650 50  0001 C CNN
 F 3 "~" H 2950 5650 50  0001 C CNN
 	1    2950 5650
@@
 F 0 "FB4" H 2787 5696 50  0000 L CNN
 F 1 "Ferrite_Bead" H 2787 5605 50  0000 L CNN
-F 2 "Inductor_SMD:L_0805_2012Metric_Pad1.15x1.40mm_HandSolder" V 2580 5650 50  0001 C CNN
+F 2 "footprints:FerriteBead_74279215" V 2580 5650 50  0001 C CNN
 F 3 "~" H 2650 5650 50  0001 C CNN
 	1    2650 5650
@@
 F 0 "R34" V 4650 5050 50  0000 C CNN
 F 1 "33" V 4550 5050 50  0000 C CNN
-F 2 "Resistor_SMD:R_0805_2012Metric_Pad1.15x1.40mm_HandSolder" V 4480 5050 50  0001 C CNN
+F 2 "Resistor_SMD:R_1206_3216Metric_Pad1.42x1.75mm_HandSolder" V 4480 5050 50  0001 C CNN
 F 3 "~" H 4550 5050 50  0001 C CNN
 	1    4550 5050
@@
 F 0 "R33" V 4450 4950 50  0000 C CNN
 F 1 "33" V 4550 4950 50  0000 C CNN
-F 2 "Resistor_SMD:R_0805_2012Metric_Pad1.15x1.40mm_HandSolder" V 4480 4950 50  0001 C CNN
+F 2 "Resistor_SMD:R_1206_3216Metric_Pad1.42x1.75mm_HandSolder" V 4480 4950 50  0001 C CNN
 F 3 "~" H 4550 4950 50  0001 C CNN
 	1    4550 4950
@@
 F 0 "R38" V 7500 5850 50  0000 C CNN
 F 1 "100" V 7600 5850 50  0000 C CNN
-F 2 "" V 7530 5850 50  0001 C CNN
+F 2 "Resistor_SMD:R_1206_3216Metric_Pad1.42x1.75mm_HandSolder" V 7530 5850 50  0001 C CNN
 F 3 "~" H 7600 5850 50  0001 C CNN
 	1    7600 5850
@@
 F 0 "R39" V 7700 5950 50  0000 C CNN
 F 1 "160" V 7600 5950 50  0000 C CNN
-F 2 "" V 7530 5950 50  0001 C CNN
+F 2 "Resistor_SMD:R_1206_3216Metric_Pad1.42x1.75mm_HandSolder" V 7530 5950 50  0001 C CNN
 F 3 "~" H 7600 5950 50  0001 C CNN
 	1    7600 5950
@@
 F 0 "R40" V 10700 4900 50  0000 C CNN
 F 1 "250" V 10800 4900 50  0000 C CNN
-F 2 "" V 10730 4900 50  0001 C CNN
+F 2 "Resistor_SMD:R_1206_3216Metric_Pad1.42x1.75mm_HandSolder" V 10730 4900 50  0001 C CNN
 F 3 "~" H 10800 4900 50  0001 C CNN
 	1    10800 4900
@@
 F 0 "R41" V 10900 5000 50  0000 C CNN
 F 1 "400" V 10800 5000 50  0000 C CNN
-F 2 "" V 10730 5000 50  0001 C CNN
+F 2 "Resistor_SMD:R_1206_3216Metric_Pad1.42x1.75mm_HandSolder" V 10730 5000 50  0001 C CNN
 F 3 "~" H 10800 5000 50  0001 C CNN
 	1    10800 5000
@@
 F 0 "C1" H 3365 4246 50  0000 L CNN
 F 1 "100u" H 3365 4155 50  0000 L CNN
-F 2 "Capacitor_SMD:C_0805_2012Metric_Pad1.15x1.40mm_HandSolder" H 3288 4050 50  0001 C CNN
+F 2 "Capacitor_SMD:C_1206_3216Metric_Pad1.42x1.75mm_HandSolder" H 3288 4050 50  0001 C CNN
 F 3 "~" H 3250 4200 50  0001 C CNN
 	1    3250 4200

Commit message: Tag you're it. Wired up the DAC, fixed the PSU footprint.
Changed lines of the file:
@@
 F1 "Artix.sch" 50
 F2 "program_b" I L 8150 5150 50
-F3 "IO_L4P_T0_D04_14" O R 10250 5300 50
-F4 "IO_L4N_T0_D05_14" O R 10250 5400 50
-F5 "IO_L5P_T0_D06_14" O R 10250 5500 50
-F6 "IO_L5P_T0_D07_14" O R 10250 5600 50
+F3 "DAC_SCK" O R 10250 5300 50
+F4 "DAC_BCK" O R 10250 5400 50
+F5 "DAC_DATA" O R 10250 5500 50
+F6 "DAC_LRCK" O R 10250 5600 50
 F7 "done" O L 8150 5050 50
 F8 "SPI_MOSI" I L 8150 5300 50

Commit message: Added in the potentiometers, fixed some faulty pins on the artix, rewired some pins on the MCU so they didn't interfere with the crystal.
Connections:
- no-connect marks 3 -> 4
Changed lines of the file:
@@
 Wire Wire Line
 	3250 4750 3350 4750
+NoConn ~ 4300 3100
 $EndSCHEMATC

Commit message: Wired up the potentiometers.
Connections:
- net labels removed: VCC
- wire segments 161 -> 155
Changed lines of the file:
@@
 Wire Wire Line
 	17200 4700 17400 4700
-Wire Wire Line
-	5300 2200 5300 2400
-$Comp
-L power:PWR_FLAG #FLG03
-U 1 1 5DEFDEF4
-P 5300 2200
-F 0 "#FLG03" H 5300 2275 50  0001 C CNN
-F 1 "PWR_FLAG" H 5300 2373 50  0000 C CNN
-F 2 "" H 5300 2200 50  0001 C CNN
-F 3 "~" H 5300 2200 50  0001 C CNN
-	1    5300 2200
-	1    0    0    -1
-$EndComp
-$Comp
-L power:VCC #PWR09
-U 1 1 5DEFCFF5
-P 5300 2400
-F 0 "#PWR09" H 5300 2250 50  0001 C CNN
-F 1 "VCC" H 5318 2573 50  0000 C CNN
-F 2 "" H 5300 2400 50  0001 C CNN
-F 3 "" H 5300 2400 50  0001 C CNN
-	1    5300 2400
-	-1   0    0    1
-$EndComp
 $Comp
 L power:+1V8 #PWR0106
@@
 	0    1    1    0
 $EndComp
-$Comp
-L power:PWR_FLAG #FLG0102
-U 1 1 5E0FA1F8
-P 5700 2200
-F 0 "#FLG0102" H 5700 2275 50  0001 C CNN
-F 1 "PWR_FLAG" H 5700 2373 50  0000 C CNN
-F 2 "" H 5700 2200 50  0001 C CNN
-F 3 "~" H 5700 2200 50  0001 C CNN
-	1    5700 2200
-	1    0    0    -1
-$EndComp
-$Comp
-L power:PWR_FLAG #FLG0103
-U 1 1 5E0FA6DB
-P 6100 2200
-F 0 "#FLG0103" H 6100 2275 50  0001 C CNN
-F 1 "PWR_FLAG" H 6100 2373 50  0000 C CNN
-F 2 "" H 6100 2200 50  0001 C CNN
-F 3 "~" H 6100 2200 50  0001 C CNN
-	1    6100 2200
-	1    0    0    -1
-$EndComp
-$Comp
-L power:PWR_FLAG #FLG0104
-U 1 1 5E0FAA2D
-P 6500 2200
-F 0 "#FLG0104" H 6500 2275 50  0001 C CNN
-F 1 "PWR_FLAG" H 6500 2373 50  0000 C CNN
-F 2 "" H 6500 2200 50  0001 C CNN
-F 3 "~" H 6500 2200 50  0001 C CNN
-	1    6500 2200
-	1    0    0    -1
-$EndComp
-$Comp
-L power:+1V0 #PWR0122
-U 1 1 5E0FB37A
-P 5700 2400
-F 0 "#PWR0122" H 5700 2250 50  0001 C CNN
-F 1 "+1V0" H 5715 2573 50  0000 C CNN
-F 2 "" H 5700 2400 50  0001 C CNN
-F 3 "" H 5700 2400 50  0001 C CNN
-	1    5700 2400
-	-1   0    0    1
-$EndComp
-$Comp
-L power:+3.3V #PWR0123
-U 1 1 5E0FDB7E
-P 6500 2400
-F 0 "#PWR0123" H 6500 2250 50  0001 C CNN
-F 1 "+3.3V" H 6515 2573 50  0000 C CNN
-F 2 "" H 6500 2400 50  0001 C CNN
-F 3 "" H 6500 2400 50  0001 C CNN
-	1    6500 2400
-	-1   0    0    1
-$EndComp
-$Comp
-L power:+1V8 #PWR0124
-U 1 1 5E0FE65C
-P 6100 2400
-F 0 "#PWR0124" H 6100 2250 50  0001 C CNN
-F 1 "+1V8" H 6115 2573 50  0000 C CNN
-F 2 "" H 6100 2400 50  0001 C CNN
-F 3 "" H 6100 2400 50  0001 C CNN
-	1    6100 2400
-	-1   0    0    1
-$EndComp
-$Comp
-L power:PWR_FLAG #FLG0105
-U 1 1 5E0FEA5A
-P 6900 2200
-F 0 "#FLG0105" H 6900 2275 50  0001 C CNN
-F 1 "PWR_FLAG" H 6900 2373 50  0000 C CNN
-F 2 "" H 6900 2200 50  0001 C CNN
-F 3 "~" H 6900 2200 50  0001 C CNN
-	1    6900 2200
-	1    0    0    -1
-$EndComp
-$Comp
-L power:+3.3VA #PWR0125
-U 1 1 5E0FF4FA
-P 6900 2400
-F 0 "#PWR0125" H 6900 2250 50  0001 C CNN
-F 1 "+3.3VA" H 6915 2573 50  0000 C CNN
-F 2 "" H 6900 2400 50  0001 C CNN
-F 3 "" H 6900 2400 50  0001 C CNN
-	1    6900 2400
-	-1   0    0    1
-$EndComp
-Wire Wire Line
-	6900 2200 6900 2400
-Wire Wire Line
-	6500 2200 6500 2400
-Wire Wire Line
-	6100 2200 6100 2400
-Wire Wire Line
-	5700 2200 5700 2400
 $Sheet
 S 9150 8000 2600 1700
@@
 	1250 13250 1250 13800
 Connection ~ 1250 13250
-Wire Wire Line
-	1250 12700 1250 13250
-Connection ~ 1250 12700
-Wire Wire Line
-	1250 12150 1250 12700
 Connection ~ 1250 12150
 Wire Wire Line
@@
 Wire Wire Line
 	3700 4750 3650 4750
-Wire Wire Line
-	4900 2200 4900 2400
-$Comp
-L power:GND #PWR0120
-U 1 1 5E0BBA07
-P 4900 2400
-F 0 "#PWR0120" H 4900 2150 50  0001 C CNN
-F 1 "GND" H 4905 2227 50  0000 C CNN
-F 2 "" H 4900 2400 50  0001 C CNN
-F 3 "" H 4900 2400 50  0001 C CNN
-	1    4900 2400
-	1    0    0    -1
-$EndComp
-$Comp
-L power:PWR_FLAG #FLG0101
-U 1 1 5E0BB0C2
-P 4900 2200
-F 0 "#FLG0101" H 4900 2275 50  0001 C CNN
-F 1 "PWR_FLAG" H 4900 2373 50  0000 C CNN
-F 2 "" H 4900 2200 50  0001 C CNN
-F 3 "~" H 4900 2200 50  0001 C CNN
-	1    4900 2200
-	1    0    0    -1
-$EndComp
 $Comp
 L power:+5V #PWR046
@@
 	3250 4750 3350 4750
 NoConn ~ 4300 3100
+Wire Wire Line
+	1250 12150 1250 12700
+Connection ~ 1250 12700
+Wire Wire Line
+	1250 12700 1250 13250
 $EndSCHEMATC

Commit message: Wire up 1V PSU. Use smaller footprints for small caps.
Parts:
- C2: value 0.1u -> 100n; footprint Capacitor_SMD:C_1206_3216Metric_Pad1.42x1.75mm_HandSolder -> Capacitor_SMD:C_0805_2012Metric_Pad1.15x1.40mm_HandSolder
Connections:
- no-connect marks 4 -> 3
Changed lines of the file:
@@
 Wire Wire Line
 	4750 4550 4650 4550
-$Comp
-L Device:C C2
-U 1 1 5D9626CB
-P 4750 4150
-F 0 "C2" H 4865 4196 50  0000 L CNN
-F 1 "0.1u" H 4865 4105 50  0000 L CNN
-F 2 "Capacitor_SMD:C_1206_3216Metric_Pad1.42x1.75mm_HandSolder" H 4788 4000 50  0001 C CNN
-F 3 "~" H 4750 4150 50  0001 C CNN
-	1    4750 4150
-	1    0    0    -1
-$EndComp
 Wire Wire Line
 	4750 4300 4750 4550
@@
 Wire Wire Line
 	3250 4750 3350 4750
-NoConn ~ 4300 3100
 Wire Wire Line
 	1250 12150 1250 12700
@@
 Wire Wire Line
 	1250 12700 1250 13250
+$Comp
+L Device:C C2
+U 1 1 5D9626CB
+P 4750 4150
+F 0 "C2" H 4865 4196 50  0000 L CNN
+F 1 "100n" H 4865 4105 50  0000 L CNN
+F 2 "Capacitor_SMD:C_0805_2012Metric_Pad1.15x1.40mm_HandSolder" H 4788 4000 50  0001 C CNN
+F 3 "~" H 4750 4150 50  0001 C CNN
+	1    4750 4150
+	1    0    0    -1
+$EndComp
 $EndSCHEMATC

Commit message: Added in a bunch of footprints to the netlist; only missing buttons and some resistors, now.
Parts:
- J1: footprint Connector_USB:USB_A_CNCTech_1001-011-01101_Horizontal -> 1932638-3:TE_1932638-3
Changed lines of the file:
@@
 F 0 "J1" H 2907 5417 50  0000 C CNN
 F 1 "USB_A" H 2907 5326 50  0000 C CNN
-F 2 "Connector_USB:USB_A_CNCTech_1001-011-01101_Horizontal" H 3000 4900 50  0001 C CNN
+F 2 "1932638-3:TE_1932638-3" H 3000 4900 50  0001 C CNN
 F 3 " ~" H 3000 4900 50  0001 C CNN
 	1    2850 4950

Commit message: Removed pull-down resistors.
Parts:
- removed R18, R19, R20, R21, R22, R23, R24, R25, R26, R27, R28, R29, R32, R35, R36, R37: R, Resistor_SMD:R_1206_3216Metric_Pad1.42x1.75mm_HandSolder, symbol Device:R
Other:
- note added: "assuming source = 8mA"
- note removed: "Not sure about this..."
