File: EFM32.sch (KiCad schematic (older format))
At the start: 7 parts

Commit message: Connect the MCU SPI pins to FPGA
Connections:
- net labels added: SPI_CLK, SPI_CS, SPI_MISO, SPI_MOSI
Changed lines of the file:
@@
 Wire Wire Line
 	6950 2100 6950 2200
-Connection ~ 6950 2100
-Connection ~ 6950 2000
-Wire Wire Line
-	6950 2000 6950 2100
-Wire Wire Line
-	6950 1900 6950 2000
-Connection ~ 6950 1900
-Connection ~ 6950 1800
-Wire Wire Line
-	6950 1800 6950 1900
-Wire Wire Line
-	6950 1700 6950 1800
 $Comp
 L Synth:EFM32GG11B4xx U?
@@
 Wire Wire Line
 	1950 2450 1950 2550
+Text HLabel 7100 1800 2    50   Input ~ 0
+SPI_MISO
+Text HLabel 7100 1900 2    50   Output ~ 0
+SPI_CLK
+Text HLabel 7100 2000 2    50   Output ~ 0
+SPI_CS
+Wire Wire Line
+	6950 1700 7100 1700
+Wire Wire Line
+	6950 1800 7100 1800
+Wire Wire Line
+	6950 1900 7100 1900
+Wire Wire Line
+	6950 2000 7100 2000
+Text HLabel 7100 1700 2    50   Output ~ 0
+SPI_MOSI
 $EndSCHEMATC

Commit message: Connect FPGA done and program_b pin to some pins on the MCU
Connections:
- net labels added: FPGA_Ready, FPGA_Reset
Changed lines of the file:
@@
 EESchema Schematic File Version 4
+LIBS:Synthesizer-cache
 EELAYER 30 0
 EELAYER END
@@
 Wire Wire Line
 	6950 2300 6950 2400
-Connection ~ 6950 2300
-Connection ~ 6950 2200
-Wire Wire Line
-	6950 2200 6950 2300
-Wire Wire Line
-	6950 2100 6950 2200
 $Comp
 L Synth:EFM32GG11B4xx U?
@@
 Text HLabel 7100 1700 2    50   Output ~ 0
 SPI_MOSI
+Text HLabel 7100 2100 2    50   Input ~ 0
+FPGA_Ready
+Text HLabel 7100 2200 2    50   Output ~ 0
+FPGA_Reset
+Wire Wire Line
+	6950 2100 7100 2100
+Wire Wire Line
+	6950 2200 7100 2200
 $EndSCHEMATC

Commit message: Add USB symbol and pins
Connections:
- net labels added: USB_D+, USB_D-, USB_VBUS, USB_VBUSEN
- wire segments 79 -> 80
- no-connect marks 6 -> 8
Changed lines of the file:
@@
 	11550 1400 10650 1400
 Wire Wire Line
-	11400 3350 10850 3350
+	12050 3350 10850 3350
 Wire Wire Line
 	10850 3550 10450 3550
@@
 L Synth:EFM32GG11B4xx U?
 U 3 1 5D8D8308
-P 12200 3900
-F 0 "U?" H 12200 4715 50  0000 C CNN
-F 1 "EFM32GG11B4xx" H 12200 4624 50  0000 C CNN
-F 2 "" H 12150 4150 50  0001 C CNN
-F 3 "" H 12150 4150 50  0001 C CNN
-	3    12200 3900
+P 12850 3900
+F 0 "U?" H 12850 4715 50  0000 C CNN
+F 1 "EFM32GG11B4xx" H 12850 4624 50  0000 C CNN
+F 2 "" H 12800 4150 50  0001 C CNN
+F 3 "" H 12800 4150 50  0001 C CNN
+	3    12850 3900
 	-1   0    0    -1
 $EndComp
 Wire Wire Line
-	10450 3450 11400 3450
+	10450 3450 12050 3450
 Wire Wire Line
 	10450 3750 10950 3750
@@
 	10950 3550 10950 3750
 Wire Wire Line
-	10950 3550 11400 3550
-$Comp
-L power:GND #PWR?
-U 1 1 5D8A3029
-P 11400 4400
-AR Path="/5D8A3029" Ref="#PWR?"  Part="1"
-AR Path="/5D8502F2/5D8A3029" Ref="#PWR?"  Part="1"
-F 0 "#PWR?" H 11400 4150 50  0001 C CNN
-F 1 "GND" V 11405 4272 50  0000 R CNN
-F 2 "" H 11400 4400 50  0001 C CNN
-F 3 "" H 11400 4400 50  0001 C CNN
-	1    11400 4400
-	0    1    1    0
-$EndComp
-Wire Wire Line
-	11400 3700 11400 3850
+	10950 3550 12050 3550
 $Comp
 L power:GND #PWR?
 U 1 1 5D9D6555
-P 13000 4600
+P 13650 4600
 AR Path="/5D9D6555" Ref="#PWR?"  Part="1"
 AR Path="/5D8502F2/5D9D6555" Ref="#PWR?"  Part="1"
-F 0 "#PWR?" H 13000 4350 50  0001 C CNN
-F 1 "GND" V 13005 4472 50  0000 R CNN
-F 2 "" H 13000 4600 50  0001 C CNN
-F 3 "" H 13000 4600 50  0001 C CNN
-	1    13000 4600
+F 0 "#PWR?" H 13650 4350 50  0001 C CNN
+F 1 "GND" V 13655 4472 50  0000 R CNN
+F 2 "" H 13650 4600 50  0001 C CNN
+F 3 "" H 13650 4600 50  0001 C CNN
+	1    13650 4600
 	0    -1   1    0
 $EndComp
 Wire Wire Line
-	13000 3350 13000 3450
-Connection ~ 13000 3450
-Wire Wire Line
-	13000 3450 13000 3550
-Connection ~ 13000 3550
-Wire Wire Line
-	13000 3550 13000 3650
-Connection ~ 13000 3650
-Wire Wire Line
-	13000 3650 13000 3800
-Connection ~ 13000 3800
-Wire Wire Line
-	13000 3800 13000 3900
-Connection ~ 13000 3900
-Wire Wire Line
-	13000 3900 13000 4000
-Connection ~ 13000 4000
-Wire Wire Line
-	13000 4000 13000 4100
-Connection ~ 13000 4100
-Wire Wire Line
-	13000 4100 13000 4200
-Connection ~ 13000 4200
-Wire Wire Line
-	13000 4200 13000 4300
-Connection ~ 13000 4300
-Wire Wire Line
-	13000 4300 13000 4400
-Connection ~ 13000 4400
-Wire Wire Line
-	13000 4400 13000 4500
-Connection ~ 13000 4500
-Wire Wire Line
-	13000 4500 13000 4600
-Connection ~ 11400 3850
-Wire Wire Line
-	11400 3850 11400 3950
-Connection ~ 11400 3950
-Wire Wire Line
-	11400 3950 11400 4100
-Connection ~ 11400 4100
-Wire Wire Line
-	11400 4100 11400 4400
+	13650 3350 13650 3450
+Connection ~ 13650 3450
+Wire Wire Line
+	13650 3450 13650 3550
+Connection ~ 13650 3550
+Wire Wire Line
+	13650 3550 13650 3650
+Connection ~ 13650 3650
+Wire Wire Line
+	13650 3650 13650 3800
+Connection ~ 13650 3800
+Wire Wire Line
+	13650 3800 13650 3900
+Connection ~ 13650 3900
+Wire Wire Line
+	13650 3900 13650 4000
+Connection ~ 13650 4000
+Wire Wire Line
+	13650 4000 13650 4100
+Connection ~ 13650 4100
+Wire Wire Line
+	13650 4100 13650 4200
+Connection ~ 13650 4200
+Wire Wire Line
+	13650 4200 13650 4300
+Connection ~ 13650 4300
+Wire Wire Line
+	13650 4300 13650 4400
+Connection ~ 13650 4400
+Wire Wire Line
+	13650 4400 13650 4500
+Connection ~ 13650 4500
+Wire Wire Line
+	13650 4500 13650 4600
 $Comp
 L power:GND #PWR?
@@
 Wire Wire Line
 	6950 2200 7100 2200
+NoConn ~ 11650 2350
+Wire Wire Line
+	11650 2450 11300 2450
+Text HLabel 11300 2650 0    50   Input ~ 0
+USB_VBUS
+Wire Wire Line
+	11650 2650 11300 2650
+$Comp
+L power:+3.3VA #PWR?
+U 1 1 5D907864
+P 11300 2450
+AR Path="/5D907864" Ref="#PWR?"  Part="1"
+AR Path="/5D8502F2/5D907864" Ref="#PWR?"  Part="1"
+F 0 "#PWR?" H 11300 2300 50  0001 C CNN
+F 1 "+3.3VA" V 11315 2577 50  0000 L CNN
+F 2 "" H 11300 2450 50  0001 C CNN
+F 3 "" H 11300 2450 50  0001 C CNN
+	1    11300 2450
+	0    -1   -1   0
+$EndComp
+Text HLabel 11750 3700 0    50   Input ~ 0
+USB_VBUSEN
+Wire Wire Line
+	11750 3700 12050 3700
+Text HLabel 11750 3850 0    50   UnSpc ~ 0
+USB_D-
+Text HLabel 11750 3950 0    50   UnSpc ~ 0
+USB_D+
+NoConn ~ 12050 4100
+Wire Wire Line
+	12050 3850 11750 3850
+Wire Wire Line
+	11750 3950 12050 3950
 $EndSCHEMATC

Commit message: Wired USB-A. Added a capacitor to USB_VBUS in the schematic. No idea what to do about VBUSEN though.
Parts:
- added C?: 1u, symbol Device:C
Connections:
- wire segments 80 -> 82
Other:
- note added: "Why are these passive?"
Changed lines of the file:
@@
 EESchema Schematic File Version 4
-LIBS:Synthesizer-cache
 EELAYER 30 0
 EELAYER END
@@
 Wire Wire Line
 	3550 2200 3550 2350
-$Comp
-L power:GND #PWR?
-U 1 1 5DA083B7
-P 1950 1550
-AR Path="/5DA083B7" Ref="#PWR?"  Part="1"
-AR Path="/5D8502F2/5DA083B7" Ref="#PWR?"  Part="1"
-F 0 "#PWR?" H 1950 1300 50  0001 C CNN
-F 1 "GND" V 1955 1422 50  0000 R CNN
-F 2 "" H 1950 1550 50  0001 C CNN
-F 3 "" H 1950 1550 50  0001 C CNN
-	1    1950 1550
-	0    1    -1   0
-$EndComp
-Wire Wire Line
-	1950 1550 1950 1650
-Connection ~ 1950 1650
-Wire Wire Line
-	1950 1650 1950 1750
-Connection ~ 1950 1750
-Wire Wire Line
-	1950 1750 1950 1850
-Connection ~ 1950 1850
 Wire Wire Line
 	1950 1850 1950 1950
@@
 USB_VBUS
 Wire Wire Line
-	11650 2650 11300 2650
+	11650 2650 11450 2650
 $Comp
 L power:+3.3VA #PWR?
@@
 Wire Wire Line
 	11750 3950 12050 3950
+Connection ~ 1950 1850
+Wire Wire Line
+	1950 1750 1950 1850
+Connection ~ 1950 1750
+Wire Wire Line
+	1950 1650 1950 1750
+$Comp
+L Device:C C?
+U 1 1 5D8E2720
+P 11450 2850
+F 0 "C?" H 11565 2896 50  0000 L CNN
+F 1 "1u" H 11565 2805 50  0000 L CNN
+F 2 "" H 11488 2700 50  0001 C CNN
+F 3 "~" H 11450 2850 50  0001 C CNN
+	1    11450 2850
+	1    0    0    -1
+$EndComp
+$Comp
+L power:GND #PWR?
+U 1 1 5D8E2F22
+P 11450 3050
+F 0 "#PWR?" H 11450 2800 50  0001 C CNN
+F 1 "GND" H 11455 2877 50  0000 C CNN
+F 2 "" H 11450 3050 50  0001 C CNN
+F 3 "" H 11450 3050 50  0001 C CNN
+	1    11450 3050
+	1    0    0    -1
+$EndComp
+Wire Wire Line
+	11450 3000 11450 3050
+Wire Wire Line
+	11450 2700 11450 2650
+Connection ~ 11450 2650
+Wire Wire Line
+	11450 2650 11300 2650
+Text Notes 11050 4050 0    50   ~ 0
+Why are these passive?
 $EndSCHEMATC

Commit message: Added ESD protection to USB-A. Connected Soft-mute.
Parts:
- added FB2: Ferrite_Bead, symbol Device:Ferrite_Bead
- added R33, R34: 15, symbol Device:R
- C5: renamed from C?; value 1u -> 100u
- gave numbers to parts that had none: 4
Connections:
- net labels added: Overcurrent, Soft-mute
- wire segments 82 -> 85
Other:
- note removed: "Why are these passive?"

Commit message: add placeholder footprints, clean up ratsnest a bit
Parts:
- C5: footprint (none) -> Capacitor_SMD:C_0805_2012Metric_Pad1.15x1.40mm_HandSolder
- FB2: footprint (none) -> Inductor_SMD:L_0805_2012Metric_Pad1.15x1.40mm_HandSolder
- R33, R34: footprint (none) -> Resistor_SMD:R_0805_2012Metric_Pad1.15x1.40mm_HandSolder
- U7: footprint (none) -> Package_QFP:TQFP-64_10x10mm_P0.5mm
Changed lines of the file:
@@
 EESchema Schematic File Version 4
+LIBS:Synthesizer-cache
 EELAYER 30 0
 EELAYER END
@@
 F 0 "U7" H 12150 2600 50  0000 C CNN
 F 1 "EFM32GG11B4xx" H 12150 2500 50  0000 C CNN
-F 2 "" H 12100 2100 50  0001 C CNN
+F 2 "Package_QFP:TQFP-64_10x10mm_P0.5mm" H 12100 2100 50  0001 C CNN
 F 3 "" H 12100 2100 50  0001 C CNN
 	4    12150 1850
@@
 F 0 "U7" H 12850 4715 50  0000 C CNN
 F 1 "EFM32GG11B4xx" H 12850 4624 50  0000 C CNN
-F 2 "" H 12800 4150 50  0001 C CNN
+F 2 "Package_QFP:TQFP-64_10x10mm_P0.5mm" H 12800 4150 50  0001 C CNN
 F 3 "" H 12800 4150 50  0001 C CNN
 	3    12850 3900
@@
 F 0 "U7" H 6150 2665 50  0000 C CNN
 F 1 "EFM32GG11B4xx" H 6150 2574 50  0000 C CNN
-F 2 "" H 6100 2300 50  0001 C CNN
+F 2 "Package_QFP:TQFP-64_10x10mm_P0.5mm" H 6100 2300 50  0001 C CNN
 F 3 "" H 6100 2300 50  0001 C CNN
 	2    6150 2050
@@
 F 0 "C5" H 11565 2896 50  0000 L CNN
 F 1 "100u" H 11565 2805 50  0000 L CNN
-F 2 "" H 11488 2700 50  0001 C CNN
+F 2 "Capacitor_SMD:C_0805_2012Metric_Pad1.15x1.40mm_HandSolder" H 11488 2700 50  0001 C CNN
 F 3 "~" H 11450 2850 50  0001 C CNN
 	1    11450 2850
@@
 F 0 "R33" V 11450 3850 50  0000 C CNN
 F 1 "15" V 11550 3850 50  0000 C CNN
-F 2 "" V 11480 3850 50  0001 C CNN
+F 2 "Resistor_SMD:R_0805_2012Metric_Pad1.15x1.40mm_HandSolder" V 11480 3850 50  0001 C CNN
 F 3 "~" H 11550 3850 50  0001 C CNN
 	1    11550 3850
@@
 F 0 "R34" V 11650 3950 50  0000 C CNN
 F 1 "15" V 11550 3950 50  0000 C CNN
-F 2 "" V 11480 3950 50  0001 C CNN
+F 2 "Resistor_SMD:R_0805_2012Metric_Pad1.15x1.40mm_HandSolder" V 11480 3950 50  0001 C CNN
 F 3 "~" H 11550 3950 50  0001 C CNN
 	1    11550 3950
@@
 F 0 "FB2" V 10826 2650 50  0000 C CNN
 F 1 "Ferrite_Bead" V 10917 2650 50  0000 C CNN
-F 2 "" V 11030 2650 50  0001 C CNN
+F 2 "Inductor_SMD:L_0805_2012Metric_Pad1.15x1.40mm_HandSolder" V 11030 2650 50  0001 C CNN
 F 3 "~" H 11100 2650 50  0001 C CNN
 	1    11100 2650
@@
 F 0 "U7" H 2750 2715 50  0000 C CNN
 F 1 "EFM32GG11B4xx" H 2750 2624 50  0000 C CNN
-F 2 "" H 2700 2300 50  0001 C CNN
+F 2 "Package_QFP:TQFP-64_10x10mm_P0.5mm" H 2700 2300 50  0001 C CNN
 F 3 "" H 2700 2300 50  0001 C CNN
 	1    2750 2050

Commit message: Connect buttons and move MCU->FPGA done/program_b pins
Parts:
- U7: footprint Package_QFP:TQFP-64_10x10mm_P0.5mm -> (none)
Connections:
- net labels added: Button0, Button1, Button10, Button11, Button12, Button13, Button14, Button15, Button2, Button3, Button4, Button5, Button6, Button7, Button8, Button9
- wire segments 85 -> 91
Changed lines of the file:
@@
 L Device:Crystal Y?
 U 1 1 5D884D58
-P 4050 2550
+P 4050 2600
 AR Path="/5D884D58" Ref="Y?"  Part="1"
 AR Path="/5D8502F2/5D884D58" Ref="Y1"  Part="1"
-F 0 "Y1" H 4050 2282 50  0000 C CNN
-F 1 "48Mhz" H 4050 2373 50  0000 C CNN
-F 2 "Crystal:Crystal_DS10_D1.0mm_L4.3mm_Vertical" H 4050 2550 50  0001 C CNN
-F 3 "~" H 4050 2550 50  0001 C CNN
-	1    4050 2550
+F 0 "Y1" V 4100 2850 50  0000 C CNN
+F 1 "48Mhz" V 4000 2850 50  0000 C CNN
+F 2 "Crystal:Crystal_DS10_D1.0mm_L4.3mm_Vertical" H 4050 2600 50  0001 C CNN
+F 3 "~" H 4050 2600 50  0001 C CNN
+	1    4050 2600
 	0    1    1    0
 $EndComp
 Wire Wire Line
-	4050 2700 3800 2700
-Wire Wire Line
-	3800 2700 3800 2600
+	4050 2750 3800 2750
+Wire Wire Line
+	3800 2750 3800 2600
 Wire Wire Line
 	3800 2600 3550 2600
 Wire Wire Line
-	3800 2500 3800 2400
-Wire Wire Line
-	3800 2400 4050 2400
+	3800 2500 3800 2450
+Wire Wire Line
+	3800 2450 4050 2450
 Wire Wire Line
 	3800 2500 3550 2500
@@
 Text HLabel 7100 1700 2    50   Output ~ 0
 SPI_MOSI
-Text HLabel 7100 2100 2    50   Input ~ 0
+Text HLabel 5200 2050 0    50   Input ~ 0
 FPGA_Ready
-Text HLabel 7100 2200 2    50   Output ~ 0
+Text HLabel 5200 1950 0    50   Output ~ 0
 FPGA_Reset
 Wire Wire Line
-	6950 2100 7100 2100
-Wire Wire Line
-	6950 2200 7100 2200
+	5350 2050 5200 2050
+Wire Wire Line
+	5350 1950 5200 1950
 NoConn ~ 11650 2350
 Wire Wire Line
@@
 Wire Wire Line
 	10950 2650 10350 2650
-Connection ~ 1950 2450
-Wire Wire Line
-	1950 2450 1950 2550
-Wire Wire Line
-	1950 2350 1950 2450
-Connection ~ 1950 2350
-Connection ~ 1950 2150
-Wire Wire Line
-	1950 2150 1950 2350
-Wire Wire Line
-	1950 2050 1950 2150
-Connection ~ 1950 2050
-Connection ~ 1950 1950
-Wire Wire Line
-	1950 1950 1950 2050
-Wire Wire Line
-	1950 1850 1950 1950
-Wire Wire Line
-	3550 2200 3550 2350
-Connection ~ 3550 2200
-Connection ~ 3550 2100
-Wire Wire Line
-	3550 2100 3550 2200
-Wire Wire Line
-	3550 1950 3550 2100
-Connection ~ 3550 1950
-Connection ~ 3550 1850
-Wire Wire Line
-	3550 1850 3550 1950
-Wire Wire Line
-	3550 1750 3550 1850
-Connection ~ 3550 1750
-Connection ~ 3550 1650
-Wire Wire Line
-	3550 1650 3550 1750
-Wire Wire Line
-	3550 1550 3550 1650
+Text HLabel 1650 1650 0    50   Output ~ 0
+Overcurrent
+Text HLabel 1650 1750 0    50   Output ~ 0
+Soft-mute
+Wire Wire Line
+	1950 1750 1650 1750
+Wire Wire Line
+	1650 1650 1950 1650
+Wire Wire Line
+	6950 1700 7100 1700
+Text HLabel 1650 1850 0    50   BiDi ~ 0
+Button0
+Text HLabel 1650 1950 0    50   BiDi ~ 0
+Button1
+Text HLabel 1650 2050 0    50   BiDi ~ 0
+Button2
+Text HLabel 1650 2150 0    50   BiDi ~ 0
+Button3
+Text HLabel 3750 1750 2    50   BiDi ~ 0
+Button5
+Text HLabel 3750 1650 2    50   BiDi ~ 0
+Button4
+Text HLabel 3750 1850 2    50   BiDi ~ 0
+Button6
+Text HLabel 3750 1950 2    50   BiDi ~ 0
+Button7
+Wire Wire Line
+	6950 2500 6950 2600
+Connection ~ 6950 2500
+Wire Wire Line
+	6950 2400 6950 2500
+Wire Wire Line
+	6950 2300 6950 2400
+Connection ~ 6950 2400
+$Comp
+L Synth:EFM32GG11B4xx U7
+U 2 1 5D8D4390
+P 6150 2050
+F 0 "U7" H 6150 2665 50  0000 C CNN
+F 1 "EFM32GG11B4xx" H 6150 2574 50  0000 C CNN
+F 2 "" H 6100 2300 50  0001 C CNN
+F 3 "" H 6100 2300 50  0001 C CNN
+	2    6150 2050
+	1    0    0    -1
+$EndComp
+Text HLabel 5200 1700 0    50   BiDi ~ 0
+Button8
+Text HLabel 5200 1800 0    50   BiDi ~ 0
+Button9
+Text HLabel 3750 2100 2    50   BiDi ~ 0
+Button10
+Text HLabel 3750 2200 2    50   BiDi ~ 0
+Button11
+Text HLabel 3750 2350 2    50   BiDi ~ 0
+Button15
+Text HLabel 1650 2350 0    50   BiDi ~ 0
+Button12
+Text HLabel 1650 2450 0    50   BiDi ~ 0
+Button13
+Text HLabel 1650 2550 0    50   BiDi ~ 0
+Button14
 $Comp
 L Synth:EFM32GG11B4xx U7
@@
 	1    0    0    -1
 $EndComp
-Text HLabel 1650 1650 0    50   Output ~ 0
-Overcurrent
-Text HLabel 1650 1750 0    50   Output ~ 0
-Soft-mute
-Wire Wire Line
-	1950 1750 1650 1750
-Wire Wire Line
-	1650 1650 1950 1650
-Wire Wire Line
-	6950 1700 7100 1700
+Wire Wire Line
+	1650 1850 1950 1850
+Wire Wire Line
+	1950 1950 1650 1950
+Wire Wire Line
+	1650 2050 1950 2050
+Wire Wire Line
+	1950 2150 1650 2150
+Wire Wire Line
+	1650 2350 1950 2350
+Wire Wire Line
+	1950 2450 1650 2450
+Wire Wire Line
+	1650 2550 1950 2550
+Wire Wire Line
+	3550 1650 3750 1650
+Wire Wire Line
+	3550 1750 3750 1750
+Wire Wire Line
+	3550 1850 3750 1850
+Wire Wire Line
+	3550 1950 3750 1950
+Wire Wire Line
+	3550 2100 3750 2100
+Wire Wire Line
+	3550 2200 3750 2200
+Wire Wire Line
+	3550 2350 3750 2350
+Wire Wire Line
+	5200 1700 5350 1700
+Wire Wire Line
+	5350 1800 5200 1800
 $EndSCHEMATC
