File: EFM32.sch (KiCad schematic (older format))
At the start: 8 parts, among them J5 MCU_debug, U7 EFM32GG11B4xx, Y1 48Mhz

Commit message: Added NPN transistor on USB and wired shield. Added LEDs, debug pins.
Parts:
- U7: footprint (none) -> Package_QFP:TQFP-64_10x10mm_P0.5mm
Connections:
- net labels added: FPGA_extra_1, FPGA_extra_2, FPGA_extra_3, FPGA_extra_4, GREEN_LED, RED_LED
- wire segments 91 -> 88
Other:
- note added: "TODO: potensiometer"
Changed lines of the file:
@@
 Wire Wire Line
 	3800 2500 3550 2500
-Wire Wire Line
-	11300 2100 11550 2100
-$Comp
-L power:+3.3VA #PWR?
-U 1 1 5D8A3009
-P 11550 1600
-AR Path="/5D8A3009" Ref="#PWR?"  Part="1"
-AR Path="/5D8502F2/5D8A3009" Ref="#PWR034"  Part="1"
-F 0 "#PWR034" H 11550 1450 50  0001 C CNN
-F 1 "+3.3VA" V 11565 1727 50  0000 L CNN
-F 2 "" H 11550 1600 50  0001 C CNN
-F 3 "" H 11550 1600 50  0001 C CNN
-	1    11550 1600
-	0    -1   -1   0
-$EndComp
 $Comp
 L power:+3.3V #PWR?
@@
 	0    -1   -1   0
 $EndComp
-$Comp
-L power:PWR_FLAG #FLG?
-U 1 1 5D8A301C
-P 12850 1400
-AR Path="/5D8A301C" Ref="#FLG?"  Part="1"
-AR Path="/5D8502F2/5D8A301C" Ref="#FLG01"  Part="1"
-F 0 "#FLG01" H 12850 1475 50  0001 C CNN
-F 1 "PWR_FLAG" H 12850 1573 50  0000 C CNN
-F 2 "" H 12850 1400 50  0001 C CNN
-F 3 "~" H 12850 1400 50  0001 C CNN
-	1    12850 1400
-	1    0    0    -1
-$EndComp
 $Sheet
 S 13200 8050 2050 1300
@@
 F1 "MCUDecouplers.sch" 50
 $EndSheet
-Wire Wire Line
-	12850 1400 12950 1400
-Wire Wire Line
-	13200 2100 12850 2100
 $Comp
 L power:GND #PWR?
@@
 	0    1    1    0
 $EndComp
-Wire Wire Line
-	13200 1600 12850 1600
 $Comp
 L Device:C C?
@@
 	0    -1   -1   0
 $EndComp
-Wire Wire Line
-	11550 1600 11550 1700
-Connection ~ 11550 1600
-Connection ~ 12850 1400
-Wire Wire Line
-	12850 1600 12850 1700
-Wire Wire Line
-	12850 1700 12850 1800
-Connection ~ 12850 1600
-Connection ~ 12850 1700
-Wire Wire Line
-	12850 2100 12850 2200
-Wire Wire Line
-	12850 2200 12850 2300
-Connection ~ 12850 2100
-Connection ~ 12850 2200
-$Comp
-L Synth:EFM32GG11B4xx U7
-U 4 1 5D8DB9AF
-P 12150 1850
-F 0 "U7" H 12150 2600 50  0000 C CNN
-F 1 "EFM32GG11B4xx" H 12150 2500 50  0000 C CNN
-F 2 "Package_QFP:TQFP-64_10x10mm_P0.5mm" H 12100 2100 50  0001 C CNN
-F 3 "" H 12100 2100 50  0001 C CNN
-	4    12150 1850
-	1    0    0    -1
-$EndComp
 $Comp
 L power:+3.3V #PWR?
@@
 	10650 1400 10650 3850
 Wire Wire Line
-	11550 1400 10650 1400
-Wire Wire Line
 	12050 3350 10850 3350
 Wire Wire Line
@@
 $EndComp
 Wire Wire Line
-	13650 3350 13650 3450
-Connection ~ 13650 3450
-Wire Wire Line
-	13650 3450 13650 3550
-Connection ~ 13650 3550
-Wire Wire Line
-	13650 3550 13650 3650
-Connection ~ 13650 3650
-Wire Wire Line
-	13650 3650 13650 3800
-Connection ~ 13650 3800
-Wire Wire Line
 	13650 3800 13650 3900
 Connection ~ 13650 3900
@@
 L power:GND #PWR?
 U 1 1 5D9DF256
-P 6950 2600
+P 7150 2500
 AR Path="/5D9DF256" Ref="#PWR?"  Part="1"
 AR Path="/5D8502F2/5D9DF256" Ref="#PWR025"  Part="1"
-F 0 "#PWR025" H 6950 2350 50  0001 C CNN
-F 1 "GND" V 6955 2472 50  0000 R CNN
-F 2 "" H 6950 2600 50  0001 C CNN
-F 3 "" H 6950 2600 50  0001 C CNN
-	1    6950 2600
+F 0 "#PWR025" H 7150 2250 50  0001 C CNN
+F 1 "GND" V 7155 2372 50  0000 R CNN
+F 2 "" H 7150 2500 50  0001 C CNN
+F 3 "" H 7150 2500 50  0001 C CNN
+	1    7150 2500
 	0    -1   1    0
-$EndComp
-Wire Wire Line
-	6950 2500 6950 2600
-Connection ~ 6950 2500
-Connection ~ 6950 2400
-Wire Wire Line
-	6950 2400 6950 2500
-Wire Wire Line
-	6950 2300 6950 2400
-$Comp
-L Synth:EFM32GG11B4xx U7
-U 2 1 5D8D4390
-P 6150 2050
-F 0 "U7" H 6150 2665 50  0000 C CNN
-F 1 "EFM32GG11B4xx" H 6150 2574 50  0000 C CNN
-F 2 "Package_QFP:TQFP-64_10x10mm_P0.5mm" H 6100 2300 50  0001 C CNN
-F 3 "" H 6100 2300 50  0001 C CNN
-	2    6150 2050
-	1    0    0    -1
 $EndComp
 $Comp
@@
 	0    1    1    0
 $EndComp
-Wire Wire Line
-	5350 1700 5350 1800
-Connection ~ 5350 1800
-Wire Wire Line
-	5350 1800 5350 1950
-Connection ~ 5350 1950
-Wire Wire Line
-	5350 1950 5350 2050
-Connection ~ 5350 2050
-Wire Wire Line
-	5350 2050 5350 2400
 $Comp
 L power:GND #PWR?
@@
 Text HLabel 7100 2000 2    50   Output ~ 0
 SPI_CS
-Wire Wire Line
-	6950 1800 7100 1800
-Wire Wire Line
-	6950 1900 7100 1900
-Wire Wire Line
-	6950 2000 7100 2000
 Text HLabel 7100 1700 2    50   Output ~ 0
 SPI_MOSI
@@
 Text HLabel 5200 1950 0    50   Output ~ 0
 FPGA_Reset
-Wire Wire Line
-	5350 2050 5200 2050
-Wire Wire Line
-	5350 1950 5200 1950
-NoConn ~ 11650 2350
-Wire Wire Line
-	11650 2450 11300 2450
 Text HLabel 10350 2650 0    50   Input ~ 0
 USB_VBUS
-Wire Wire Line
-	11650 2650 11450 2650
 $Comp
 L power:+3.3VA #PWR?
@@
 Wire Wire Line
 	1650 1650 1950 1650
-Wire Wire Line
-	6950 1700 7100 1700
 Text HLabel 1650 1850 0    50   BiDi ~ 0
 Button0
@@
 Text HLabel 3750 1950 2    50   BiDi ~ 0
 Button7
-Wire Wire Line
-	6950 2500 6950 2600
-Connection ~ 6950 2500
-Wire Wire Line
-	6950 2400 6950 2500
-Wire Wire Line
-	6950 2300 6950 2400
-Connection ~ 6950 2400
-$Comp
-L Synth:EFM32GG11B4xx U7
-U 2 1 5D8D4390
-P 6150 2050
-F 0 "U7" H 6150 2665 50  0000 C CNN
-F 1 "EFM32GG11B4xx" H 6150 2574 50  0000 C CNN
-F 2 "" H 6100 2300 50  0001 C CNN
-F 3 "" H 6100 2300 50  0001 C CNN
-	2    6150 2050
-	1    0    0    -1
-$EndComp
 Text HLabel 5200 1700 0    50   BiDi ~ 0
 Button8
@@
 Wire Wire Line
 	3550 2350 3750 2350
+Connection ~ 12850 2100
+Wire Wire Line
+	13200 2100 12850 2100
+Connection ~ 12850 1600
+Wire Wire Line
+	13200 1600 12850 1600
+Wire Wire Line
+	11650 2650 11450 2650
+Wire Wire Line
+	11650 2450 11300 2450
+NoConn ~ 11650 2350
+Connection ~ 12850 1400
+Wire Wire Line
+	12850 1400 12950 1400
+$Comp
+L power:PWR_FLAG #FLG?
+U 1 1 5D8A301C
+P 12850 1400
+AR Path="/5D8A301C" Ref="#FLG?"  Part="1"
+AR Path="/5D8502F2/5D8A301C" Ref="#FLG01"  Part="1"
+F 0 "#FLG01" H 12850 1475 50  0001 C CNN
+F 1 "PWR_FLAG" H 12850 1573 50  0000 C CNN
+F 2 "" H 12850 1400 50  0001 C CNN
+F 3 "~" H 12850 1400 50  0001 C CNN
+	1    12850 1400
+	1    0    0    -1
+$EndComp
+Wire Wire Line
+	11300 2100 11550 2100
+Connection ~ 12850 1700
+Wire Wire Line
+	12850 1700 12850 1800
+Wire Wire Line
+	12850 1600 12850 1700
+Connection ~ 12850 2200
+Wire Wire Line
+	12850 2200 12850 2300
+Wire Wire Line
+	12850 2100 12850 2200
+Wire Wire Line
+	11550 1400 10650 1400
+$Comp
+L Synth:EFM32GG11B4xx U7
+U 4 1 5D8DB9AF
+P 12150 1850
+F 0 "U7" H 12150 2600 50  0000 C CNN
+F 1 "EFM32GG11B4xx" H 12150 2500 50  0000 C CNN
+F 2 "Package_QFP:TQFP-64_10x10mm_P0.5mm" H 12100 2100 50  0001 C CNN
+F 3 "" H 12100 2100 50  0001 C CNN
+	4    12150 1850
+	1    0    0    -1
+$EndComp
+Connection ~ 11550 1600
+Wire Wire Line
+	11550 1600 11550 1700
+$Comp
+L power:+3.3VA #PWR?
+U 1 1 5D8A3009
+P 11550 1600
+AR Path="/5D8A3009" Ref="#PWR?"  Part="1"
+AR Path="/5D8502F2/5D8A3009" Ref="#PWR034"  Part="1"
+F 0 "#PWR034" H 11550 1450 50  0001 C CNN
+F 1 "+3.3VA" V 11565 1727 50  0000 L CNN
+F 2 "" H 11550 1600 50  0001 C CNN
+F 3 "" H 11550 1600 50  0001 C CNN
+	1    11550 1600
+	0    -1   -1   0
+$EndComp
+Text HLabel 7200 2300 2    50   Output ~ 0
+RED_LED
+Text HLabel 7200 2400 2    50   Output ~ 0
+GREEN_LED
+Wire Wire Line
+	5350 2050 5200 2050
+Wire Wire Line
+	5350 2050 5350 2400
+Connection ~ 5350 2050
+Wire Wire Line
+	5350 1950 5200 1950
+Wire Wire Line
+	5350 1950 5350 2050
+Connection ~ 5350 1950
+Wire Wire Line
+	6950 2500 7150 2500
+Wire Wire Line
+	6950 2000 7100 2000
+Wire Wire Line
+	6950 1900 7100 1900
+Wire Wire Line
+	6950 1800 7100 1800
+Wire Wire Line
+	6950 1700 7100 1700
+Wire Wire Line
+	5350 1800 5200 1800
+Wire Wire Line
+	5350 1800 5350 1950
+Connection ~ 5350 1800
 Wire Wire Line
 	5200 1700 5350 1700
 Wire Wire Line
-	5350 1800 5200 1800
+	5350 1700 5350 1800
+$Comp
+L Synth:EFM32GG11B4xx U7
+U 2 1 5D8D4390
+P 6150 2050
+F 0 "U7" H 6150 2665 50  0000 C CNN
+F 1 "EFM32GG11B4xx" H 6150 2574 50  0000 C CNN
+F 2 "Package_QFP:TQFP-64_10x10mm_P0.5mm" H 6100 2300 50  0001 C CNN
+F 3 "" H 6100 2300 50  0001 C CNN
+	2    6150 2050
+	1    0    0    -1
+$EndComp
+Wire Wire Line
+	6950 2400 7200 2400
+Wire Wire Line
+	7200 2300 6950 2300
+Text HLabel 13850 3350 2    50   Output ~ 0
+FPGA_extra_1
+Text HLabel 13850 3450 2    50   Output ~ 0
+FPGA_extra_2
+Text HLabel 13850 3550 2    50   Output ~ 0
+FPGA_extra_3
+Text HLabel 13850 3650 2    50   Output ~ 0
+FPGA_extra_4
+Wire Wire Line
+	13650 3650 13850 3650
+Wire Wire Line
+	13850 3550 13650 3550
+Wire Wire Line
+	13650 3450 13850 3450
+Wire Wire Line
+	13850 3350 13650 3350
+Text Notes 7100 2200 0    50   ~ 0
+TODO: potensiometer
 $EndSCHEMATC

Commit message: Fixed buttons, FPGA wires that were accidentally connected to GND.
Connections:
- wire segments 88 -> 84
Changed lines of the file:
@@
 	0    -1   1    0
-$EndComp
-$Comp
-L power:GND #PWR?
-U 1 1 5D9E9467
-P 5350 2400
-AR Path="/5D9E9467" Ref="#PWR?"  Part="1"
-AR Path="/5D8502F2/5D9E9467" Ref="#PWR024"  Part="1"
-F 0 "#PWR024" H 5350 2150 50  0001 C CNN
-F 1 "GND" V 5355 2272 50  0000 R CNN
-F 2 "" H 5350 2400 50  0001 C CNN
-F 3 "" H 5350 2400 50  0001 C CNN
-	1    5350 2400
-	0    1    1    0
-$EndComp
-$Comp
-L power:GND #PWR?
-U 1 1 5D9FC703
-P 3550 1550
-AR Path="/5D9FC703" Ref="#PWR?"  Part="1"
-AR Path="/5D8502F2/5D9FC703" Ref="#PWR023"  Part="1"
-F 0 "#PWR023" H 3550 1300 50  0001 C CNN
-F 1 "GND" V 3555 1422 50  0000 R CNN
-F 2 "" H 3550 1550 50  0001 C CNN
-F 3 "" H 3550 1550 50  0001 C CNN
-	1    3550 1550
-	0    -1   -1   0
 $EndComp
 Text HLabel 7100 1800 2    50   Input ~ 0
@@
 	5350 2050 5200 2050
 Wire Wire Line
-	5350 2050 5350 2400
-Connection ~ 5350 2050
-Wire Wire Line
 	5350 1950 5200 1950
 Wire Wire Line
-	5350 1950 5350 2050
-Connection ~ 5350 1950
-Wire Wire Line
 	6950 2500 7150 2500
 Wire Wire Line
@@
 	5350 1800 5200 1800
 Wire Wire Line
-	5350 1800 5350 1950
-Connection ~ 5350 1800
-Wire Wire Line
 	5200 1700 5350 1700
-Wire Wire Line
-	5350 1700 5350 1800
 $Comp
 L Synth:EFM32GG11B4xx U7

Commit message: Add header for MCU GPIO
Parts:
- added J6: 67997-410HLF, footprints:67997-410HLF, symbol Header:67997-410HLF
Connections:
- wire segments 84 -> 110
Other:
- moved on the sheet: C5, C6

Commit message: Fix USB connections and various cleanup
Parts:
- removed R33, R34: 15, Resistor_SMD:R_0805_2012Metric_Pad1.15x1.40mm_HandSolder, symbol Device:R
Connections:
- wire segments 110 -> 107
Changed lines of the file:
@@
 AR Path="/5D8502F2/5D8A3009" Ref="#PWR034"  Part="1"
 F 0 "#PWR034" H 4100 3950 50  0001 C CNN
-F 1 "+3.3VA" V 4115 4227 50  0000 L CNN
+F 1 "+3.3VA" H 3800 4100 50  0000 L CNN
 F 2 "" H 4100 4100 50  0001 C CNN
 F 3 "" H 4100 4100 50  0001 C CNN
 	1    4100 4100
-	0    -1   -1   0
+	1    0    0    -1
 $EndComp
 $Comp
@@
 AR Path="/5D8502F2/5D8A300F" Ref="#PWR028"  Part="1"
 F 0 "#PWR028" H 3850 4450 50  0001 C CNN
-F 1 "+3.3V" V 3865 4728 50  0000 L CNN
+F 1 "+3.3V" H 3750 4550 50  0000 L CNN
 F 2 "" H 3850 4600 50  0001 C CNN
 F 3 "" H 3850 4600 50  0001 C CNN
 	1    3850 4600
-	0    -1   -1   0
+	1    0    0    -1
 $EndComp
 $Comp
@@
 Wire Wire Line
 	5400 3900 5500 3900
-Wire Wire Line
-	5750 4600 5400 4600
 $Comp
 L power:GND #PWR?
 U 1 1 5D8A3015
-P 5750 4600
+P 5400 4850
 AR Path="/5D8A3015" Ref="#PWR?"  Part="1"
 AR Path="/5D8502F2/5D8A3015" Ref="#PWR039"  Part="1"
-F 0 "#PWR039" H 5750 4350 50  0001 C CNN
-F 1 "GND" H 5755 4427 50  0000 C CNN
-F 2 "" H 5750 4600 50  0001 C CNN
-F 3 "" H 5750 4600 50  0001 C CNN
-	1    5750 4600
-	0    -1   -1   0
+F 0 "#PWR039" H 5400 4600 50  0001 C CNN
+F 1 "GND" H 5405 4677 50  0000 C CNN
+F 2 "" H 5400 4850 50  0001 C CNN
+F 3 "" H 5400 4850 50  0001 C CNN
+	1    5400 4850
+	1    0    0    -1
 $EndComp
 $Comp
@@
 AR Path="/5D8A2FF5" Ref="C?"  Part="1"
 AR Path="/5D8502F2/5D8A2FF5" Ref="C6"  Part="1"
-F 0 "C6" H 5700 4000 50  0000 L CNN
-F 1 "1u" H 5700 3800 50  0000 L CNN
+F 0 "C6" V 5600 3950 50  0000 L CNN
+F 1 "1u" V 5600 3750 50  0000 L CNN
 F 2 "Capacitor_SMD:C_0805_2012Metric_Pad1.15x1.40mm_HandSolder" H 5688 3750 50  0001 C CNN
 F 3 "~" H 5650 3900 50  0001 C CNN
@@
 Wire Wire Line
 	5400 4700 5400 4800
-Connection ~ 5400 4600
 Connection ~ 5400 4700
 $Comp
@@
 AR Path="/5D8502F2/5D907864" Ref="#PWR030"  Part="1"
 F 0 "#PWR030" H 3850 4800 50  0001 C CNN
-F 1 "+3.3VA" V 3865 5077 50  0000 L CNN
+F 1 "+3.3VA" H 3750 4900 50  0000 L CNN
 F 2 "" H 3850 4950 50  0001 C CNN
 F 3 "" H 3850 4950 50  0001 C CNN
 	1    3850 4950
-	0    -1   -1   0
+	1    0    0    -1
 $EndComp
 $Comp
@@
 Wire Wire Line
 	5350 1950 5200 1950
-Connection ~ 6950 2400
-Wire Wire Line
-	6950 2300 6950 2400
-Connection ~ 6950 2300
 Wire Wire Line
 	6950 2200 6950 2100
@@
 Wire Wire Line
 	6200 6750 6450 6750
-Wire Wire Line
-	4250 6700 4600 6700
-Wire Wire Line
-	4250 6600 4600 6600
-Wire Wire Line
-	3850 6600 3950 6600
-Wire Wire Line
-	3950 6700 3850 6700
-$Comp
-L Device:R R34
-U 1 1 5D8F8046
-P 4100 6700
-F 0 "R34" V 4200 6700 50  0000 C CNN
-F 1 "15" V 4100 6700 50  0000 C CNN
-F 2 "Resistor_SMD:R_0805_2012Metric_Pad1.15x1.40mm_HandSolder" V 4030 6700 50  0001 C CNN
-F 3 "~" H 4100 6700 50  0001 C CNN
-	1    4100 6700
-	0    1    1    0
-$EndComp
-$Comp
-L Device:R R33
-U 1 1 5D8F7A40
-P 4100 6600
-F 0 "R33" V 4000 6600 50  0000 C CNN
-F 1 "15" V 4100 6600 50  0000 C CNN
-F 2 "Resistor_SMD:R_0805_2012Metric_Pad1.15x1.40mm_HandSolder" V 4030 6600 50  0001 C CNN
-F 3 "~" H 4100 6600 50  0001 C CNN
-	1    4100 6600
-	0    1    1    0
-$EndComp
 $Comp
 L power:GND #PWR032
@@
 $EndComp
 NoConn ~ 4600 6850
-Text HLabel 3850 6700 0    50   UnSpc ~ 0
-USB_D+
-Text HLabel 3850 6600 0    50   UnSpc ~ 0
-USB_D-
 Wire Wire Line
 	4300 6450 4600 6450
@@
 Wire Wire Line
 	2300 3900 4100 3900
+Wire Wire Line
+	5400 4850 5400 4800
+Connection ~ 5400 4800
+Entry Wire Line
+	10100 6050 10200 6150
+Text HLabel 4300 6700 0    50   UnSpc ~ 0
+USB_D+
+Text HLabel 4300 6600 0    50   UnSpc ~ 0
+USB_D-
+Wire Wire Line
+	4300 6600 4600 6600
+Wire Wire Line
+	4600 6700 4300 6700
 $EndSCHEMATC

Commit message: Fixed LED bugs again. I think it's right now.
Connections:
- wire segments 107 -> 106
Other:
- note added: "why the PWR_FLAG?"
Changed lines of the file:
@@
 	5350 1950 5200 1950
-Wire Wire Line
-	6950 2200 6950 2100
 Wire Wire Line
 	6950 2000 7100 2000
@@
 Wire Wire Line
 	4600 6700 4300 6700
+Text Notes 5000 3650 0    50   ~ 0
+why the PWR_FLAG?
 $EndSCHEMATC

Commit message: Updated component footprints. The PCB is now an unholy mess.
Parts:
- C5, C6: footprint Capacitor_SMD:C_0805_2012Metric_Pad1.15x1.40mm_HandSolder -> Capacitor_SMD:C_1206_3216Metric_Pad1.42x1.75mm_HandSolder
- FB2: footprint Inductor_SMD:L_0805_2012Metric_Pad1.15x1.40mm_HandSolder -> footprints:FerriteBead_74279215
- Y1: footprint Crystal:Crystal_DS10_D1.0mm_L4.3mm_Vertical -> footprints:Crystal_SMD_Abracon_L11.4mm_W4.70mm_2pin
Changed lines of the file:
@@
 F 0 "Y1" V 4100 2850 50  0000 C CNN
 F 1 "48Mhz" V 4000 2850 50  0000 C CNN
-F 2 "Crystal:Crystal_DS10_D1.0mm_L4.3mm_Vertical" H 4050 2600 50  0001 C CNN
+F 2 "footprints:Crystal_SMD_Abracon_L11.4mm_W4.70mm_2pin" H 4050 2600 50  0001 C CNN
 F 3 "~" H 4050 2600 50  0001 C CNN
 	1    4050 2600
@@
 F 0 "C6" V 5600 3950 50  0000 L CNN
 F 1 "1u" V 5600 3750 50  0000 L CNN
-F 2 "Capacitor_SMD:C_0805_2012Metric_Pad1.15x1.40mm_HandSolder" H 5688 3750 50  0001 C CNN
+F 2 "Capacitor_SMD:C_1206_3216Metric_Pad1.42x1.75mm_HandSolder" H 5688 3750 50  0001 C CNN
 F 3 "~" H 5650 3900 50  0001 C CNN
 	1    5650 3900
@@
 F 0 "C5" H 4115 5396 50  0000 L CNN
 F 1 "100u" H 4115 5305 50  0000 L CNN
-F 2 "Capacitor_SMD:C_0805_2012Metric_Pad1.15x1.40mm_HandSolder" H 4038 5200 50  0001 C CNN
+F 2 "Capacitor_SMD:C_1206_3216Metric_Pad1.42x1.75mm_HandSolder" H 4038 5200 50  0001 C CNN
 F 3 "~" H 4000 5350 50  0001 C CNN
 	1    4000 5350
@@
 F 0 "FB2" V 3376 5150 50  0000 C CNN
 F 1 "Ferrite_Bead" V 3467 5150 50  0000 C CNN
-F 2 "Inductor_SMD:L_0805_2012Metric_Pad1.15x1.40mm_HandSolder" V 3580 5150 50  0001 C CNN
+F 2 "footprints:FerriteBead_74279215" V 3580 5150 50  0001 C CNN
 F 3 "~" H 3650 5150 50  0001 C CNN
 	1    3650 5150

Commit message: Added potentiometers to EFM32. Haven't updated the physical layout for it.
Parts:
- added RV? (x2): R_POT, symbol Device:R_POT
Connections:
- wire segments 106 -> 118
- no-connect marks 8 -> 9
Other:
- note removed: "TODO: potensiometer"
Changed lines of the file:
@@
 L power:GND #PWR?
 U 1 1 5D8A3015
-P 5400 4850
+P 5450 4850
 AR Path="/5D8A3015" Ref="#PWR?"  Part="1"
 AR Path="/5D8502F2/5D8A3015" Ref="#PWR039"  Part="1"
-F 0 "#PWR039" H 5400 4600 50  0001 C CNN
-F 1 "GND" H 5405 4677 50  0000 C CNN
-F 2 "" H 5400 4850 50  0001 C CNN
-F 3 "" H 5400 4850 50  0001 C CNN
-	1    5400 4850
+F 0 "#PWR039" H 5450 4600 50  0001 C CNN
+F 1 "GND" H 5455 4677 50  0000 C CNN
+F 2 "" H 5450 4850 50  0001 C CNN
+F 3 "" H 5450 4850 50  0001 C CNN
+	1    5450 4850
 	1    0    0    -1
 $EndComp
@@
 Connection ~ 5400 4100
 Connection ~ 5400 4200
-Wire Wire Line
-	5400 4600 5400 4700
-Wire Wire Line
-	5400 4700 5400 4800
-Connection ~ 5400 4700
 $Comp
 L Synth:EFM32GG11B4xx U7
@@
 	4    4700 4350
 	1    0    0    -1
-$EndComp
-$Comp
-L power:GND #PWR?
-U 1 1 5D9DF256
-P 7150 2500
-AR Path="/5D9DF256" Ref="#PWR?"  Part="1"
-AR Path="/5D8502F2/5D9DF256" Ref="#PWR025"  Part="1"
-F 0 "#PWR025" H 7150 2250 50  0001 C CNN
-F 1 "GND" V 7155 2372 50  0000 R CNN
-F 2 "" H 7150 2500 50  0001 C CNN
-F 3 "" H 7150 2500 50  0001 C CNN
-	1    7150 2500
-	0    -1   1    0
 $EndComp
 Text HLabel 7100 1800 2    50   Input ~ 0
@@
 Wire Wire Line
 	7200 2300 6950 2300
-Text Notes 7100 2200 0    50   ~ 0
-TODO: potensiometer
-Wire Wire Line
-	7150 2500 6950 2500
 $Comp
 L power:+3.3V #PWR?
@@
 L power:+3.3V #PWR?
 U 1 1 5D972A16
-P 6750 6600
+P 6700 6600
 AR Path="/5D972A16" Ref="#PWR?"  Part="1"
 AR Path="/5D8502F2/5D972A16" Ref="#PWR0133"  Part="1"
-F 0 "#PWR0133" H 6750 6450 50  0001 C CNN
-F 1 "+3.3V" V 6765 6728 50  0000 L CNN
-F 2 "" H 6750 6600 50  0001 C CNN
-F 3 "" H 6750 6600 50  0001 C CNN
-	1    6750 6600
+F 0 "#PWR0133" H 6700 6450 50  0001 C CNN
+F 1 "+3.3V" V 6715 6728 50  0000 L CNN
+F 2 "" H 6700 6600 50  0001 C CNN
+F 3 "" H 6700 6600 50  0001 C CNN
+	1    6700 6600
 	0    -1   -1   0
 $EndComp
@@
 Wire Wire Line
 	2300 3900 4100 3900
-Wire Wire Line
-	5400 4850 5400 4800
-Connection ~ 5400 4800
 Entry Wire Line
 	10100 6050 10200 6150
@@
 Text Notes 5000 3650 0    50   ~ 0
 why the PWR_FLAG?
+Wire Wire Line
+	6700 6600 6750 6600
+$Comp
+L power:+3.3V #PWR?
+U 1 1 5D9CE084
+P 8500 2150
+F 0 "#PWR?" H 8500 2000 50  0001 C CNN
+F 1 "+3.3V" V 8515 2278 50  0000 L CNN
+F 2 "" H 8500 2150 50  0001 C CNN
+F 3 "" H 8500 2150 50  0001 C CNN
+	1    8500 2150
+	0    1    1    0
+$EndComp
+Wire Wire Line
+	8500 2150 8250 2150
+$Comp
+L Device:R_POT RV?
+U 1 1 5D9D9119
+P 8250 2450
+F 0 "RV?" H 8180 2404 50  0000 R CNN
+F 1 "R_POT" H 8180 2495 50  0000 R CNN
+F 2 "" H 8250 2450 50  0001 C CNN
+F 3 "~" H 8250 2450 50  0001 C CNN
+	1    8250 2450
+	-1   0    0    1
+$EndComp
+Wire Wire Line
+	8250 2300 8250 2150
+Connection ~ 8250 2150
+Wire Wire Line
+	8100 2450 7850 2450
+Wire Wire Line
+	7850 2450 7850 2200
+Wire Wire Line
+	7850 2200 6950 2200
+Wire Wire Line
+	8250 2150 8250 2000
+$Comp
+L Device:R_POT RV?
+U 1 1 5D9AAA27
+P 8250 1850
+F 0 "RV?" H 8180 1804 50  0000 R CNN
+F 1 "R_POT" H 8180 1895 50  0000 R CNN
+F 2 "" H 8250 1850 50  0001 C CNN
+F 3 "~" H 8250 1850 50  0001 C CNN
+	1    8250 1850
+	-1   0    0    1
+$EndComp
+Wire Wire Line
+	6950 2100 7850 2100
+Wire Wire Line
+	7850 2100 7850 1850
+Wire Wire Line
+	7850 1850 8100 1850
+NoConn ~ 6950 2500
+Wire Wire Line
+	5400 4800 5450 4800
+Wire Wire Line
+	5450 4800 5450 4850
+Wire Wire Line
+	5450 4800 5450 4700
+Wire Wire Line
+	5450 4700 5400 4700
+Connection ~ 5450 4800
+Wire Wire Line
+	5450 4700 5450 4600
+Wire Wire Line
+	5450 4600 5400 4600
+Connection ~ 5450 4700
 $EndSCHEMATC

Commit message: I forgot to annotate things again
Parts:
- gave numbers to parts that had none: 2
Connections:
- no-connect marks 9 -> 11
Changed lines of the file:
@@
 	6700 6600 6750 6600
 $Comp
-L power:+3.3V #PWR?
+L power:+3.3V #PWR024
 U 1 1 5D9CE084
 P 8500 2150
-F 0 "#PWR?" H 8500 2000 50  0001 C CNN
+F 0 "#PWR024" H 8500 2000 50  0001 C CNN
 F 1 "+3.3V" V 8515 2278 50  0000 L CNN
 F 2 "" H 8500 2150 50  0001 C CNN
@@
 	8500 2150 8250 2150
 $Comp
-L Device:R_POT RV?
+L Device:R_POT RV2
 U 1 1 5D9D9119
 P 8250 2450
-F 0 "RV?" H 8180 2404 50  0000 R CNN
+F 0 "RV2" H 8180 2404 50  0000 R CNN
 F 1 "R_POT" H 8180 2495 50  0000 R CNN
 F 2 "" H 8250 2450 50  0001 C CNN
@@
 	8250 2150 8250 2000
 $Comp
-L Device:R_POT RV?
+L Device:R_POT RV1
 U 1 1 5D9AAA27
 P 8250 1850
-F 0 "RV?" H 8180 1804 50  0000 R CNN
+F 0 "RV1" H 8180 1804 50  0000 R CNN
 F 1 "R_POT" H 8180 1895 50  0000 R CNN
 F 2 "" H 8250 1850 50  0001 C CNN
@@
 	5450 4600 5400 4600
 Connection ~ 5450 4700
+NoConn ~ 8250 2600
+NoConn ~ 8250 1700
 $EndSCHEMATC
