File: Artix.sch (KiCad schematic (older format))
At the start: 14 parts, among them J1 FPGA_debug, U2 S25FL127S, U3 XC7A100T-FTG256, U4 Oscillator

Commit message: Connect FPGA done and program_b pin to some pins on the MCU
Parts:
- renumbered C10 to C?, C11 to C?, J1 to J?, R8 to R?, R3 to R?, R1 to R?, R4 to R?, R5 to R?, R2 to R?, R6 to R?, R7 to R?, U3 to U?, U2 to U?, U4 to U?
Changed lines of the file:
@@
 EESchema Schematic File Version 4
+LIBS:Synthesizer-cache
 EELAYER 30 0
 EELAYER END
@@
 $EndDescr
 $Comp
-L FPGA_Xilinx_Artix7:XC7A100T-FTG256 U3
+L FPGA_Xilinx_Artix7:XC7A100T-FTG256 U?
 U 2 1 5D8696A8
 P 18000 5400
-F 0 "U3" H 18000 2425 50  0000 C CNN
+F 0 "U?" H 18000 2425 50  0000 C CNN
 F 1 "XC7A100T-FTG256" H 18000 2334 50  0000 C CNN
 F 2 "Package_BGA:Xilinx_FTG256" H 18000 5400 50  0001 C CNN
@@
 $EndComp
 $Comp
-L FPGA_Xilinx_Artix7:XC7A100T-FTG256 U3
+L FPGA_Xilinx_Artix7:XC7A100T-FTG256 U?
 U 3 1 5D86EF6E
 P 4900 6600
-F 0 "U3" H 3620 6653 50  0000 R CNN
+F 0 "U?" H 3620 6653 50  0000 R CNN
 F 1 "XC7A100T-FTG256" H 3620 6562 50  0000 R CNN
 F 2 "Package_BGA:Xilinx_FTG256" H 4900 6600 50  0001 C CNN
@@
 $EndComp
 $Comp
-L FPGA_Xilinx_Artix7:XC7A100T-FTG256 U3
+L FPGA_Xilinx_Artix7:XC7A100T-FTG256 U?
 U 4 1 5D871AA2
 P 2950 12150
-F 0 "U3" H 2950 13717 50  0000 C CNN
+F 0 "U?" H 2950 13717 50  0000 C CNN
 F 1 "XC7A100T-FTG256" H 2950 13626 50  0000 C CNN
 F 2 "Package_BGA:Xilinx_FTG256" H 2950 12150 50  0001 C CNN
@@
 	3250 3700 3250 3400
 $Comp
-L Device:R R1
+L Device:R R?
 U 1 1 5D8D19E7
 P 1400 2750
-F 0 "R1" H 1470 2796 50  0000 L CNN
+F 0 "R?" H 1470 2796 50  0000 L CNN
 F 1 "2.4k" H 1470 2705 50  0000 L CNN
 F 2 "Resistor_SMD:R_0805_2012Metric_Pad1.15x1.40mm_HandSolder" V 1330 2750 50  0001 C CNN
@@
 	1400 3400 1400 3150
 $Comp
-L Device:R R3
+L Device:R R?
 U 1 1 5D8D15D8
 P 1750 2750
-F 0 "R3" H 1820 2796 50  0000 L CNN
+F 0 "R?" H 1820 2796 50  0000 L CNN
 F 1 "4.7k" H 1820 2705 50  0000 L CNN
 F 2 "Resistor_SMD:R_0805_2012Metric_Pad1.15x1.40mm_HandSolder" V 1680 2750 50  0001 C CNN
@@
 Connection ~ 2750 2400
 $Comp
-L Device:R R8
+L Device:R R?
 U 1 1 5D8D0364
 P 3100 2800
-F 0 "R8" H 3170 2846 50  0000 L CNN
+F 0 "R?" H 3170 2846 50  0000 L CNN
 F 1 "4.7k" H 3170 2755 50  0000 L CNN
 F 2 "Resistor_SMD:R_0805_2012Metric_Pad1.15x1.40mm_HandSolder" V 3030 2800 50  0001 C CNN
@@
 	1300 3500 1300 3050
 $Comp
-L power:GND #PWR023
+L power:GND #PWR?
 U 1 1 5D95B8C6
 P 6800 3850
-F 0 "#PWR023" H 6800 3600 50  0001 C CNN
+F 0 "#PWR?" H 6800 3600 50  0001 C CNN
 F 1 "GND" H 6805 3677 50  0000 C CNN
 F 2 "" H 6800 3850 50  0001 C CNN
@@
 	1600 3400 1400 3400
 $Comp
-L Synth:S25FL127S U2
+L Synth:S25FL127S U?
 U 1 1 5D8B8019
 P 1950 3500
-F 0 "U2" H 2175 3865 50  0000 C CNN
+F 0 "U?" H 2175 3865 50  0000 C CNN
 F 1 "S25FL127S" H 2175 3774 50  0000 C CNN
 F 2 "Package_SO:SOIC-8-1EP_3.9x4.9mm_P1.27mm_EP2.41x3.81mm" H 1950 3500 50  0001 C CNN
@@
 Connection ~ 1000 3850
 $Comp
-L power:GND #PWR013
+L power:GND #PWR?
 U 1 1 5D8B9BD9
 P 1000 3850
-F 0 "#PWR013" H 1000 3600 50  0001 C CNN
+F 0 "#PWR?" H 1000 3600 50  0001 C CNN
 F 1 "GND" H 1005 3677 50  0000 C CNN
 F 2 "" H 1000 3850 50  0001 C CNN
@@
 $EndComp
 $Comp
-L Device:C C10
+L Device:C C?
 U 1 1 5D8D3873
 P 1000 2800
-F 0 "C10" H 1115 2846 50  0000 L CNN
+F 0 "C?" H 1115 2846 50  0000 L CNN
 F 1 "100n" H 1115 2755 50  0000 L CNN
 F 2 "Capacitor_SMD:C_0805_2012Metric_Pad1.15x1.40mm_HandSolder" H 1038 2650 50  0001 C CNN
@@
 	2850 3600 2850 6300
 $Comp
-L Device:R R4
+L Device:R R?
 U 1 1 5DB16E52
 P 1750 4850
-F 0 "R4" H 1820 4896 50  0000 L CNN
+F 0 "R?" H 1820 4896 50  0000 L CNN
 F 1 "10k" H 1820 4805 50  0000 L CNN
 F 2 "Resistor_SMD:R_0805_2012Metric_Pad1.15x1.40mm_HandSolder" V 1680 4850 50  0001 C CNN
@@
 $EndComp
 $Comp
-L Device:R R5
+L Device:R R?
 U 1 1 5DB1753D
 P 2000 4850
-F 0 "R5" H 2070 4896 50  0000 L CNN
+F 0 "R?" H 2070 4896 50  0000 L CNN
 F 1 "4.7k" H 2070 4805 50  0000 L CNN
 F 2 "Resistor_SMD:R_0805_2012Metric_Pad1.15x1.40mm_HandSolder" V 1930 4850 50  0001 C CNN
@@
 $EndComp
 $Comp
-L Device:R R2
+L Device:R R?
 U 1 1 5DB17AAB
 P 1500 4850
-F 0 "R2" H 1570 4896 50  0000 L CNN
+F 0 "R?" H 1570 4896 50  0000 L CNN
 F 1 "10k" H 1570 4805 50  0000 L CNN
 F 2 "Resistor_SMD:R_0805_2012Metric_Pad1.15x1.40mm_HandSolder" V 1430 4850 50  0001 C CNN
@@
 $EndComp
 $Comp
-L Device:R R6
+L Device:R R?
 U 1 1 5DB18145
 P 2250 4850
-F 0 "R6" H 2320 4896 50  0000 L CNN
+F 0 "R?" H 2320 4896 50  0000 L CNN
 F 1 "4.7k" H 2320 4805 50  0000 L CNN
 F 2 "Resistor_SMD:R_0805_2012Metric_Pad1.15x1.40mm_HandSolder" V 2180 4850 50  0001 C CNN
@@
 $EndComp
 $Comp
-L Device:R R7
+L Device:R R?
 U 1 1 5DB18715
 P 2450 4850
-F 0 "R7" H 2520 4896 50  0000 L CNN
+F 0 "R?" H 2520 4896 50  0000 L CNN
 F 1 "330" H 2520 4805 50  0000 L CNN
 F 2 "Resistor_SMD:R_0805_2012Metric_Pad1.15x1.40mm_HandSolder" V 2380 4850 50  0001 C CNN
@@
 $EndComp
 $Comp
-L Synth:FPGA_debug J1
+L Synth:FPGA_debug J?
 U 1 1 5DB1FB59
 P 1100 5900
-F 0 "J1" H 1100 6425 50  0000 C CNN
+F 0 "J?" H 1100 6425 50  0000 C CNN
 F 1 "FPGA_debug" H 1100 6334 50  0000 C CNN
 F 2 "Connector_PinHeader_2.00mm:PinHeader_2x07_P2.00mm_Vertical" H 1100 6300 50  0001 C CNN
@@
 $EndComp
 $Comp
-L power:GND #PWR012
+L power:GND #PWR?
 U 1 1 5DB20A30
 P 850 6450
-F 0 "#PWR012" H 850 6200 50  0001 C CNN
+F 0 "#PWR?" H 850 6200 50  0001 C CNN
 F 1 "GND" H 855 6277 50  0000 C CNN
 F 2 "" H 850 6450 50  0001 C CNN
@@
 	2500 5000 2450 5000
 $Comp
-L power:GND #PWR020
+L power:GND #PWR?
 U 1 1 5DB930FB
 P 3200 8400
-F 0 "#PWR020" H 3200 8150 50  0001 C CNN
+F 0 "#PWR?" H 3200 8150 50  0001 C CNN
 F 1 "GND" H 3205 8227 50  0000 C CNN
 F 2 "" H 3200 8400 50  0001 C CNN
@@
 	8200 5800 6900 5800
 $Comp
-L Synth:Oscillator U4
+L Synth:Oscillator U?
 U 1 1 5DBDB09B
 P 6650 5750
-F 0 "U4" H 6683 6125 50  0000 C CNN
+F 0 "U?" H 6683 6125 50  0000 C CNN
 F 1 "Oscillator" H 6683 6034 50  0000 C CNN
 F 2 "Oscillator:Oscillator_SMD_Abracon_ASCO-4Pin_1.6x1.2mm" H 6700 5700 50  0001 C CNN
@@
 $EndComp
 $Comp
-L power:GND #PWR025
+L power:GND #PWR?
 U 1 1 5DC0D0A3
 P 7300 6000
-F 0 "#PWR025" H 7300 5750 50  0001 C CNN
+F 0 "#PWR?" H 7300 5750 50  0001 C CNN
 F 1 "GND" H 7305 5827 50  0000 C CNN
 F 2 "" H 7300 6000 50  0001 C CNN
@@
 	7100 5900 7100 5600
 $Comp
-L Device:C C11
+L Device:C C?
 U 1 1 5DC18FF3
 P 7400 5450
-F 0 "C11" H 7515 5496 50  0000 L CNN
+F 0 "C?" H 7515 5496 50  0000 L CNN
 F 1 "100n" H 7515 5405 50  0000 L CNN
 F 2 "Capacitor_SMD:C_0805_2012Metric_Pad1.15x1.40mm_HandSolder" H 7438 5300 50  0001 C CNN
@@
 Connection ~ 1950 11650
 $Comp
-L power:GND #PWR019
+L power:GND #PWR?
 U 1 1 5DC8F87F
 P 2950 13650
-F 0 "#PWR019" H 2950 13400 50  0001 C CNN
+F 0 "#PWR?" H 2950 13400 50  0001 C CNN
 F 1 "GND" H 2955 13477 50  0000 C CNN
 F 2 "" H 2950 13650 50  0001 C CNN
@@
 	1850 11550 1850 13650
 $Comp
-L power:GND #PWR027
+L power:GND #PWR?
 U 1 1 5DD18602
 P 18050 2500
-F 0 "#PWR027" H 18050 2250 50  0001 C CNN
+F 0 "#PWR?" H 18050 2250 50  0001 C CNN
 F 1 "GND" H 18055 2327 50  0000 C CNN
 F 2 "" H 18050 2500 50  0001 C CNN
@@
 	3800 4900 3800 5000
 $Comp
-L power:GND #PWR026
+L power:GND #PWR?
 U 1 1 5D8EC9FF
 P 10200 2500
-F 0 "#PWR026" H 10200 2250 50  0001 C CNN
+F 0 "#PWR?" H 10200 2250 50  0001 C CNN
 F 1 "GND" H 10205 2327 50  0000 C CNN
 F 2 "" H 10200 2500 50  0001 C CNN
@@
 	1200 11550 1200 11650
 $Comp
-L power:+1V8 #PWR0102
+L power:+1V8 #PWR?
 U 1 1 5E1CD4BD
 P 1800 10850
-F 0 "#PWR0102" H 1800 10700 50  0001 C CNN
+F 0 "#PWR?" H 1800 10700 50  0001 C CNN
 F 1 "+1V8" H 1815 11023 50  0000 C CNN
 F 2 "" H 1800 10850 50  0001 C CNN
@@
 $EndComp
 $Comp
-L power:+1V0 #PWR0103
+L power:+1V0 #PWR?
 U 1 1 5E1CEB46
 P 1200 11550
-F 0 "#PWR0103" H 1200 11400 50  0001 C CNN
+F 0 "#PWR?" H 1200 11400 50  0001 C CNN
 F 1 "+1V0" H 1215 11723 50  0000 C CNN
 F 2 "" H 1200 11550 50  0001 C CNN
@@
 $EndComp
 $Comp
-L power:+1V0 #PWR0104
+L power:+1V0 #PWR?
 U 1 1 5E1D1568
 P 4200 10850
-F 0 "#PWR0104" H 4200 10700 50  0001 C CNN
+F 0 "#PWR?" H 4200 10700 50  0001 C CNN
 F 1 "+1V0" V 4215 10978 50  0000 L CNN
 F 2 "" H 4200 10850 50  0001 C CNN
@@
 $EndComp
 $Comp
-L power:+3.3V #PWR0132
+L power:+3.3V #PWR?
 U 1 1 5D914A91
 P 7100 5050
-F 0 "#PWR0132" H 7100 4900 50  0001 C CNN
+F 0 "#PWR?" H 7100 4900 50  0001 C CNN
 F 1 "+3.3V" H 7115 5223 50  0000 C CNN
 F 2 "" H 7100 5050 50  0001 C CNN
@@
 $EndComp
 $Comp
-L power:+3.3V #PWR0133
+L power:+3.3V #PWR?
 U 1 1 5D9199D3
 P 3800 4900
-F 0 "#PWR0133" H 3800 4750 50  0001 C CNN
+F 0 "#PWR?" H 3800 4750 50  0001 C CNN
 F 1 "+3.3V" H 3815 5073 50  0000 C CNN
 F 2 "" H 3800 4900 50  0001 C CNN
@@
 $EndComp
 $Comp
-L power:+3.3V #PWR0134
+L power:+3.3V #PWR?
 U 1 1 5D91E70E
 P 2000 4300
-F 0 "#PWR0134" H 2000 4150 50  0001 C CNN
+F 0 "#PWR?" H 2000 4150 50  0001 C CNN
 F 1 "+3.3V" H 2015 4473 50  0000 C CNN
 F 2 "" H 2000 4300 50  0001 C CNN
@@
 $EndComp
 $Comp
-L power:+3.3V #PWR0135
+L power:+3.3V #PWR?
 U 1 1 5D920C94
 P 2750 2400
-F 0 "#PWR0135" H 2750 2250 50  0001 C CNN
+F 0 "#PWR?" H 2750 2250 50  0001 C CNN
 F 1 "+3.3V" H 2765 2573 50  0000 C CNN
 F 2 "" H 2750 2400 50  0001 C CNN
@@
 $EndComp
 $Comp
-L power:+3.3V #PWR0136
+L power:+3.3V #PWR?
 U 1 1 5D936054
 P 2700 6400
-F 0 "#PWR0136" H 2700 6250 50  0001 C CNN
+F 0 "#PWR?" H 2700 6250 50  0001 C CNN
 F 1 "+3.3V" H 2715 6573 50  0000 C CNN
 F 2 "" H 2700 6400 50  0001 C CNN
@@
 Connection ~ 8700 2500
 $Comp
-L FPGA_Xilinx_Artix7:XC7A100T-FTG256 U3
+L FPGA_Xilinx_Artix7:XC7A100T-FTG256 U?
 U 1 1 5D866531
 P 10200 5400
-F 0 "U3" H 10200 2425 50  0000 C CNN
+F 0 "U?" H 10200 2425 50  0000 C CNN
 F 1 "XC7A100T-FTG256" H 10200 2334 50  0000 C CNN
 F 2 "Package_BGA:Xilinx_FTG256" H 10200 5400 50  0001 C CNN

Commit message: Added forgotten USB-B power source, powered bank 14 of FPGA.
Parts:
- gave numbers to parts that had none: 14
Connections:
- wire segments 195 -> 199

Commit message: Re-add SPI connections inside Artix sheet Thank mr. kicad for fantastic VCS support
Connections:
- net labels added: SPI_CLK, SPI_CS, SPI_MISO, SPI_MOSI
- wire segments 199 -> 203
- no-connect marks 163 -> 159
Changed lines of the file:
@@
 NoConn ~ 8200 3900
 NoConn ~ 8200 4500
-NoConn ~ 8200 4600
-NoConn ~ 8200 4700
-NoConn ~ 8200 4800
-NoConn ~ 8200 4900
 NoConn ~ 8200 5000
 NoConn ~ 8200 5100
@@
 	11300 2500 11300 2300
 Connection ~ 11300 2500
+Text HLabel 7800 4600 0    50   Input ~ 0
+SPI_MOSI
+Text HLabel 7800 4700 0    50   Output ~ 0
+SPI_MISO
+Text HLabel 7800 4800 0    50   Input ~ 0
+SPI_CLK
+Text HLabel 7800 4900 0    50   Input ~ 0
+SPI_CS
+Wire Wire Line
+	7800 4600 8200 4600
+Wire Wire Line
+	7800 4700 8200 4700
+Wire Wire Line
+	8200 4800 7800 4800
+Wire Wire Line
+	7800 4900 8200 4900
 $EndSCHEMATC

Commit message: Added NPN transistor on USB and wired shield. Added LEDs, debug pins.
Connections:
- net labels added: GREEN_LED, MCU_extra_1, MCU_extra_2, MCU_extra_3, MCU_extra_4, RED_LED
- wire segments 203 -> 209
- no-connect marks 159 -> 153
Changed lines of the file:
@@
 NoConn ~ 8200 3900
 NoConn ~ 8200 4500
-NoConn ~ 8200 5000
-NoConn ~ 8200 5100
-NoConn ~ 8200 5200
-NoConn ~ 8200 5300
-NoConn ~ 8200 5400
-NoConn ~ 8200 5500
 NoConn ~ 8200 5600
 NoConn ~ 8200 5700
@@
 Wire Wire Line
 	7800 4900 8200 4900
+Text HLabel 7800 5000 0    50   Output ~ 0
+RED_LED
+Text HLabel 7800 5100 0    50   Output ~ 0
+GREEN_LED
+Wire Wire Line
+	7800 5100 8200 5100
+Wire Wire Line
+	8200 5000 7800 5000
+Text HLabel 7800 5200 0    50   Output ~ 0
+MCU_extra_1
+Text HLabel 7800 5300 0    50   Output ~ 0
+MCU_extra_2
+Text HLabel 7800 5400 0    50   Output ~ 0
+MCU_extra_3
+Text HLabel 7800 5500 0    50   Output ~ 0
+MCU_extra_4
+Wire Wire Line
+	7800 5500 8200 5500
+Wire Wire Line
+	8200 5400 7800 5400
+Wire Wire Line
+	7800 5300 8200 5300
+Wire Wire Line
+	8200 5200 7800 5200
 $EndSCHEMATC
