File: Artix.sch (KiCad schematic (older format))
At the start: 14 parts, among them J4 FPGA_debug, U2 S25FL127S, U3 XC7A100T-FTG256, U4 Oscillator

Commit message: Rearrange PCB components to more closely match schematics and take up less space
Connections:
- wire segments 209 -> 208
Changed lines of the file:
@@
 Connection ~ 7100 5050
-Wire Wire Line
-	7100 5050 7100 5000
 Wire Wire Line
 	7400 5700 7400 5600

Commit message: Updated component footprints. The PCB is now an unholy mess.
Parts:
- C3, C4: footprint Capacitor_SMD:C_0805_2012Metric_Pad1.15x1.40mm_HandSolder -> Capacitor_SMD:C_1206_3216Metric_Pad1.42x1.75mm_HandSolder
- R1, R2, R3, R4, R5, R6, R7, R8: footprint Resistor_SMD:R_0805_2012Metric_Pad1.15x1.40mm_HandSolder -> Resistor_SMD:R_1206_3216Metric_Pad1.42x1.75mm_HandSolder
Changed lines of the file:
@@
 F 0 "R1" H 1470 2796 50  0000 L CNN
 F 1 "2.4k" H 1470 2705 50  0000 L CNN
-F 2 "Resistor_SMD:R_0805_2012Metric_Pad1.15x1.40mm_HandSolder" V 1330 2750 50  0001 C CNN
+F 2 "Resistor_SMD:R_1206_3216Metric_Pad1.42x1.75mm_HandSolder" V 1330 2750 50  0001 C CNN
 F 3 "~" H 1400 2750 50  0001 C CNN
 	1    1400 2750
@@
 F 0 "R3" H 1820 2796 50  0000 L CNN
 F 1 "4.7k" H 1820 2705 50  0000 L CNN
-F 2 "Resistor_SMD:R_0805_2012Metric_Pad1.15x1.40mm_HandSolder" V 1680 2750 50  0001 C CNN
+F 2 "Resistor_SMD:R_1206_3216Metric_Pad1.42x1.75mm_HandSolder" V 1680 2750 50  0001 C CNN
 F 3 "~" H 1750 2750 50  0001 C CNN
 	1    1750 2750
@@
 F 0 "R8" H 3170 2846 50  0000 L CNN
 F 1 "4.7k" H 3170 2755 50  0000 L CNN
-F 2 "Resistor_SMD:R_0805_2012Metric_Pad1.15x1.40mm_HandSolder" V 3030 2800 50  0001 C CNN
+F 2 "Resistor_SMD:R_1206_3216Metric_Pad1.42x1.75mm_HandSolder" V 3030 2800 50  0001 C CNN
 F 3 "~" H 3100 2800 50  0001 C CNN
 	1    3100 2800
@@
 F 0 "C3" H 1115 2846 50  0000 L CNN
 F 1 "100n" H 1115 2755 50  0000 L CNN
-F 2 "Capacitor_SMD:C_0805_2012Metric_Pad1.15x1.40mm_HandSolder" H 1038 2650 50  0001 C CNN
+F 2 "Capacitor_SMD:C_1206_3216Metric_Pad1.42x1.75mm_HandSolder" H 1038 2650 50  0001 C CNN
 F 3 "~" H 1000 2800 50  0001 C CNN
 	1    1000 2800
@@
 F 0 "R4" H 1820 4896 50  0000 L CNN
 F 1 "10k" H 1820 4805 50  0000 L CNN
-F 2 "Resistor_SMD:R_0805_2012Metric_Pad1.15x1.40mm_HandSolder" V 1680 4850 50  0001 C CNN
+F 2 "Resistor_SMD:R_1206_3216Metric_Pad1.42x1.75mm_HandSolder" V 1680 4850 50  0001 C CNN
 F 3 "~" H 1750 4850 50  0001 C CNN
 	1    1750 4850
@@
 F 0 "R5" H 2070 4896 50  0000 L CNN
 F 1 "4.7k" H 2070 4805 50  0000 L CNN
-F 2 "Resistor_SMD:R_0805_2012Metric_Pad1.15x1.40mm_HandSolder" V 1930 4850 50  0001 C CNN
+F 2 "Resistor_SMD:R_1206_3216Metric_Pad1.42x1.75mm_HandSolder" V 1930 4850 50  0001 C CNN
 F 3 "~" H 2000 4850 50  0001 C CNN
 	1    2000 4850
@@
 F 0 "R2" H 1570 4896 50  0000 L CNN
 F 1 "10k" H 1570 4805 50  0000 L CNN
-F 2 "Resistor_SMD:R_0805_2012Metric_Pad1.15x1.40mm_HandSolder" V 1430 4850 50  0001 C CNN
+F 2 "Resistor_SMD:R_1206_3216Metric_Pad1.42x1.75mm_HandSolder" V 1430 4850 50  0001 C CNN
 F 3 "~" H 1500 4850 50  0001 C CNN
 	1    1500 4850
@@
 F 0 "R6" H 2320 4896 50  0000 L CNN
 F 1 "4.7k" H 2320 4805 50  0000 L CNN
-F 2 "Resistor_SMD:R_0805_2012Metric_Pad1.15x1.40mm_HandSolder" V 2180 4850 50  0001 C CNN
+F 2 "Resistor_SMD:R_1206_3216Metric_Pad1.42x1.75mm_HandSolder" V 2180 4850 50  0001 C CNN
 F 3 "~" H 2250 4850 50  0001 C CNN
 	1    2250 4850
@@
 F 0 "R7" H 2520 4896 50  0000 L CNN
 F 1 "330" H 2520 4805 50  0000 L CNN
-F 2 "Resistor_SMD:R_0805_2012Metric_Pad1.15x1.40mm_HandSolder" V 2380 4850 50  0001 C CNN
+F 2 "Resistor_SMD:R_1206_3216Metric_Pad1.42x1.75mm_HandSolder" V 2380 4850 50  0001 C CNN
 F 3 "~" H 2450 4850 50  0001 C CNN
 	1    2450 4850
@@
 F 0 "C4" H 7515 5496 50  0000 L CNN
 F 1 "100n" H 7515 5405 50  0000 L CNN
-F 2 "Capacitor_SMD:C_0805_2012Metric_Pad1.15x1.40mm_HandSolder" H 7438 5300 50  0001 C CNN
+F 2 "Capacitor_SMD:C_1206_3216Metric_Pad1.42x1.75mm_HandSolder" H 7438 5300 50  0001 C CNN
 F 3 "~" H 7400 5450 50  0001 C CNN
 	1    7400 5450

Commit message: Tag you're it. Wired up the DAC, fixed the PSU footprint.
Parts:
- renumbered C3 to C?, C4 to C?, R8 to R?, R3 to R?, R1 to R?, R4 to R?, R5 to R?, R2 to R?, R6 to R?, R7 to R?, U3 to U?, U2 to U?, U4 to U?
Changed lines of the file:
@@
 $EndDescr
 $Comp
-L FPGA_Xilinx_Artix7:XC7A100T-FTG256 U3
+L FPGA_Xilinx_Artix7:XC7A100T-FTG256 U?
 U 2 1 5D8696A8
 P 18000 5400
-F 0 "U3" H 18000 2425 50  0000 C CNN
+F 0 "U?" H 18000 2425 50  0000 C CNN
 F 1 "XC7A100T-FTG256" H 18000 2334 50  0000 C CNN
 F 2 "Package_BGA:Xilinx_FTG256" H 18000 5400 50  0001 C CNN
@@
 $EndComp
 $Comp
-L FPGA_Xilinx_Artix7:XC7A100T-FTG256 U3
+L FPGA_Xilinx_Artix7:XC7A100T-FTG256 U?
 U 3 1 5D86EF6E
 P 4900 6600
-F 0 "U3" H 3620 6653 50  0000 R CNN
+F 0 "U?" H 3620 6653 50  0000 R CNN
 F 1 "XC7A100T-FTG256" H 3620 6562 50  0000 R CNN
 F 2 "Package_BGA:Xilinx_FTG256" H 4900 6600 50  0001 C CNN
@@
 $EndComp
 $Comp
-L FPGA_Xilinx_Artix7:XC7A100T-FTG256 U3
+L FPGA_Xilinx_Artix7:XC7A100T-FTG256 U?
 U 4 1 5D871AA2
 P 2950 12150
-F 0 "U3" H 2950 13717 50  0000 C CNN
+F 0 "U?" H 2950 13717 50  0000 C CNN
 F 1 "XC7A100T-FTG256" H 2950 13626 50  0000 C CNN
 F 2 "Package_BGA:Xilinx_FTG256" H 2950 12150 50  0001 C CNN
@@
 	3250 3700 3250 3400
 $Comp
-L Device:R R1
+L Device:R R?
 U 1 1 5D8D19E7
 P 1400 2750
-F 0 "R1" H 1470 2796 50  0000 L CNN
+F 0 "R?" H 1470 2796 50  0000 L CNN
 F 1 "2.4k" H 1470 2705 50  0000 L CNN
 F 2 "Resistor_SMD:R_1206_3216Metric_Pad1.42x1.75mm_HandSolder" V 1330 2750 50  0001 C CNN
@@
 	1400 3400 1400 3150
 $Comp
-L Device:R R3
+L Device:R R?
 U 1 1 5D8D15D8
 P 1750 2750
-F 0 "R3" H 1820 2796 50  0000 L CNN
+F 0 "R?" H 1820 2796 50  0000 L CNN
 F 1 "4.7k" H 1820 2705 50  0000 L CNN
 F 2 "Resistor_SMD:R_1206_3216Metric_Pad1.42x1.75mm_HandSolder" V 1680 2750 50  0001 C CNN
@@
 Connection ~ 2750 2400
 $Comp
-L Device:R R8
+L Device:R R?
 U 1 1 5D8D0364
 P 3100 2800
-F 0 "R8" H 3170 2846 50  0000 L CNN
+F 0 "R?" H 3170 2846 50  0000 L CNN
 F 1 "4.7k" H 3170 2755 50  0000 L CNN
 F 2 "Resistor_SMD:R_1206_3216Metric_Pad1.42x1.75mm_HandSolder" V 3030 2800 50  0001 C CNN
@@
 	1300 3500 1300 3050
 $Comp
-L power:GND #PWR018
+L power:GND #PWR?
 U 1 1 5D95B8C6
 P 6800 3850
-F 0 "#PWR018" H 6800 3600 50  0001 C CNN
+F 0 "#PWR?" H 6800 3600 50  0001 C CNN
 F 1 "GND" H 6805 3677 50  0000 C CNN
 F 2 "" H 6800 3850 50  0001 C CNN
@@
 	1600 3400 1400 3400
 $Comp
-L Synth:S25FL127S U2
+L Synth:S25FL127S U?
 U 1 1 5D8B8019
 P 1950 3500
-F 0 "U2" H 2175 3865 50  0000 C CNN
+F 0 "U?" H 2175 3865 50  0000 C CNN
 F 1 "S25FL127S" H 2175 3774 50  0000 C CNN
 F 2 "Package_SO:SOIC-8-1EP_3.9x4.9mm_P1.27mm_EP2.41x3.81mm" H 1950 3500 50  0001 C CNN
@@
 Connection ~ 1000 3850
 $Comp
-L power:GND #PWR07
+L power:GND #PWR?
 U 1 1 5D8B9BD9
 P 1000 3850
-F 0 "#PWR07" H 1000 3600 50  0001 C CNN
+F 0 "#PWR?" H 1000 3600 50  0001 C CNN
 F 1 "GND" H 1005 3677 50  0000 C CNN
 F 2 "" H 1000 3850 50  0001 C CNN
@@
 $EndComp
 $Comp
-L Device:C C3
+L Device:C C?
 U 1 1 5D8D3873
 P 1000 2800
-F 0 "C3" H 1115 2846 50  0000 L CNN
+F 0 "C?" H 1115 2846 50  0000 L CNN
 F 1 "100n" H 1115 2755 50  0000 L CNN
 F 2 "Capacitor_SMD:C_1206_3216Metric_Pad1.42x1.75mm_HandSolder" H 1038 2650 50  0001 C CNN
@@
 	2850 3600 2850 6300
 $Comp
-L Device:R R4
+L Device:R R?
 U 1 1 5DB16E52
 P 1750 4850
-F 0 "R4" H 1820 4896 50  0000 L CNN
+F 0 "R?" H 1820 4896 50  0000 L CNN
 F 1 "10k" H 1820 4805 50  0000 L CNN
 F 2 "Resistor_SMD:R_1206_3216Metric_Pad1.42x1.75mm_HandSolder" V 1680 4850 50  0001 C CNN
@@
 $EndComp
 $Comp
-L Device:R R5
+L Device:R R?
 U 1 1 5DB1753D
 P 2000 4850
-F 0 "R5" H 2070 4896 50  0000 L CNN
+F 0 "R?" H 2070 4896 50  0000 L CNN
 F 1 "4.7k" H 2070 4805 50  0000 L CNN
 F 2 "Resistor_SMD:R_1206_3216Metric_Pad1.42x1.75mm_HandSolder" V 1930 4850 50  0001 C CNN
@@
 $EndComp
 $Comp
-L Device:R R2
+L Device:R R?
 U 1 1 5DB17AAB
 P 1500 4850
-F 0 "R2" H 1570 4896 50  0000 L CNN
+F 0 "R?" H 1570 4896 50  0000 L CNN
 F 1 "10k" H 1570 4805 50  0000 L CNN
 F 2 "Resistor_SMD:R_1206_3216Metric_Pad1.42x1.75mm_HandSolder" V 1430 4850 50  0001 C CNN
@@
 $EndComp
 $Comp
-L Device:R R6
+L Device:R R?
 U 1 1 5DB18145
 P 2250 4850
-F 0 "R6" H 2320 4896 50  0000 L CNN
+F 0 "R?" H 2320 4896 50  0000 L CNN
 F 1 "4.7k" H 2320 4805 50  0000 L CNN
 F 2 "Resistor_SMD:R_1206_3216Metric_Pad1.42x1.75mm_HandSolder" V 2180 4850 50  0001 C CNN
@@
 $EndComp
 $Comp
-L Device:R R7
+L Device:R R?
 U 1 1 5DB18715
 P 2450 4850
-F 0 "R7" H 2520 4896 50  0000 L CNN
+F 0 "R?" H 2520 4896 50  0000 L CNN
 F 1 "330" H 2520 4805 50  0000 L CNN
 F 2 "Resistor_SMD:R_1206_3216Metric_Pad1.42x1.75mm_HandSolder" V 2380 4850 50  0001 C CNN
@@
 $EndComp
 $Comp
-L Synth:FPGA_debug J4
+L Synth:FPGA_debug J?
 U 1 1 5DB1FB59
 P 1100 5900
-AR Path="/5DB1FB59" Ref="J4"  Part="1"
+AR Path="/5DB1FB59" Ref="J?"  Part="1"
 AR Path="/5D81B1F5/5DB1FB59" Ref="J4"  Part="1"
-F 0 "J4" H 1100 6425 50  0000 C CNN
+F 0 "J?" H 1100 6425 50  0000 C CNN
 F 1 "FPGA_debug" H 1100 6334 50  0000 C CNN
 F 2 "Connector_PinHeader_2.00mm:PinHeader_2x07_P2.00mm_Vertical" H 1100 6300 50  0001 C CNN
@@
 $EndComp
 $Comp
-L power:GND #PWR06
+L power:GND #PWR?
 U 1 1 5DB20A30
 P 850 6450
-F 0 "#PWR06" H 850 6200 50  0001 C CNN
+F 0 "#PWR?" H 850 6200 50  0001 C CNN
 F 1 "GND" H 855 6277 50  0000 C CNN
 F 2 "" H 850 6450 50  0001 C CNN
@@
 	3400 6800 2450 6800
 $Comp
-L power:GND #PWR015
+L power:GND #PWR?
 U 1 1 5DB930FB
 P 3200 8400
-F 0 "#PWR015" H 3200 8150 50  0001 C CNN
+F 0 "#PWR?" H 3200 8150 50  0001 C CNN
 F 1 "GND" H 3205 8227 50  0000 C CNN
 F 2 "" H 3200 8400 50  0001 C CNN
@@
 	9200 5800 6900 5800
 $Comp
-L Synth:Oscillator U4
+L Synth:Oscillator U?
 U 1 1 5DBDB09B
 P 6650 5750
-F 0 "U4" H 6683 6125 50  0000 C CNN
+F 0 "U?" H 6683 6125 50  0000 C CNN
 F 1 "Oscillator" H 6683 6034 50  0000 C CNN
 F 2 "Oscillator:Oscillator_SMD_Abracon_ASCO-4Pin_1.6x1.2mm" H 6700 5700 50  0001 C CNN
@@
 $EndComp
 $Comp
-L power:GND #PWR020
+L power:GND #PWR?
 U 1 1 5DC0D0A3
 P 7300 6000
-F 0 "#PWR020" H 7300 5750 50  0001 C CNN
+F 0 "#PWR?" H 7300 5750 50  0001 C CNN
 F 1 "GND" H 7305 5827 50  0000 C CNN
 F 2 "" H 7300 6000 50  0001 C CNN
@@
 	7100 5900 7100 5600
 $Comp
-L Device:C C4
+L Device:C C?
 U 1 1 5DC18FF3
 P 7400 5450
-F 0 "C4" H 7515 5496 50  0000 L CNN
+F 0 "C?" H 7515 5496 50  0000 L CNN
 F 1 "100n" H 7515 5405 50  0000 L CNN
 F 2 "Capacitor_SMD:C_1206_3216Metric_Pad1.42x1.75mm_HandSolder" H 7438 5300 50  0001 C CNN
@@
 Connection ~ 1950 11650
 $Comp
-L power:GND #PWR014
+L power:GND #PWR?
 U 1 1 5DC8F87F
 P 2950 13650
-F 0 "#PWR014" H 2950 13400 50  0001 C CNN
+F 0 "#PWR?" H 2950 13400 50  0001 C CNN
 F 1 "GND" H 2955 13477 50  0000 C CNN
 F 2 "" H 2950 13650 50  0001 C CNN
@@
 	1850 11550 1850 13650
 $Comp
-L power:GND #PWR022
+L power:GND #PWR?
 U 1 1 5DD18602
 P 18050 2500
-F 0 "#PWR022" H 18050 2250 50  0001 C CNN
+F 0 "#PWR?" H 18050 2250 50  0001 C CNN
 F 1 "GND" H 18055 2327 50  0000 C CNN
 F 2 "" H 18050 2500 50  0001 C CNN
@@
 	3800 4900 3800 5000
 $Comp
-L power:GND #PWR021
+L power:GND #PWR?
 U 1 1 5D8EC9FF
 P 12300 2350
-F 0 "#PWR021" H 12300 2100 50  0001 C CNN
+F 0 "#PWR?" H 12300 2100 50  0001 C CNN
 F 1 "GND" H 12305 2177 50  0000 C CNN
 F 2 "" H 12300 2350 50  0001 C CNN
@@
 	1200 11550 1200 11650
 $Comp
-L power:+1V8 #PWR010
+L power:+1V8 #PWR?
 U 1 1 5E1CD4BD
 P 1800 10850
-F 0 "#PWR010" H 1800 10700 50  0001 C CNN
+F 0 "#PWR?" H 1800 10700 50  0001 C CNN
 F 1 "+1V8" H 1815 11023 50  0000 C CNN
 F 2 "" H 1800 10850 50  0001 C CNN
@@
 $EndComp
 $Comp
-L power:+1V0 #PWR08
+L power:+1V0 #PWR?
 U 1 1 5E1CEB46
 P 1200 11550
-F 0 "#PWR08" H 1200 11400 50  0001 C CNN
+F 0 "#PWR?" H 1200 11400 50  0001 C CNN
 F 1 "+1V0" H 1215 11723 50  0000 C CNN
 F 2 "" H 1200 11550 50  0001 C CNN
@@
 $EndComp
 $Comp
-L power:+1V0 #PWR017
+L power:+1V0 #PWR?
 U 1 1 5E1D1568
 P 4200 10850
-F 0 "#PWR017" H 4200 10700 50  0001 C CNN
+F 0 "#PWR?" H 4200 10700 50  0001 C CNN
 F 1 "+1V0" V 4215 10978 50  0000 L CNN
 F 2 "" H 4200 10850 50  0001 C CNN
@@
 $EndComp
 $Comp
-L power:+3.3V #PWR019
+L power:+3.3V #PWR?
 U 1 1 5D914A91
 P 7100 5050
-F 0 "#PWR019" H 7100 4900 50  0001 C CNN
+F 0 "#PWR?" H 7100 4900 50  0001 C CNN
 F 1 "+3.3V" H 7115 5223 50  0000 C CNN
 F 2 "" H 7100 5050 50  0001 C CNN
@@
 $EndComp
 $Comp
-L power:+3.3V #PWR016
+L power:+3.3V #PWR?
 U 1 1 5D9199D3
 P 3800 4900
-F 0 "#PWR016" H 3800 4750 50  0001 C CNN
+F 0 "#PWR?" H 3800 4750 50  0001 C CNN
 F 1 "+3.3V" H 3815 5073 50  0000 C CNN
 F 2 "" H 3800 4900 50  0001 C CNN
@@
 $EndComp
 $Comp
-L power:+3.3V #PWR011
+L power:+3.3V #PWR?
 U 1 1 5D91E70E
 P 2000 4300
-F 0 "#PWR011" H 2000 4150 50  0001 C CNN
+F 0 "#PWR?" H 2000 4150 50  0001 C CNN
 F 1 "+3.3V" H 2015 4473 50  0000 C CNN
 F 2 "" H 2000 4300 50  0001 C CNN
@@
 $EndComp
 $Comp
-L power:+3.3V #PWR013
+L power:+3.3V #PWR?
 U 1 1 5D920C94
 P 2750 2400
-F 0 "#PWR013" H 2750 2250 50  0001 C CNN
+F 0 "#PWR?" H 2750 2250 50  0001 C CNN
 F 1 "+3.3V" H 2765 2573 50  0000 C CNN
 F 2 "" H 2750 2400 50  0001 C CNN
@@
 $EndComp
 $Comp
-L power:+3.3V #PWR012
+L power:+3.3V #PWR?
 U 1 1 5D936054
 P 2700 6400
-F 0 "#PWR012" H 2700 6250 50  0001 C CNN
+F 0 "#PWR?" H 2700 6250 50  0001 C CNN
 F 1 "+3.3V" H 2715 6573 50  0000 C CNN
 F 2 "" H 2700 6400 50  0001 C CNN
@@
 	12400 2500 12300 2500
 $Comp
-L FPGA_Xilinx_Artix7:XC7A100T-FTG256 U3
+L FPGA_Xilinx_Artix7:XC7A100T-FTG256 U?
 U 1 1 5D866531
 P 11200 5400
-F 0 "U3" H 11200 2425 50  0000 C CNN
+F 0 "U?" H 11200 2425 50  0000 C CNN
 F 1 "XC7A100T-FTG256" H 11200 2334 50  0000 C CNN
 F 2 "Package_BGA:Xilinx_FTG256" H 11200 5400 50  0001 C CNN
@@
 	9600 2500 9600 2400
 $Comp
-L power:+3.3V #PWR048
+L power:+3.3V #PWR?
 U 1 1 5D9F7116
 P 10100 2300
-F 0 "#PWR048" H 10100 2150 50  0001 C CNN
+F 0 "#PWR?" H 10100 2150 50  0001 C CNN
 F 1 "+3.3V" H 10115 2473 50  0000 C CNN
 F 2 "" H 10100 2300 50  0001 C CNN

Commit message: I forgot to annotate things again
Parts:
- gave numbers to parts that had none: 13
Changed lines of the file:
@@
 $EndDescr
 $Comp
-L FPGA_Xilinx_Artix7:XC7A100T-FTG256 U?
+L FPGA_Xilinx_Artix7:XC7A100T-FTG256 U3
 U 2 1 5D8696A8
 P 18000 5400
-F 0 "U?" H 18000 2425 50  0000 C CNN
+F 0 "U3" H 18000 2425 50  0000 C CNN
 F 1 "XC7A100T-FTG256" H 18000 2334 50  0000 C CNN
 F 2 "Package_BGA:Xilinx_FTG256" H 18000 5400 50  0001 C CNN
@@
 $EndComp
 $Comp
-L FPGA_Xilinx_Artix7:XC7A100T-FTG256 U?
+L FPGA_Xilinx_Artix7:XC7A100T-FTG256 U3
 U 3 1 5D86EF6E
 P 4900 6600
-F 0 "U?" H 3620 6653 50  0000 R CNN
+F 0 "U3" H 3620 6653 50  0000 R CNN
 F 1 "XC7A100T-FTG256" H 3620 6562 50  0000 R CNN
 F 2 "Package_BGA:Xilinx_FTG256" H 4900 6600 50  0001 C CNN
@@
 $EndComp
 $Comp
-L FPGA_Xilinx_Artix7:XC7A100T-FTG256 U?
+L FPGA_Xilinx_Artix7:XC7A100T-FTG256 U3
 U 4 1 5D871AA2
 P 2950 12150
-F 0 "U?" H 2950 13717 50  0000 C CNN
+F 0 "U3" H 2950 13717 50  0000 C CNN
 F 1 "XC7A100T-FTG256" H 2950 13626 50  0000 C CNN
 F 2 "Package_BGA:Xilinx_FTG256" H 2950 12150 50  0001 C CNN
@@
 	3250 3700 3250 3400
 $Comp
-L Device:R R?
+L Device:R R1
 U 1 1 5D8D19E7
 P 1400 2750
-F 0 "R?" H 1470 2796 50  0000 L CNN
+F 0 "R1" H 1470 2796 50  0000 L CNN
 F 1 "2.4k" H 1470 2705 50  0000 L CNN
 F 2 "Resistor_SMD:R_1206_3216Metric_Pad1.42x1.75mm_HandSolder" V 1330 2750 50  0001 C CNN
@@
 	1400 3400 1400 3150
 $Comp
-L Device:R R?
+L Device:R R3
 U 1 1 5D8D15D8
 P 1750 2750
-F 0 "R?" H 1820 2796 50  0000 L CNN
+F 0 "R3" H 1820 2796 50  0000 L CNN
 F 1 "4.7k" H 1820 2705 50  0000 L CNN
 F 2 "Resistor_SMD:R_1206_3216Metric_Pad1.42x1.75mm_HandSolder" V 1680 2750 50  0001 C CNN
@@
 Connection ~ 2750 2400
 $Comp
-L Device:R R?
+L Device:R R8
 U 1 1 5D8D0364
 P 3100 2800
-F 0 "R?" H 3170 2846 50  0000 L CNN
+F 0 "R8" H 3170 2846 50  0000 L CNN
 F 1 "4.7k" H 3170 2755 50  0000 L CNN
 F 2 "Resistor_SMD:R_1206_3216Metric_Pad1.42x1.75mm_HandSolder" V 3030 2800 50  0001 C CNN
@@
 	1300 3500 1300 3050
 $Comp
-L power:GND #PWR?
+L power:GND #PWR018
 U 1 1 5D95B8C6
 P 6800 3850
-F 0 "#PWR?" H 6800 3600 50  0001 C CNN
+F 0 "#PWR018" H 6800 3600 50  0001 C CNN
 F 1 "GND" H 6805 3677 50  0000 C CNN
 F 2 "" H 6800 3850 50  0001 C CNN
@@
 	1600 3400 1400 3400
 $Comp
-L Synth:S25FL127S U?
+L Synth:S25FL127S U2
 U 1 1 5D8B8019
 P 1950 3500
-F 0 "U?" H 2175 3865 50  0000 C CNN
+F 0 "U2" H 2175 3865 50  0000 C CNN
 F 1 "S25FL127S" H 2175 3774 50  0000 C CNN
 F 2 "Package_SO:SOIC-8-1EP_3.9x4.9mm_P1.27mm_EP2.41x3.81mm" H 1950 3500 50  0001 C CNN
@@
 Connection ~ 1000 3850
 $Comp
-L power:GND #PWR?
+L power:GND #PWR07
 U 1 1 5D8B9BD9
 P 1000 3850
-F 0 "#PWR?" H 1000 3600 50  0001 C CNN
+F 0 "#PWR07" H 1000 3600 50  0001 C CNN
 F 1 "GND" H 1005 3677 50  0000 C CNN
 F 2 "" H 1000 3850 50  0001 C CNN
@@
 $EndComp
 $Comp
-L Device:C C?
+L Device:C C3
 U 1 1 5D8D3873
 P 1000 2800
-F 0 "C?" H 1115 2846 50  0000 L CNN
+F 0 "C3" H 1115 2846 50  0000 L CNN
 F 1 "100n" H 1115 2755 50  0000 L CNN
 F 2 "Capacitor_SMD:C_1206_3216Metric_Pad1.42x1.75mm_HandSolder" H 1038 2650 50  0001 C CNN
@@
 	2850 3600 2850 6300
 $Comp
-L Device:R R?
+L Device:R R4
 U 1 1 5DB16E52
 P 1750 4850
-F 0 "R?" H 1820 4896 50  0000 L CNN
+F 0 "R4" H 1820 4896 50  0000 L CNN
 F 1 "10k" H 1820 4805 50  0000 L CNN
 F 2 "Resistor_SMD:R_1206_3216Metric_Pad1.42x1.75mm_HandSolder" V 1680 4850 50  0001 C CNN
@@
 $EndComp
 $Comp
-L Device:R R?
+L Device:R R5
 U 1 1 5DB1753D
 P 2000 4850
-F 0 "R?" H 2070 4896 50  0000 L CNN
+F 0 "R5" H 2070 4896 50  0000 L CNN
 F 1 "4.7k" H 2070 4805 50  0000 L CNN
 F 2 "Resistor_SMD:R_1206_3216Metric_Pad1.42x1.75mm_HandSolder" V 1930 4850 50  0001 C CNN
@@
 $EndComp
 $Comp
-L Device:R R?
+L Device:R R2
 U 1 1 5DB17AAB
 P 1500 4850
-F 0 "R?" H 1570 4896 50  0000 L CNN
+F 0 "R2" H 1570 4896 50  0000 L CNN
 F 1 "10k" H 1570 4805 50  0000 L CNN
 F 2 "Resistor_SMD:R_1206_3216Metric_Pad1.42x1.75mm_HandSolder" V 1430 4850 50  0001 C CNN
@@
 $EndComp
 $Comp
-L Device:R R?
+L Device:R R6
 U 1 1 5DB18145
 P 2250 4850
-F 0 "R?" H 2320 4896 50  0000 L CNN
+F 0 "R6" H 2320 4896 50  0000 L CNN
 F 1 "4.7k" H 2320 4805 50  0000 L CNN
 F 2 "Resistor_SMD:R_1206_3216Metric_Pad1.42x1.75mm_HandSolder" V 2180 4850 50  0001 C CNN
@@
 $EndComp
 $Comp
-L Device:R R?
+L Device:R R7
 U 1 1 5DB18715
 P 2450 4850
-F 0 "R?" H 2520 4896 50  0000 L CNN
+F 0 "R7" H 2520 4896 50  0000 L CNN
 F 1 "330" H 2520 4805 50  0000 L CNN
 F 2 "Resistor_SMD:R_1206_3216Metric_Pad1.42x1.75mm_HandSolder" V 2380 4850 50  0001 C CNN
@@
 AR Path="/5DB1FB59" Ref="J?"  Part="1"
 AR Path="/5D81B1F5/5DB1FB59" Ref="J4"  Part="1"
-F 0 "J?" H 1100 6425 50  0000 C CNN
+F 0 "J4" H 1100 6425 50  0000 C CNN
 F 1 "FPGA_debug" H 1100 6334 50  0000 C CNN
 F 2 "Connector_PinHeader_2.00mm:PinHeader_2x07_P2.00mm_Vertical" H 1100 6300 50  0001 C CNN
@@
 $EndComp
 $Comp
-L power:GND #PWR?
+L power:GND #PWR06
 U 1 1 5DB20A30
 P 850 6450
-F 0 "#PWR?" H 850 6200 50  0001 C CNN
+F 0 "#PWR06" H 850 6200 50  0001 C CNN
 F 1 "GND" H 855 6277 50  0000 C CNN
 F 2 "" H 850 6450 50  0001 C CNN
@@
 	3400 6800 2450 6800
 $Comp
-L power:GND #PWR?
+L power:GND #PWR015
 U 1 1 5DB930FB
 P 3200 8400
-F 0 "#PWR?" H 3200 8150 50  0001 C CNN
+F 0 "#PWR015" H 3200 8150 50  0001 C CNN
 F 1 "GND" H 3205 8227 50  0000 C CNN
 F 2 "" H 3200 8400 50  0001 C CNN
@@
 	9200 5800 6900 5800
 $Comp
-L Synth:Oscillator U?
+L Synth:Oscillator U4
 U 1 1 5DBDB09B
 P 6650 5750
-F 0 "U?" H 6683 6125 50  0000 C CNN
+F 0 "U4" H 6683 6125 50  0000 C CNN
 F 1 "Oscillator" H 6683 6034 50  0000 C CNN
 F 2 "Oscillator:Oscillator_SMD_Abracon_ASCO-4Pin_1.6x1.2mm" H 6700 5700 50  0001 C CNN
@@
 $EndComp
 $Comp
-L power:GND #PWR?
+L power:GND #PWR020
 U 1 1 5DC0D0A3
 P 7300 6000
-F 0 "#PWR?" H 7300 5750 50  0001 C CNN
+F 0 "#PWR020" H 7300 5750 50  0001 C CNN
 F 1 "GND" H 7305 5827 50  0000 C CNN
 F 2 "" H 7300 6000 50  0001 C CNN
@@
 	7100 5900 7100 5600
 $Comp
-L Device:C C?
+L Device:C C4
 U 1 1 5DC18FF3
 P 7400 5450
-F 0 "C?" H 7515 5496 50  0000 L CNN
+F 0 "C4" H 7515 5496 50  0000 L CNN
 F 1 "100n" H 7515 5405 50  0000 L CNN
 F 2 "Capacitor_SMD:C_1206_3216Metric_Pad1.42x1.75mm_HandSolder" H 7438 5300 50  0001 C CNN
@@
 Connection ~ 1950 11650
 $Comp
-L power:GND #PWR?
+L power:GND #PWR014
 U 1 1 5DC8F87F
 P 2950 13650
-F 0 "#PWR?" H 2950 13400 50  0001 C CNN
+F 0 "#PWR014" H 2950 13400 50  0001 C CNN
 F 1 "GND" H 2955 13477 50  0000 C CNN
 F 2 "" H 2950 13650 50  0001 C CNN
@@
 	1850 11550 1850 13650
 $Comp
-L power:GND #PWR?
+L power:GND #PWR023
 U 1 1 5DD18602
 P 18050 2500
-F 0 "#PWR?" H 18050 2250 50  0001 C CNN
+F 0 "#PWR023" H 18050 2250 50  0001 C CNN
 F 1 "GND" H 18055 2327 50  0000 C CNN
 F 2 "" H 18050 2500 50  0001 C CNN
@@
 	3800 4900 3800 5000
 $Comp
-L power:GND #PWR?
+L power:GND #PWR022
 U 1 1 5D8EC9FF
 P 12300 2350
-F 0 "#PWR?" H 12300 2100 50  0001 C CNN
+F 0 "#PWR022" H 12300 2100 50  0001 C CNN
 F 1 "GND" H 12305 2177 50  0000 C CNN
 F 2 "" H 12300 2350 50  0001 C CNN
@@
 	1200 11550 1200 11650
 $Comp
-L power:+1V8 #PWR?
+L power:+1V8 #PWR010
 U 1 1 5E1CD4BD
 P 1800 10850
-F 0 "#PWR?" H 1800 10700 50  0001 C CNN
+F 0 "#PWR010" H 1800 10700 50  0001 C CNN
 F 1 "+1V8" H 1815 11023 50  0000 C CNN
 F 2 "" H 1800 10850 50  0001 C CNN
@@
 $EndComp
 $Comp
-L power:+1V0 #PWR?
+L power:+1V0 #PWR08
 U 1 1 5E1CEB46
 P 1200 11550
-F 0 "#PWR?" H 1200 11400 50  0001 C CNN
+F 0 "#PWR08" H 1200 11400 50  0001 C CNN
 F 1 "+1V0" H 1215 11723 50  0000 C CNN
 F 2 "" H 1200 11550 50  0001 C CNN
@@
 $EndComp
 $Comp
-L power:+1V0 #PWR?
+L power:+1V0 #PWR017
 U 1 1 5E1D1568
 P 4200 10850
-F 0 "#PWR?" H 4200 10700 50  0001 C CNN
+F 0 "#PWR017" H 4200 10700 50  0001 C CNN
 F 1 "+1V0" V 4215 10978 50  0000 L CNN
 F 2 "" H 4200 10850 50  0001 C CNN
@@
 $EndComp
 $Comp
-L power:+3.3V #PWR?
+L power:+3.3V #PWR019
 U 1 1 5D914A91
 P 7100 5050
-F 0 "#PWR?" H 7100 4900 50  0001 C CNN
+F 0 "#PWR019" H 7100 4900 50  0001 C CNN
 F 1 "+3.3V" H 7115 5223 50  0000 C CNN
 F 2 "" H 7100 5050 50  0001 C CNN
@@
 $EndComp
 $Comp
-L power:+3.3V #PWR?
+L power:+3.3V #PWR016
 U 1 1 5D9199D3
 P 3800 4900
-F 0 "#PWR?" H 3800 4750 50  0001 C CNN
+F 0 "#PWR016" H 3800 4750 50  0001 C CNN
 F 1 "+3.3V" H 3815 5073 50  0000 C CNN
 F 2 "" H 3800 4900 50  0001 C CNN
@@
 $EndComp
 $Comp
-L power:+3.3V #PWR?
+L power:+3.3V #PWR011
 U 1 1 5D91E70E
 P 2000 4300
-F 0 "#PWR?" H 2000 4150 50  0001 C CNN
+F 0 "#PWR011" H 2000 4150 50  0001 C CNN
 F 1 "+3.3V" H 2015 4473 50  0000 C CNN
 F 2 "" H 2000 4300 50  0001 C CNN
@@
 $EndComp
 $Comp
-L power:+3.3V #PWR?
+L power:+3.3V #PWR013
 U 1 1 5D920C94
 P 2750 2400
-F 0 "#PWR?" H 2750 2250 50  0001 C CNN
+F 0 "#PWR013" H 2750 2250 50  0001 C CNN
 F 1 "+3.3V" H 2765 2573 50  0000 C CNN
 F 2 "" H 2750 2400 50  0001 C CNN
@@
 $EndComp
 $Comp
-L power:+3.3V #PWR?
+L power:+3.3V #PWR012
 U 1 1 5D936054
 P 2700 6400
-F 0 "#PWR?" H 2700 6250 50  0001 C CNN
+F 0 "#PWR012" H 2700 6250 50  0001 C CNN
 F 1 "+3.3V" H 2715 6573 50  0000 C CNN
 F 2 "" H 2700 6400 50  0001 C CNN
@@
 	12400 2500 12300 2500
 $Comp
-L FPGA_Xilinx_Artix7:XC7A100T-FTG256 U?
+L FPGA_Xilinx_Artix7:XC7A100T-FTG256 U3
 U 1 1 5D866531
 P 11200 5400
-F 0 "U?" H 11200 2425 50  0000 C CNN
+F 0 "U3" H 11200 2425 50  0000 C CNN
 F 1 "XC7A100T-FTG256" H 11200 2334 50  0000 C CNN
 F 2 "Package_BGA:Xilinx_FTG256" H 11200 5400 50  0001 C CNN
@@
 	9600 2500 9600 2400
 $Comp
-L power:+3.3V #PWR?
+L power:+3.3V #PWR021
 U 1 1 5D9F7116
 P 10100 2300
-F 0 "#PWR?" H 10100 2150 50  0001 C CNN
+F 0 "#PWR021" H 10100 2150 50  0001 C CNN
 F 1 "+3.3V" H 10115 2473 50  0000 C CNN
 F 2 "" H 10100 2300 50  0001 C CNN
