File: Artix.sch (KiCad schematic (older format))
At the start: 14 parts, among them J4 FPGA_debug, U2 S25FL127S, U3 XC7A100T-FTG256, U4 Oscillator

Commit message: Added in the potentiometers, fixed some faulty pins on the artix, rewired some pins on the MCU so they didn't interfere with the crystal.
Connections:
- net labels added: DAC_BCK, DAC_DATA, DAC_LRCK, DAC_SCK
- net labels removed: IO_L4N_T0_D05_14, IO_L4P_T0_D04_14, IO_L5P_T0_D06_14, IO_L5P_T0_D07_14
Changed lines of the file:
@@
 $EndComp
 Text HLabel 7800 4000 0    50   Output ~ 0
-IO_L4P_T0_D04_14
+DAC_SCK
 Text HLabel 7800 4100 0    50   Output ~ 0
-IO_L4N_T0_D05_14
+DAC_BCK
 Text HLabel 7800 4200 0    50   Output ~ 0
-IO_L5P_T0_D06_14
+DAC_DATA
 Text HLabel 7800 4300 0    50   Output ~ 0
-IO_L5P_T0_D07_14
+DAC_LRCK
 Wire Wire Line
 	9200 4000 7800 4000

Commit message: Wired up the potentiometers.
Connections:
- wire segments 208 -> 211
Changed lines of the file:
@@
 	1800 10750 1800 10850
 Wire Wire Line
-	1800 10850 1950 10850
-Wire Wire Line
 	1950 11650 1200 11650
-Wire Wire Line
-	1950 11150 1950 11050
-Connection ~ 1950 10850
-Connection ~ 1950 10950
-Wire Wire Line
-	1950 10950 1950 10850
-Connection ~ 1950 11050
-Wire Wire Line
-	1950 11050 1950 10950
 Wire Wire Line
 	1950 11750 1950 11650
@@
 	3950 11350 3950 11450
 Wire Wire Line
-	1950 11450 1800 11450
-Wire Wire Line
-	1800 11450 1800 10850
+	1800 11450 1800 11150
 Connection ~ 1800 10850
 Wire Wire Line
@@
 L power:+1V8 #PWR010
 U 1 1 5E1CD4BD
-P 1800 10850
-F 0 "#PWR010" H 1800 10700 50  0001 C CNN
-F 1 "+1V8" H 1815 11023 50  0000 C CNN
-F 2 "" H 1800 10850 50  0001 C CNN
-F 3 "" H 1800 10850 50  0001 C CNN
-	1    1800 10850
+P 1800 10750
+F 0 "#PWR010" H 1800 10600 50  0001 C CNN
+F 1 "+1V8" H 1815 10923 50  0000 C CNN
+F 2 "" H 1800 10750 50  0001 C CNN
+F 3 "" H 1800 10750 50  0001 C CNN
+	1    1800 10750
 	1    0    0    -1
 $EndComp
@@
 Text HLabel 7800 4200 0    50   Output ~ 0
 DAC_DATA
-Text HLabel 7800 4300 0    50   Output ~ 0
-DAC_LRCK
 Wire Wire Line
 	9200 4000 7800 4000
@@
 Wire Wire Line
 	9200 5400 8350 5400
+Text HLabel 7800 4300 0    50   Output ~ 0
+DAC_LRCK
+Wire Wire Line
+	1950 11150 1800 11150
+Connection ~ 1800 11150
+Wire Wire Line
+	1800 11150 1800 11050
+Wire Wire Line
+	1950 11050 1800 11050
+Connection ~ 1800 11050
+Wire Wire Line
+	1800 11050 1800 10950
+Wire Wire Line
+	1950 10950 1800 10950
+Connection ~ 1800 10950
+Wire Wire Line
+	1800 10950 1800 10850
+Wire Wire Line
+	1950 10850 1800 10850
+Wire Wire Line
+	1950 11450 1800 11450
 $EndSCHEMATC

Commit message: Started wiring the flash chip.
Changed lines of the file:
@@
 	1    0    0    -1
 $EndComp
-Wire Wire Line
-	6900 5900 7100 5900
-Wire Wire Line
-	7100 5900 7100 5600
 $Comp
 L Device:C C4
@@
 Wire Wire Line
 	6900 5700 7300 5700
-Wire Wire Line
-	7100 5600 6900 5600
-Connection ~ 7100 5600
-Wire Wire Line
-	7100 5600 7100 5050
 Wire Wire Line
 	7300 5700 7300 6000
@@
 Wire Wire Line
 	1950 11450 1800 11450
+Wire Wire Line
+	7100 5050 7100 5600
+Wire Wire Line
+	7100 5900 6900 5900
+Wire Wire Line
+	6900 5600 7100 5600
+Connection ~ 7100 5600
+Wire Wire Line
+	7100 5600 7100 5900
 $EndSCHEMATC

Commit message: Wire up 1V PSU. Use smaller footprints for small caps.
Parts:
- C3, C4: footprint Capacitor_SMD:C_1206_3216Metric_Pad1.42x1.75mm_HandSolder -> Capacitor_SMD:C_0805_2012Metric_Pad1.15x1.40mm_HandSolder
Changed lines of the file:
@@
 F 0 "C3" H 1115 2846 50  0000 L CNN
 F 1 "100n" H 1115 2755 50  0000 L CNN
-F 2 "Capacitor_SMD:C_1206_3216Metric_Pad1.42x1.75mm_HandSolder" H 1038 2650 50  0001 C CNN
+F 2 "Capacitor_SMD:C_0805_2012Metric_Pad1.15x1.40mm_HandSolder" H 1038 2650 50  0001 C CNN
 F 3 "~" H 1000 2800 50  0001 C CNN
 	1    1000 2800
@@
 F 0 "C4" H 7515 5496 50  0000 L CNN
 F 1 "100n" H 7515 5405 50  0000 L CNN
-F 2 "Capacitor_SMD:C_1206_3216Metric_Pad1.42x1.75mm_HandSolder" H 7438 5300 50  0001 C CNN
+F 2 "Capacitor_SMD:C_0805_2012Metric_Pad1.15x1.40mm_HandSolder" H 7438 5300 50  0001 C CNN
 F 3 "~" H 7400 5450 50  0001 C CNN
 	1    7400 5450
