File: Artix.sch (KiCad schematic (older format))
At the start: 14 parts, among them J4 FPGA_debug, U2 S25FL127S, U3 XC7A100T-FTG256, U4 Oscillator

Commit message: Rearrange and rewire most of the PCB
Parts:
- added J?: 67997-410HLF, footprints:67997-410HLF, symbol Header:67997-410HLF
Connections:
- wire segments 211 -> 244
- no-connect marks 153 -> 145
Changed lines of the file:
@@
 NoConn ~ 9200 6300
 NoConn ~ 9200 6400
-NoConn ~ 9200 6500
-NoConn ~ 9200 6600
-NoConn ~ 9200 6700
-NoConn ~ 9200 6800
-NoConn ~ 9200 6900
-NoConn ~ 9200 7000
-NoConn ~ 9200 7100
-NoConn ~ 9200 7200
 NoConn ~ 9200 7300
 NoConn ~ 9200 7400
@@
 Wire Wire Line
 	7100 5600 7100 5900
+$Comp
+L Header:67997-410HLF J?
+U 1 1 5D918194
+P 7800 7900
+F 0 "J?" H 8450 8387 60  0000 C CNN
+F 1 "67997-410HLF" H 8450 8281 60  0000 C CNN
+F 2 "footprints:67997-410HLF" H 8450 8240 60  0001 C CNN
+F 3 "" H 7800 8050 60  0000 C CNN
+	1    7800 7900
+	0    -1   -1   0
+$EndComp
+$Comp
+L power:+3.3V #PWR?
+U 1 1 5D9235DF
+P 7500 7900
+F 0 "#PWR?" H 7500 7750 50  0001 C CNN
+F 1 "+3.3V" H 7515 8073 50  0000 C CNN
+F 2 "" H 7500 7900 50  0001 C CNN
+F 3 "" H 7500 7900 50  0001 C CNN
+	1    7500 7900
+	0    -1   -1   0
+$EndComp
+Wire Wire Line
+	7500 7900 7650 7900
+$Comp
+L power:GND #PWR?
+U 1 1 5D939EBE
+P 8200 6600
+F 0 "#PWR?" H 8200 6350 50  0001 C CNN
+F 1 "GND" H 8205 6427 50  0000 C CNN
+F 2 "" H 8200 6600 50  0001 C CNN
+F 3 "" H 8200 6600 50  0001 C CNN
+	1    8200 6600
+	0    -1   -1   0
+$EndComp
+Wire Wire Line
+	8050 6600 8200 6600
+Wire Wire Line
+	7950 6600 7950 6500
+Wire Wire Line
+	7950 6500 8450 6500
+Wire Wire Line
+	8450 6500 8450 6800
+Wire Wire Line
+	8450 6800 9200 6800
+Wire Wire Line
+	8550 6700 8550 6400
+Wire Wire Line
+	8550 6400 7850 6400
+Wire Wire Line
+	7850 6400 7850 6600
+Wire Wire Line
+	8550 6700 9200 6700
+Wire Wire Line
+	7750 6600 7750 6300
+Wire Wire Line
+	7750 6300 8650 6300
+Wire Wire Line
+	8650 6300 8650 6600
+Wire Wire Line
+	8650 6600 9200 6600
+Wire Wire Line
+	7650 6600 7650 6200
+Wire Wire Line
+	7650 6200 8750 6200
+Wire Wire Line
+	8750 6200 8750 6500
+Wire Wire Line
+	8750 6500 9200 6500
+Wire Wire Line
+	8050 7900 8450 7900
+Wire Wire Line
+	8450 7900 8450 6900
+Wire Wire Line
+	8450 6900 9200 6900
+Wire Wire Line
+	7950 7900 7950 8000
+Wire Wire Line
+	7950 8000 8550 8000
+Wire Wire Line
+	8550 8000 8550 7000
+Wire Wire Line
+	8550 7000 9200 7000
+Wire Wire Line
+	7850 7900 7850 8100
+Wire Wire Line
+	7850 8100 8650 8100
+Wire Wire Line
+	8650 8100 8650 7100
+Wire Wire Line
+	8650 7100 9200 7100
+Wire Wire Line
+	7750 7900 7750 8200
+Wire Wire Line
+	7750 8200 8750 8200
+Wire Wire Line
+	8750 8200 8750 7200
+Wire Wire Line
+	8750 7200 9200 7200
 $EndSCHEMATC

Commit message: Added in a bunch of footprints to the netlist; only missing buttons and some resistors, now.
Parts:
- gave numbers to parts that had none: 1
Changed lines of the file:
@@
 	7100 5600 7100 5900
 $Comp
-L Header:67997-410HLF J?
+L Header:67997-410HLF J7
 U 1 1 5D918194
 P 7800 7900
-F 0 "J?" H 8450 8387 60  0000 C CNN
+F 0 "J7" H 8450 8387 60  0000 C CNN
 F 1 "67997-410HLF" H 8450 8281 60  0000 C CNN
 F 2 "footprints:67997-410HLF" H 8450 8240 60  0001 C CNN
@@
 $EndComp
 $Comp
-L power:+3.3V #PWR?
+L power:+3.3V #PWR0120
 U 1 1 5D9235DF
 P 7500 7900
-F 0 "#PWR?" H 7500 7750 50  0001 C CNN
+F 0 "#PWR0120" H 7500 7750 50  0001 C CNN
 F 1 "+3.3V" H 7515 8073 50  0000 C CNN
 F 2 "" H 7500 7900 50  0001 C CNN
@@
 	7500 7900 7650 7900
 $Comp
-L power:GND #PWR?
+L power:GND #PWR0122
 U 1 1 5D939EBE
 P 8200 6600
-F 0 "#PWR?" H 8200 6350 50  0001 C CNN
+F 0 "#PWR0122" H 8200 6350 50  0001 C CNN
 F 1 "GND" H 8205 6427 50  0000 C CNN
 F 2 "" H 8200 6600 50  0001 C CNN

Commit message: Fix a few more noclipping objects and labels
Parts:
- J7: value 67997-410HLF -> FPGA_GPIO
Changed lines of the file:
@@
 P 7800 7900
 F 0 "J7" H 8450 8387 60  0000 C CNN
-F 1 "67997-410HLF" H 8450 8281 60  0000 C CNN
+F 1 "FPGA_GPIO" H 8450 8281 60  0000 C CNN
 F 2 "footprints:67997-410HLF" H 8450 8240 60  0001 C CNN
 F 3 "" H 7800 8050 60  0000 C CNN

Commit message: Fixed pin header footprints, rewired. I think it's done?
Parts:
- J4: footprint Connector_PinHeader_2.00mm:PinHeader_2x07_P2.00mm_Vertical -> Connector_PinHeader_2.54mm:PinHeader_2x07_P2.54mm_Vertical
Changed lines of the file:
@@
 F 0 "J4" H 1100 6425 50  0000 C CNN
 F 1 "FPGA_debug" H 1100 6334 50  0000 C CNN
-F 2 "Connector_PinHeader_2.00mm:PinHeader_2x07_P2.00mm_Vertical" H 1100 6300 50  0001 C CNN
+F 2 "Connector_PinHeader_2.54mm:PinHeader_2x07_P2.54mm_Vertical" H 1100 6300 50  0001 C CNN
 F 3 "" H 1100 6300 50  0001 C CNN
 	1    1100 5900
