File: PSU.sch (KiCad schematic (older format))
At the start: 34 parts, among them U5 TPS54325, U6 TPS54294

Commit message: Fixed u being written as µ (my bad.) Tried doing work on the PSU but it's eldritch.
Parts:
- C50, C51, C67, C68: value 22µ -> 22u
- C62: value 1µ -> 1u
Changed lines of the file:
@@
 AR Path="/5DC1AA2E/5DCDC93D" Ref="C67"  Part="1"
 F 0 "C67" H 8015 4846 50  0000 L CNN
-F 1 "22µ" H 8015 4755 50  0000 L CNN
+F 1 "22u" H 8015 4755 50  0000 L CNN
 F 2 "Capacitor_SMD:C_0805_2012Metric_Pad1.15x1.40mm_HandSolder" H 7938 4650 50  0001 C CNN
 F 3 "~" H 7900 4800 50  0001 C CNN
@@
 AR Path="/5DC1AA2E/5DCDC943" Ref="C68"  Part="1"
 F 0 "C68" H 8365 4846 50  0000 L CNN
-F 1 "22µ" H 8365 4755 50  0000 L CNN
+F 1 "22u" H 8365 4755 50  0000 L CNN
 F 2 "Capacitor_SMD:C_0805_2012Metric_Pad1.15x1.40mm_HandSolder" H 8288 4650 50  0001 C CNN
 F 3 "~" H 8250 4800 50  0001 C CNN
@@
 AR Path="/5DC1AA2E/5DCDC9C1" Ref="C51"  Part="1"
 F 0 "C51" H 3150 4900 50  0000 L CNN
-F 1 "22µ" H 3150 4700 50  0000 L CNN
+F 1 "22u" H 3150 4700 50  0000 L CNN
 F 2 "Capacitor_SMD:C_0805_2012Metric_Pad1.15x1.40mm_HandSolder" H 3188 4650 50  0001 C CNN
 F 3 "~" H 3150 4800 50  0001 C CNN
@@
 AR Path="/5DC1AA2E/5DCDC9C7" Ref="C50"  Part="1"
 F 0 "C50" H 2900 4900 50  0000 L CNN
-F 1 "22µ" H 2900 4700 50  0000 L CNN
+F 1 "22u" H 2900 4700 50  0000 L CNN
 F 2 "Capacitor_SMD:C_0805_2012Metric_Pad1.15x1.40mm_HandSolder" H 2938 4650 50  0001 C CNN
 F 3 "~" H 2900 4800 50  0001 C CNN
@@
 AR Path="/5DC1AA2E/5DCDC8F8" Ref="C62"  Part="1"
 F 0 "C62" H 6665 5146 50  0000 L CNN
-F 1 "1µ" H 6665 5055 50  0000 L CNN
+F 1 "1u" H 6665 5055 50  0000 L CNN
 F 2 "Capacitor_SMD:C_0805_2012Metric_Pad1.15x1.40mm_HandSolder" H 6588 4950 50  0001 C CNN
 F 3 "~" H 6550 5100 50  0001 C CNN

Commit message: Updated component footprints. The PCB is now an unholy mess.
Parts:
- C50, C51, C52, C53, C54, C55, C56, C57, C58, C59, C60, C61, C62, C63, C64, C65, C66, C67, C68: footprint Capacitor_SMD:C_0805_2012Metric_Pad1.15x1.40mm_HandSolder -> Capacitor_SMD:C_1206_3216Metric_Pad1.42x1.75mm_HandSolder
- FB5: renamed from L4; footprint Inductor_SMD:L_0805_2012Metric_Pad1.15x1.40mm_HandSolder -> footprints:FerriteBead_74279215
- R10, R11, R12, R13, R14, R15, R16, R17, R9: footprint Resistor_SMD:R_0805_2012Metric_Pad1.15x1.40mm_HandSolder -> Resistor_SMD:R_1206_3216Metric_Pad1.42x1.75mm_HandSolder
Changed lines of the file:
@@
 F 0 "C54" H 4250 4500 50  0000 L CNN
 F 1 "0.1u" H 4250 4300 50  0000 L CNN
-F 2 "Capacitor_SMD:C_0805_2012Metric_Pad1.15x1.40mm_HandSolder" H 4288 4250 50  0001 C CNN
+F 2 "Capacitor_SMD:C_1206_3216Metric_Pad1.42x1.75mm_HandSolder" H 4288 4250 50  0001 C CNN
 F 3 "~" H 4250 4400 50  0001 C CNN
 	1    4250 4400
@@
 F 0 "R14" H 6970 5146 50  0000 L CNN
 F 1 "100k" H 6970 5055 50  0000 L CNN
-F 2 "Resistor_SMD:R_0805_2012Metric_Pad1.15x1.40mm_HandSolder" V 6830 5100 50  0001 C CNN
+F 2 "Resistor_SMD:R_1206_3216Metric_Pad1.42x1.75mm_HandSolder" V 6830 5100 50  0001 C CNN
 F 3 "~" H 6900 5100 50  0001 C CNN
 	1    6900 5100
@@
 F 0 "C64" H 6915 4396 50  0000 L CNN
 F 1 "0.1u" H 6915 4305 50  0000 L CNN
-F 2 "Capacitor_SMD:C_0805_2012Metric_Pad1.15x1.40mm_HandSolder" H 6838 4200 50  0001 C CNN
+F 2 "Capacitor_SMD:C_1206_3216Metric_Pad1.42x1.75mm_HandSolder" H 6838 4200 50  0001 C CNN
 F 3 "~" H 6800 4350 50  0001 C CNN
 	1    6800 4350
@@
 F 0 "R16" H 7520 5246 50  0000 L CNN
 F 1 "22.1k" H 7520 5155 50  0000 L CNN
-F 2 "Resistor_SMD:R_0805_2012Metric_Pad1.15x1.40mm_HandSolder" V 7380 5200 50  0001 C CNN
+F 2 "Resistor_SMD:R_1206_3216Metric_Pad1.42x1.75mm_HandSolder" V 7380 5200 50  0001 C CNN
 F 3 "~" H 7450 5200 50  0001 C CNN
 	1    7450 5200
@@
 F 0 "R15" H 7520 4846 50  0000 L CNN
 F 1 "73.2k" H 7520 4755 50  0000 L CNN
-F 2 "Resistor_SMD:R_0805_2012Metric_Pad1.15x1.40mm_HandSolder" V 7380 4800 50  0001 C CNN
+F 2 "Resistor_SMD:R_1206_3216Metric_Pad1.42x1.75mm_HandSolder" V 7380 4800 50  0001 C CNN
 F 3 "~" H 7450 4800 50  0001 C CNN
 	1    7450 4800
@@
 F 0 "C67" H 8015 4846 50  0000 L CNN
 F 1 "22u" H 8015 4755 50  0000 L CNN
-F 2 "Capacitor_SMD:C_0805_2012Metric_Pad1.15x1.40mm_HandSolder" H 7938 4650 50  0001 C CNN
+F 2 "Capacitor_SMD:C_1206_3216Metric_Pad1.42x1.75mm_HandSolder" H 7938 4650 50  0001 C CNN
 F 3 "~" H 7900 4800 50  0001 C CNN
 	1    7900 4800
@@
 F 0 "C68" H 8365 4846 50  0000 L CNN
 F 1 "22u" H 8365 4755 50  0000 L CNN
-F 2 "Capacitor_SMD:C_0805_2012Metric_Pad1.15x1.40mm_HandSolder" H 8288 4650 50  0001 C CNN
+F 2 "Capacitor_SMD:C_1206_3216Metric_Pad1.42x1.75mm_HandSolder" H 8288 4650 50  0001 C CNN
 F 3 "~" H 8250 4800 50  0001 C CNN
 	1    8250 4800
@@
 P 9000 4550
 AR Path="/5DCDC955" Ref="L?"  Part="1"
-AR Path="/5DC1AA2E/5DCDC955" Ref="L4"  Part="1"
-F 0 "L4" V 9274 4550 50  0000 C CNN
+AR Path="/5DC1AA2E/5DCDC955" Ref="FB5"  Part="1"
+F 0 "FB5" V 9274 4550 50  0000 C CNN
 F 1 "Ferrite_Bead" V 9183 4550 50  0000 C CNN
-F 2 "Inductor_SMD:L_0805_2012Metric_Pad1.15x1.40mm_HandSolder" V 8930 4550 50  0001 C CNN
+F 2 "footprints:FerriteBead_74279215" V 8930 4550 50  0001 C CNN
 F 3 "~" H 9000 4550 50  0001 C CNN
 	1    9000 4550
@@
 F 0 "R17" V 9293 4550 50  0000 C CNN
 F 1 "1" V 9384 4550 50  0000 C CNN
-F 2 "Resistor_SMD:R_0805_2012Metric_Pad1.15x1.40mm_HandSolder" V 9430 4550 50  0001 C CNN
+F 2 "Resistor_SMD:R_1206_3216Metric_Pad1.42x1.75mm_HandSolder" V 9430 4550 50  0001 C CNN
 F 3 "~" H 9500 4550 50  0001 C CNN
 	1    9500 4550
@@
 F 0 "C58" H 6200 4150 50  0000 L CNN
 F 1 "10u" H 6200 3950 50  0000 L CNN
-F 2 "Capacitor_SMD:C_0805_2012Metric_Pad1.15x1.40mm_HandSolder" H 6238 3900 50  0001 C CNN
+F 2 "Capacitor_SMD:C_1206_3216Metric_Pad1.42x1.75mm_HandSolder" H 6238 3900 50  0001 C CNN
 F 3 "~" H 6200 4050 50  0001 C CNN
 	1    6200 4050
@@
 F 0 "C60" H 6515 4096 50  0000 L CNN
 F 1 "100n" H 6500 4000 50  0000 L CNN
-F 2 "Capacitor_SMD:C_0805_2012Metric_Pad1.15x1.40mm_HandSolder" H 6438 3900 50  0001 C CNN
+F 2 "Capacitor_SMD:C_1206_3216Metric_Pad1.42x1.75mm_HandSolder" H 6438 3900 50  0001 C CNN
 F 3 "~" H 6400 4050 50  0001 C CNN
 	1    6400 4050
@@
 F 0 "C52" H 3415 4096 50  0000 L CNN
 F 1 "10u" H 3415 4005 50  0000 L CNN
-F 2 "Capacitor_SMD:C_0805_2012Metric_Pad1.15x1.40mm_HandSolder" H 3338 3900 50  0001 C CNN
+F 2 "Capacitor_SMD:C_1206_3216Metric_Pad1.42x1.75mm_HandSolder" H 3338 3900 50  0001 C CNN
 F 3 "~" H 3300 4050 50  0001 C CNN
 	1    3300 4050
@@
 F 0 "C53" H 3765 4096 50  0000 L CNN
 F 1 "100n" H 3765 4005 50  0000 L CNN
-F 2 "Capacitor_SMD:C_0805_2012Metric_Pad1.15x1.40mm_HandSolder" H 3688 3900 50  0001 C CNN
+F 2 "Capacitor_SMD:C_1206_3216Metric_Pad1.42x1.75mm_HandSolder" H 3688 3900 50  0001 C CNN
 F 3 "~" H 3650 4050 50  0001 C CNN
 	1    3650 4050
@@
 F 0 "R10" H 3520 5246 50  0000 L CNN
 F 1 "22.1k" H 3520 5155 50  0000 L CNN
-F 2 "Resistor_SMD:R_0805_2012Metric_Pad1.15x1.40mm_HandSolder" V 3380 5200 50  0001 C CNN
+F 2 "Resistor_SMD:R_1206_3216Metric_Pad1.42x1.75mm_HandSolder" V 3380 5200 50  0001 C CNN
 F 3 "~" H 3450 5200 50  0001 C CNN
 	1    3450 5200
@@
 F 0 "R9" H 3520 4846 50  0000 L CNN
 F 1 "30.1k" H 3520 4755 50  0000 L CNN
-F 2 "Resistor_SMD:R_0805_2012Metric_Pad1.15x1.40mm_HandSolder" V 3380 4800 50  0001 C CNN
+F 2 "Resistor_SMD:R_1206_3216Metric_Pad1.42x1.75mm_HandSolder" V 3380 4800 50  0001 C CNN
 F 3 "~" H 3450 4800 50  0001 C CNN
 	1    3450 4800
@@
 F 0 "C51" H 3150 4900 50  0000 L CNN
 F 1 "22u" H 3150 4700 50  0000 L CNN
-F 2 "Capacitor_SMD:C_0805_2012Metric_Pad1.15x1.40mm_HandSolder" H 3188 4650 50  0001 C CNN
+F 2 "Capacitor_SMD:C_1206_3216Metric_Pad1.42x1.75mm_HandSolder" H 3188 4650 50  0001 C CNN
 F 3 "~" H 3150 4800 50  0001 C CNN
 	1    3150 4800
@@
 F 0 "C50" H 2900 4900 50  0000 L CNN
 F 1 "22u" H 2900 4700 50  0000 L CNN
-F 2 "Capacitor_SMD:C_0805_2012Metric_Pad1.15x1.40mm_HandSolder" H 2938 4650 50  0001 C CNN
+F 2 "Capacitor_SMD:C_1206_3216Metric_Pad1.42x1.75mm_HandSolder" H 2938 4650 50  0001 C CNN
 F 3 "~" H 2900 4800 50  0001 C CNN
 	1    2900 4800
@@
 F 0 "R11" V 3700 2750 50  0000 C CNN
 F 1 "100k" V 3800 2750 50  0000 C CNN
-F 2 "Resistor_SMD:R_0805_2012Metric_Pad1.15x1.40mm_HandSolder" V 3730 2750 50  0001 C CNN
+F 2 "Resistor_SMD:R_1206_3216Metric_Pad1.42x1.75mm_HandSolder" V 3730 2750 50  0001 C CNN
 F 3 "~" H 3800 2750 50  0001 C CNN
 	1    3800 2750
@@
 F 0 "C56" H 4550 3150 50  0000 L CNN
 F 1 "1u" H 4550 2950 50  0000 L CNN
-F 2 "Capacitor_SMD:C_0805_2012Metric_Pad1.15x1.40mm_HandSolder" H 4588 2900 50  0001 C CNN
+F 2 "Capacitor_SMD:C_1206_3216Metric_Pad1.42x1.75mm_HandSolder" H 4588 2900 50  0001 C CNN
 F 3 "~" H 4550 3050 50  0001 C CNN
 	1    4550 3050
@@
 F 0 "C57" H 6100 3350 50  0000 L CNN
 F 1 "100n" H 6100 3150 50  0000 L CNN
-F 2 "Capacitor_SMD:C_0805_2012Metric_Pad1.15x1.40mm_HandSolder" H 6138 3100 50  0001 C CNN
+F 2 "Capacitor_SMD:C_1206_3216Metric_Pad1.42x1.75mm_HandSolder" H 6138 3100 50  0001 C CNN
 F 3 "~" H 6100 3250 50  0001 C CNN
 	1    6100 3250
@@
 F 0 "C59" H 6300 3350 50  0000 L CNN
 F 1 "10u" H 6300 3150 50  0000 L CNN
-F 2 "Capacitor_SMD:C_0805_2012Metric_Pad1.15x1.40mm_HandSolder" H 6338 3100 50  0001 C CNN
+F 2 "Capacitor_SMD:C_1206_3216Metric_Pad1.42x1.75mm_HandSolder" H 6338 3100 50  0001 C CNN
 F 3 "~" H 6300 3250 50  0001 C CNN
 	1    6300 3250
@@
 F 0 "C61" H 6615 3296 50  0000 L CNN
 F 1 "100u" H 6615 3205 50  0000 L CNN
-F 2 "Capacitor_SMD:C_0805_2012Metric_Pad1.15x1.40mm_HandSolder" H 6500 3250 50  0001 C CNN
+F 2 "Capacitor_SMD:C_1206_3216Metric_Pad1.42x1.75mm_HandSolder" H 6500 3250 50  0001 C CNN
 F 3 "~" H 6500 3250 50  0001 C CNN
 	1    6500 3250
@@
 F 0 "C65" H 7450 3350 50  0000 L CNN
 F 1 "22u" H 7450 3150 50  0000 L CNN
-F 2 "Capacitor_SMD:C_0805_2012Metric_Pad1.15x1.40mm_HandSolder" H 7488 3100 50  0001 C CNN
+F 2 "Capacitor_SMD:C_1206_3216Metric_Pad1.42x1.75mm_HandSolder" H 7488 3100 50  0001 C CNN
 F 3 "~" H 7450 3250 50  0001 C CNN
 	1    7450 3250
@@
 F 0 "C66" H 7650 3350 50  0000 L CNN
 F 1 "22u" H 7650 3150 50  0000 L CNN
-F 2 "Capacitor_SMD:C_0805_2012Metric_Pad1.15x1.40mm_HandSolder" H 7688 3100 50  0001 C CNN
+F 2 "Capacitor_SMD:C_1206_3216Metric_Pad1.42x1.75mm_HandSolder" H 7688 3100 50  0001 C CNN
 F 3 "~" H 7650 3250 50  0001 C CNN
 	1    7650 3250
@@
 F 0 "R12" V 3900 2950 50  0000 C CNN
 F 1 "6.81k" V 4000 2950 50  0000 C CNN
-F 2 "Resistor_SMD:R_0805_2012Metric_Pad1.15x1.40mm_HandSolder" V 3930 2950 50  0001 C CNN
+F 2 "Resistor_SMD:R_1206_3216Metric_Pad1.42x1.75mm_HandSolder" V 3930 2950 50  0001 C CNN
 F 3 "~" H 4000 2950 50  0001 C CNN
 	1    4000 2950
@@
 F 0 "R13" V 3900 3350 50  0000 C CNN
 F 1 "22.1k" V 4000 3350 50  0000 C CNN
-F 2 "Resistor_SMD:R_0805_2012Metric_Pad1.15x1.40mm_HandSolder" V 3930 3350 50  0001 C CNN
+F 2 "Resistor_SMD:R_1206_3216Metric_Pad1.42x1.75mm_HandSolder" V 3930 3350 50  0001 C CNN
 F 3 "~" H 4000 3350 50  0001 C CNN
 	1    4000 3350
@@
 F 0 "C55" H 4300 3150 50  0000 L CNN
 F 1 "3.3n" H 4300 2950 50  0000 L CNN
-F 2 "Capacitor_SMD:C_0805_2012Metric_Pad1.15x1.40mm_HandSolder" H 4338 2900 50  0001 C CNN
+F 2 "Capacitor_SMD:C_1206_3216Metric_Pad1.42x1.75mm_HandSolder" H 4338 2900 50  0001 C CNN
 F 3 "~" H 4300 3050 50  0001 C CNN
 	1    4300 3050
@@
 F 0 "C62" H 6665 5146 50  0000 L CNN
 F 1 "1u" H 6665 5055 50  0000 L CNN
-F 2 "Capacitor_SMD:C_0805_2012Metric_Pad1.15x1.40mm_HandSolder" H 6588 4950 50  0001 C CNN
+F 2 "Capacitor_SMD:C_1206_3216Metric_Pad1.42x1.75mm_HandSolder" H 6588 4950 50  0001 C CNN
 F 3 "~" H 6550 5100 50  0001 C CNN
 	1    6550 5100
@@
 F 0 "C63" H 6650 3050 50  0000 L CNN
 F 1 "100n" H 6550 2850 50  0000 L CNN
-F 2 "Capacitor_SMD:C_0805_2012Metric_Pad1.15x1.40mm_HandSolder" H 6788 2800 50  0001 C CNN
+F 2 "Capacitor_SMD:C_1206_3216Metric_Pad1.42x1.75mm_HandSolder" H 6788 2800 50  0001 C CNN
 F 3 "~" H 6750 2950 50  0001 C CNN
 	1    6750 2950

Commit message: Tag you're it. Wired up the DAC, fixed the PSU footprint.
Parts:
- U5: footprint Package_SO:HTSSOP-32-1EP_6.1x11mm_P0.65mm_EP5.2x11mm_Mask4.11x4.36mm -> Package_SO:TSSOP-14-1EP_4.4x5mm_P0.65mm
Changed lines of the file:
@@
 F 0 "U5" H 5000 2450 50  0000 C CNN
 F 1 "TPS54325" H 5450 2450 50  0000 C CNN
-F 2 "Package_SO:HTSSOP-32-1EP_6.1x11mm_P0.65mm_EP5.2x11mm_Mask4.11x4.36mm" H 5150 2450 50  0001 C CNN
+F 2 "Package_SO:TSSOP-14-1EP_4.4x5mm_P0.65mm" H 5150 2450 50  0001 C CNN
 F 3 "" H 5150 2450 50  0001 C CNN
 	1    5150 2450
@@
 Text HLabel 9900 4450 1    50   Input ~ 0
 3.3VA
-Text HLabel 2650 4500 1    50   Input ~ 0
+Text HLabel 2650 4500 1    50   Output ~ 0
 1.8V
 Text HLabel 8000 2550 1    50   Input ~ 0

Commit message: Wire up 1V PSU. Use smaller footprints for small caps.
Parts:
- C53, C55, C56, C57, C60, C63: footprint Capacitor_SMD:C_1206_3216Metric_Pad1.42x1.75mm_HandSolder -> Capacitor_SMD:C_0805_2012Metric_Pad1.15x1.40mm_HandSolder
- C54: value 0.1u -> 100n; footprint Capacitor_SMD:C_1206_3216Metric_Pad1.42x1.75mm_HandSolder -> Capacitor_SMD:C_0805_2012Metric_Pad1.15x1.40mm_HandSolder
- C64: value 0.1u -> 100n
Changed lines of the file:
@@
 AR Path="/5DC1AA2E/5DCDC8D6" Ref="C54"  Part="1"
 F 0 "C54" H 4250 4500 50  0000 L CNN
-F 1 "0.1u" H 4250 4300 50  0000 L CNN
-F 2 "Capacitor_SMD:C_1206_3216Metric_Pad1.42x1.75mm_HandSolder" H 4288 4250 50  0001 C CNN
+F 1 "100n" H 4250 4300 50  0000 L CNN
+F 2 "Capacitor_SMD:C_0805_2012Metric_Pad1.15x1.40mm_HandSolder" H 4288 4250 50  0001 C CNN
 F 3 "~" H 4250 4400 50  0001 C CNN
 	1    4250 4400
@@
 AR Path="/5DC1AA2E/5DCDC907" Ref="C64"  Part="1"
 F 0 "C64" H 6915 4396 50  0000 L CNN
-F 1 "0.1u" H 6915 4305 50  0000 L CNN
+F 1 "100n" H 6915 4305 50  0000 L CNN
 F 2 "Capacitor_SMD:C_1206_3216Metric_Pad1.42x1.75mm_HandSolder" H 6838 4200 50  0001 C CNN
 F 3 "~" H 6800 4350 50  0001 C CNN
@@
 F 0 "C60" H 6515 4096 50  0000 L CNN
 F 1 "100n" H 6500 4000 50  0000 L CNN
-F 2 "Capacitor_SMD:C_1206_3216Metric_Pad1.42x1.75mm_HandSolder" H 6438 3900 50  0001 C CNN
+F 2 "Capacitor_SMD:C_0805_2012Metric_Pad1.15x1.40mm_HandSolder" H 6438 3900 50  0001 C CNN
 F 3 "~" H 6400 4050 50  0001 C CNN
 	1    6400 4050
@@
 F 0 "C53" H 3765 4096 50  0000 L CNN
 F 1 "100n" H 3765 4005 50  0000 L CNN
-F 2 "Capacitor_SMD:C_1206_3216Metric_Pad1.42x1.75mm_HandSolder" H 3688 3900 50  0001 C CNN
+F 2 "Capacitor_SMD:C_0805_2012Metric_Pad1.15x1.40mm_HandSolder" H 3688 3900 50  0001 C CNN
 F 3 "~" H 3650 4050 50  0001 C CNN
 	1    3650 4050
@@
 F 0 "C56" H 4550 3150 50  0000 L CNN
 F 1 "1u" H 4550 2950 50  0000 L CNN
-F 2 "Capacitor_SMD:C_1206_3216Metric_Pad1.42x1.75mm_HandSolder" H 4588 2900 50  0001 C CNN
+F 2 "Capacitor_SMD:C_0805_2012Metric_Pad1.15x1.40mm_HandSolder" H 4588 2900 50  0001 C CNN
 F 3 "~" H 4550 3050 50  0001 C CNN
 	1    4550 3050
@@
 F 0 "C57" H 6100 3350 50  0000 L CNN
 F 1 "100n" H 6100 3150 50  0000 L CNN
-F 2 "Capacitor_SMD:C_1206_3216Metric_Pad1.42x1.75mm_HandSolder" H 6138 3100 50  0001 C CNN
+F 2 "Capacitor_SMD:C_0805_2012Metric_Pad1.15x1.40mm_HandSolder" H 6138 3100 50  0001 C CNN
 F 3 "~" H 6100 3250 50  0001 C CNN
 	1    6100 3250
@@
 F 0 "C55" H 4300 3150 50  0000 L CNN
 F 1 "3.3n" H 4300 2950 50  0000 L CNN
-F 2 "Capacitor_SMD:C_1206_3216Metric_Pad1.42x1.75mm_HandSolder" H 4338 2900 50  0001 C CNN
+F 2 "Capacitor_SMD:C_0805_2012Metric_Pad1.15x1.40mm_HandSolder" H 4338 2900 50  0001 C CNN
 F 3 "~" H 4300 3050 50  0001 C CNN
 	1    4300 3050
@@
 F 0 "C63" H 6650 3050 50  0000 L CNN
 F 1 "100n" H 6550 2850 50  0000 L CNN
-F 2 "Capacitor_SMD:C_1206_3216Metric_Pad1.42x1.75mm_HandSolder" H 6788 2800 50  0001 C CNN
+F 2 "Capacitor_SMD:C_0805_2012Metric_Pad1.15x1.40mm_HandSolder" H 6788 2800 50  0001 C CNN
 F 3 "~" H 6750 2950 50  0001 C CNN
 	1    6750 2950

Commit message: Added in a bunch of footprints to the netlist; only missing buttons and some resistors, now.
Parts:
- C61: footprint Capacitor_SMD:C_1206_3216Metric_Pad1.42x1.75mm_HandSolder -> Capacitor_THT:CP_Radial_D10.0mm_P5.00mm
- L1, L2, L3: footprint Inductor_SMD:L_0805_2012Metric_Pad1.15x1.40mm_HandSolder -> footprints:L_SPM3015
Changed lines of the file:
@@
 F 0 "L2" V 7340 4550 50  0000 C CNN
 F 1 "2.2u" V 7249 4550 50  0000 C CNN
-F 2 "Inductor_SMD:L_0805_2012Metric_Pad1.15x1.40mm_HandSolder" H 7150 4550 50  0001 C CNN
+F 2 "footprints:L_SPM3015" H 7150 4550 50  0001 C CNN
 F 3 "~" H 7150 4550 50  0001 C CNN
 	1    7150 4550
@@
 F 0 "L1" V 4190 4600 50  0000 C CNN
 F 1 "1.5u" V 4099 4600 50  0000 C CNN
-F 2 "Inductor_SMD:L_0805_2012Metric_Pad1.15x1.40mm_HandSolder" H 4000 4600 50  0001 C CNN
+F 2 "footprints:L_SPM3015" H 4000 4600 50  0001 C CNN
 F 3 "~" H 4000 4600 50  0001 C CNN
 	1    4000 4600
@@
 F 0 "C61" H 6615 3296 50  0000 L CNN
 F 1 "100u" H 6615 3205 50  0000 L CNN
-F 2 "Capacitor_SMD:C_1206_3216Metric_Pad1.42x1.75mm_HandSolder" H 6500 3250 50  0001 C CNN
+F 2 "Capacitor_THT:CP_Radial_D10.0mm_P5.00mm" H 6500 3250 50  0001 C CNN
 F 3 "~" H 6500 3250 50  0001 C CNN
 	1    6500 3250
@@
 F 0 "L3" V 7350 2750 50  0000 C CNN
 F 1 "1.5u" V 7200 2750 50  0000 C CNN
-F 2 "Inductor_SMD:L_0805_2012Metric_Pad1.15x1.40mm_HandSolder" H 7250 2750 50  0001 C CNN
+F 2 "footprints:L_SPM3015" H 7250 2750 50  0001 C CNN
 F 3 "~" H 7250 2750 50  0001 C CNN
 	1    7250 2750

Commit message: Merge in USB footprint changes. Add new footprints for polarised caps and fix layout to match
Parts:
- C61: footprint Capacitor_THT:CP_Radial_D10.0mm_P5.00mm -> Capacitor_THT:CP_Radial_D5.0mm_P2.00mm
Changed lines of the file:
@@
 F 0 "C61" H 6615 3296 50  0000 L CNN
 F 1 "100u" H 6615 3205 50  0000 L CNN
-F 2 "Capacitor_THT:CP_Radial_D10.0mm_P5.00mm" H 6500 3250 50  0001 C CNN
+F 2 "Capacitor_THT:CP_Radial_D5.0mm_P2.00mm" H 6500 3250 50  0001 C CNN
 F 3 "~" H 6500 3250 50  0001 C CNN
 	1    6500 3250

Commit message: Removed pull-down resistors.
Parts:
- C62: footprint Capacitor_SMD:C_1206_3216Metric_Pad1.42x1.75mm_HandSolder -> Capacitor_THT:CP_Radial_D4.0mm_P1.50mm
Changed lines of the file:
@@
 F 0 "C62" H 6665 5146 50  0000 L CNN
 F 1 "1u" H 6665 5055 50  0000 L CNN
-F 2 "Capacitor_SMD:C_1206_3216Metric_Pad1.42x1.75mm_HandSolder" H 6588 4950 50  0001 C CNN
+F 2 "Capacitor_THT:CP_Radial_D4.0mm_P1.50mm" H 6588 4950 50  0001 C CNN
 F 3 "~" H 6550 5100 50  0001 C CNN
 	1    6550 5100
