File: AudioDac.sch (KiCad schematic (older format))
At the start: 15 parts, among them U8 PCM5102

Commit message: Better footprints
Parts:
- C69, C70, C71, C72, C73, C74, C75, C76, C77, C78, C79, C80: footprint Capacitor_SMD:C_0805_2012Metric -> Capacitor_SMD:C_0805_2012Metric_Pad1.15x1.40mm_HandSolder
- R30, R31: footprint Resistor_SMD:R_0805_2012Metric -> Resistor_SMD:R_0805_2012Metric_Pad1.15x1.40mm_HandSolder
Connections:
- net labels removed: GNDA
- wire segments 73 -> 72
Changed lines of the file:
@@
 F 0 "C69" V 4898 3000 50  0000 C CNN
 F 1 "0.1u" V 4989 3000 50  0000 C CNN
-F 2 "Capacitor_SMD:C_0805_2012Metric" H 5188 2850 50  0001 C CNN
+F 2 "Capacitor_SMD:C_0805_2012Metric_Pad1.15x1.40mm_HandSolder" H 5188 2850 50  0001 C CNN
 F 3 "~" H 5150 3000 50  0001 C CNN
 	1    5150 3000
@@
 F 0 "C71" H 6265 3846 50  0000 L CNN
 F 1 "2.2u" H 6265 3755 50  0000 L CNN
-F 2 "Capacitor_SMD:C_0805_2012Metric" H 6188 3650 50  0001 C CNN
+F 2 "Capacitor_SMD:C_0805_2012Metric_Pad1.15x1.40mm_HandSolder" H 6188 3650 50  0001 C CNN
 F 3 "~" H 6150 3800 50  0001 C CNN
 	1    6150 3800
@@
 F 0 "C70" V 5548 4650 50  0000 C CNN
 F 1 "2.2u" V 5639 4650 50  0000 C CNN
-F 2 "Capacitor_SMD:C_0805_2012Metric" H 5838 4500 50  0001 C CNN
+F 2 "Capacitor_SMD:C_0805_2012Metric_Pad1.15x1.40mm_HandSolder" H 5838 4500 50  0001 C CNN
 F 3 "~" H 5800 4650 50  0001 C CNN
 	1    5800 4650
@@
 F 0 "R30" V 6350 3300 50  0000 C CNN
 F 1 "470" V 6450 3300 50  0000 C CNN
-F 2 "Resistor_SMD:R_0805_2012Metric" V 6380 3300 50  0001 C CNN
+F 2 "Resistor_SMD:R_0805_2012Metric_Pad1.15x1.40mm_HandSolder" V 6380 3300 50  0001 C CNN
 F 3 "~" H 6450 3300 50  0001 C CNN
 	1    6450 3300
@@
 F 0 "R31" V 6350 3500 50  0000 C CNN
 F 1 "470" V 6450 3500 50  0000 C CNN
-F 2 "Resistor_SMD:R_0805_2012Metric" V 6380 3500 50  0001 C CNN
+F 2 "Resistor_SMD:R_0805_2012Metric_Pad1.15x1.40mm_HandSolder" V 6380 3500 50  0001 C CNN
 F 3 "~" H 6450 3500 50  0001 C CNN
 	1    6450 3500
@@
 F 0 "C72" V 5898 4150 50  0000 C CNN
 F 1 "0.1u" V 5989 4150 50  0000 C CNN
-F 2 "Capacitor_SMD:C_0805_2012Metric" H 6188 4000 50  0001 C CNN
+F 2 "Capacitor_SMD:C_0805_2012Metric_Pad1.15x1.40mm_HandSolder" H 6188 4000 50  0001 C CNN
 F 3 "~" H 6150 4150 50  0001 C CNN
 	1    6150 4150
@@
 F 0 "C73" V 6448 4150 50  0000 C CNN
 F 1 "0.1u" V 6539 4150 50  0000 C CNN
-F 2 "Capacitor_SMD:C_0805_2012Metric" H 6738 4000 50  0001 C CNN
+F 2 "Capacitor_SMD:C_0805_2012Metric_Pad1.15x1.40mm_HandSolder" H 6738 4000 50  0001 C CNN
 F 3 "~" H 6700 4150 50  0001 C CNN
 	1    6700 4150
@@
 Wire Wire Line
 	5550 4900 6500 4900
-Wire Wire Line
-	6500 4900 6500 5000
 Connection ~ 6500 4900
 Wire Wire Line
@@
 F 0 "C75" H 7615 4196 50  0000 L CNN
 F 1 "10u" H 7615 4105 50  0000 L CNN
-F 2 "Capacitor_SMD:C_0805_2012Metric" H 7500 4150 50  0001 C CNN
+F 2 "Capacitor_SMD:C_0805_2012Metric_Pad1.15x1.40mm_HandSolder" H 7500 4150 50  0001 C CNN
 F 3 "~" H 7500 4150 50  0001 C CNN
 	1    7500 4150
@@
 F 0 "C76" V 6402 4350 50  0000 C CNN
 F 1 "10u" V 6311 4350 50  0000 C CNN
-F 2 "Capacitor_SMD:C_0805_2012Metric" H 6150 4350 50  0001 C CNN
+F 2 "Capacitor_SMD:C_0805_2012Metric_Pad1.15x1.40mm_HandSolder" H 6150 4350 50  0001 C CNN
 F 3 "~" H 6150 4350 50  0001 C CNN
 	1    6150 4350
@@
 F 0 "C79" H 7865 3846 50  0000 L CNN
 F 1 "2.2n" H 7865 3755 50  0000 L CNN
-F 2 "Capacitor_SMD:C_0805_2012Metric" H 7788 3650 50  0001 C CNN
+F 2 "Capacitor_SMD:C_0805_2012Metric_Pad1.15x1.40mm_HandSolder" H 7788 3650 50  0001 C CNN
 F 3 "~" H 7750 3800 50  0001 C CNN
 	1    7750 3800
@@
 F 0 "C80" H 8265 3846 50  0000 L CNN
 F 1 "2.2n" H 8265 3755 50  0000 L CNN
-F 2 "Capacitor_SMD:C_0805_2012Metric" H 8188 3650 50  0001 C CNN
+F 2 "Capacitor_SMD:C_0805_2012Metric_Pad1.15x1.40mm_HandSolder" H 8188 3650 50  0001 C CNN
 F 3 "~" H 8150 3800 50  0001 C CNN
 	1    8150 3800
@@
 F 0 "C78" H 7215 4196 50  0000 L CNN
 F 1 "0.1u" H 7215 4105 50  0000 L CNN
-F 2 "Capacitor_SMD:C_0805_2012Metric" H 7138 4000 50  0001 C CNN
+F 2 "Capacitor_SMD:C_0805_2012Metric_Pad1.15x1.40mm_HandSolder" H 7138 4000 50  0001 C CNN
 F 3 "~" H 7100 4150 50  0001 C CNN
 	1    7100 4150
@@
 Wire Wire Line
 	7500 3100 7550 3100
-$Comp
-L power:GNDA #PWR0146
-U 1 1 5D840CE8
-P 6500 5000
-F 0 "#PWR0146" H 6500 4750 50  0001 C CNN
-F 1 "GNDA" H 6505 4827 50  0000 C CNN
-F 2 "" H 6500 5000 50  0001 C CNN
-F 3 "" H 6500 5000 50  0001 C CNN
-	1    6500 5000
-	1    0    0    -1
-$EndComp
 Wire Wire Line
 	6300 4150 6400 4150
@@
 F 0 "C77" V 6448 4350 50  0000 C CNN
 F 1 "10u" V 6539 4350 50  0000 C CNN
-F 2 "Capacitor_SMD:C_0805_2012Metric" H 6700 4350 50  0001 C CNN
+F 2 "Capacitor_SMD:C_0805_2012Metric_Pad1.15x1.40mm_HandSolder" H 6700 4350 50  0001 C CNN
 F 3 "~" H 6700 4350 50  0001 C CNN
 	1    6700 4350
@@
 F 0 "C74" V 4898 2600 50  0000 C CNN
 F 1 "10u" V 4989 2600 50  0000 C CNN
-F 2 "Capacitor_SMD:C_0805_2012Metric" H 5150 2600 50  0001 C CNN
+F 2 "Capacitor_SMD:C_0805_2012Metric_Pad1.15x1.40mm_HandSolder" H 5150 2600 50  0001 C CNN
 F 3 "~" H 5150 2600 50  0001 C CNN
 	1    5150 2600
@@
 Wire Wire Line
 	5350 2600 5350 3000
+$Comp
+L power:GND #PWR0146
+U 1 1 5D87C2CB
+P 6500 4900
+F 0 "#PWR0146" H 6500 4650 50  0001 C CNN
+F 1 "GND" H 6505 4727 50  0000 C CNN
+F 2 "" H 6500 4900 50  0001 C CNN
+F 3 "" H 6500 4900 50  0001 C CNN
+	1    6500 4900
+	1    0    0    -1
+$EndComp
 $EndSCHEMATC

Commit message: Fix USB connections and various cleanup
Connections:
- wire segments 72 -> 70
Other:
- moved on the sheet: C72, C73
Changed lines of the file:
@@
 P 5350 4700
 F 0 "#PWR0142" H 5350 4450 50  0001 C CNN
-F 1 "GND" H 5355 4527 50  0000 C CNN
+F 1 "GND" H 5250 4700 50  0000 C CNN
 F 2 "" H 5350 4700 50  0001 C CNN
 F 3 "" H 5350 4700 50  0001 C CNN
@@
 L Device:C C72
 U 1 1 5D8637F0
-P 6150 4150
-F 0 "C72" V 5898 4150 50  0000 C CNN
-F 1 "0.1u" V 5989 4150 50  0000 C CNN
-F 2 "Capacitor_SMD:C_0805_2012Metric_Pad1.15x1.40mm_HandSolder" H 6188 4000 50  0001 C CNN
-F 3 "~" H 6150 4150 50  0001 C CNN
-	1    6150 4150
-	0    1    1    0
-$EndComp
-Wire Wire Line
-	5950 4150 6000 4150
+P 6250 4300
+F 0 "C72" H 6150 4200 50  0000 C CNN
+F 1 "0.1u" H 6250 4400 50  0000 C CNN
+F 2 "Capacitor_SMD:C_0805_2012Metric_Pad1.15x1.40mm_HandSolder" H 6288 4150 50  0001 C CNN
+F 3 "~" H 6250 4300 50  0001 C CNN
+	1    6250 4300
+	-1   0    0    1
+$EndComp
 $Comp
 L Device:C C73
 U 1 1 5D86553E
-P 6700 4150
-F 0 "C73" V 6448 4150 50  0000 C CNN
-F 1 "0.1u" V 6539 4150 50  0000 C CNN
-F 2 "Capacitor_SMD:C_0805_2012Metric_Pad1.15x1.40mm_HandSolder" H 6738 4000 50  0001 C CNN
-F 3 "~" H 6700 4150 50  0001 C CNN
-	1    6700 4150
-	0    1    1    0
+P 6550 4300
+F 0 "C73" H 6250 4200 50  0000 C CNN
+F 1 "0.1u" H 6350 4400 50  0000 C CNN
+F 2 "Capacitor_SMD:C_0805_2012Metric_Pad1.15x1.40mm_HandSolder" H 6588 4150 50  0001 C CNN
+F 3 "~" H 6550 4300 50  0001 C CNN
+	1    6550 4300
+	-1   0    0    1
 $EndComp
 Wire Wire Line
@@
 	5550 4900 6500 4900
 Connection ~ 6500 4900
-Wire Wire Line
-	6500 4900 6700 4900
 Text HLabel 4500 3350 0    50   Input ~ 0
 Left-right-word-clock
@@
 L Device:CP1 C76
 U 1 1 5D8329EA
-P 6150 4350
-F 0 "C76" V 6402 4350 50  0000 C CNN
-F 1 "10u" V 6311 4350 50  0000 C CNN
-F 2 "Capacitor_SMD:C_0805_2012Metric_Pad1.15x1.40mm_HandSolder" H 6150 4350 50  0001 C CNN
-F 3 "~" H 6150 4350 50  0001 C CNN
-	1    6150 4350
-	0    -1   -1   0
+P 6050 4300
+F 0 "C76" H 6150 4400 50  0000 C CNN
+F 1 "10u" H 6050 4200 50  0000 C CNN
+F 2 "Capacitor_SMD:C_0805_2012Metric_Pad1.15x1.40mm_HandSolder" H 6050 4300 50  0001 C CNN
+F 3 "~" H 6050 4300 50  0001 C CNN
+	1    6050 4300
+	1    0    0    -1
 $EndComp
 Wire Wire Line
 	5950 4250 5950 4650
-Wire Wire Line
-	6000 4350 6000 4150
-Connection ~ 6000 4150
 $Comp
 L Device:C C79
@@
 Wire Wire Line
 	7500 3100 7550 3100
-Wire Wire Line
-	6300 4150 6400 4150
 $Comp
 L Device:CP1 C77
 U 1 1 5D8414C9
-P 6700 4350
-F 0 "C77" V 6448 4350 50  0000 C CNN
-F 1 "10u" V 6539 4350 50  0000 C CNN
-F 2 "Capacitor_SMD:C_0805_2012Metric_Pad1.15x1.40mm_HandSolder" H 6700 4350 50  0001 C CNN
-F 3 "~" H 6700 4350 50  0001 C CNN
-	1    6700 4350
-	0    1    1    0
-$EndComp
-Wire Wire Line
-	6400 4800 6400 4600
-Connection ~ 6400 4150
-Wire Wire Line
-	6400 4150 6550 4150
-Wire Wire Line
-	6550 4350 6400 4350
-Connection ~ 6400 4350
-Wire Wire Line
-	6400 4350 6400 4150
-Wire Wire Line
-	6400 4350 6300 4350
-Wire Wire Line
-	6850 4350 6850 4150
-Connection ~ 6850 4150
-Wire Wire Line
-	6700 4900 6700 4550
-Wire Wire Line
-	6700 4550 7100 4550
+P 6750 4300
+F 0 "C77" H 6550 4400 50  0000 C CNN
+F 1 "10u" H 6550 4200 50  0000 C CNN
+F 2 "Capacitor_SMD:C_0805_2012Metric_Pad1.15x1.40mm_HandSolder" H 6750 4300 50  0001 C CNN
+F 3 "~" H 6750 4300 50  0001 C CNN
+	1    6750 4300
+	1    0    0    -1
+$EndComp
+Wire Wire Line
+	7100 4900 7100 4550
 Connection ~ 7750 4550
 $Comp
 L power:GND #PWR0151
 U 1 1 5D8587ED
-P 6400 4600
-F 0 "#PWR0151" H 6400 4350 50  0001 C CNN
-F 1 "GND" V 6405 4472 50  0000 R CNN
-F 2 "" H 6400 4600 50  0001 C CNN
-F 3 "" H 6400 4600 50  0001 C CNN
-	1    6400 4600
-	0    -1   -1   0
-$EndComp
-Connection ~ 6400 4600
-Wire Wire Line
-	6400 4600 6400 4350
+P 5450 4800
+F 0 "#PWR0151" H 5450 4550 50  0001 C CNN
+F 1 "GND" H 5500 4650 50  0000 R CNN
+F 2 "" H 5450 4800 50  0001 C CNN
+F 3 "" H 5450 4800 50  0001 C CNN
+	1    5450 4800
+	1    0    0    -1
+$EndComp
 Wire Wire Line
 	7100 4300 7100 4550
@@
 	1    0    0    -1
 $EndComp
+Wire Wire Line
+	6500 4900 7100 4900
+Connection ~ 5450 4800
+Wire Wire Line
+	6550 4150 6750 4150
+Connection ~ 6750 4150
+Wire Wire Line
+	6750 4150 6850 4150
+Wire Wire Line
+	6750 4450 6550 4450
+Connection ~ 6550 4450
+Wire Wire Line
+	6550 4450 6400 4450
+Wire Wire Line
+	5950 4150 6050 4150
+Connection ~ 6050 4150
+Wire Wire Line
+	6050 4150 6250 4150
+Wire Wire Line
+	6400 4800 6400 4450
+Connection ~ 6400 4450
+Wire Wire Line
+	6050 4450 6250 4450
+Connection ~ 6250 4450
+Wire Wire Line
+	6250 4450 6400 4450
 $EndSCHEMATC

Commit message: Rearrange PCB components to more closely match schematics and take up less space
Other:
- moved on the sheet: C78, C79, C80
Changed lines of the file:
@@
-	-1   0    0    1
-$EndComp
-$Comp
-L Device:C C73
-U 1 1 5D86553E
-P 6550 4300
-F 0 "C73" H 6250 4200 50  0000 C CNN
-F 1 "0.1u" H 6350 4400 50  0000 C CNN
-F 2 "Capacitor_SMD:C_0805_2012Metric_Pad1.15x1.40mm_HandSolder" H 6588 4150 50  0001 C CNN
-F 3 "~" H 6550 4300 50  0001 C CNN
-	1    6550 4300
 	-1   0    0    1
 $EndComp
@@
 	6600 3300 8150 3300
 Wire Wire Line
-	8150 3650 8150 3300
-Wire Wire Line
-	7750 3650 7750 3500
-Wire Wire Line
-	8150 4550 8150 3950
+	8150 4050 8150 3300
+Wire Wire Line
+	7750 4050 7750 3500
+Wire Wire Line
+	8150 4550 8150 4350
 Wire Wire Line
 	7750 4550 8150 4550
 Wire Wire Line
-	7750 4550 7750 3950
+	7750 4550 7750 4350
 $Comp
 L Device:CP1 C75
 U 1 1 5D88C8BF
-P 7500 4150
-F 0 "C75" H 7615 4196 50  0000 L CNN
-F 1 "10u" H 7615 4105 50  0000 L CNN
-F 2 "Capacitor_SMD:C_0805_2012Metric_Pad1.15x1.40mm_HandSolder" H 7500 4150 50  0001 C CNN
-F 3 "~" H 7500 4150 50  0001 C CNN
-	1    7500 4150
+P 7500 3800
+F 0 "C75" H 7615 3846 50  0000 L CNN
+F 1 "10u" H 7615 3755 50  0000 L CNN
+F 2 "Capacitor_SMD:C_0805_2012Metric_Pad1.15x1.40mm_HandSolder" H 7500 3800 50  0001 C CNN
+F 3 "~" H 7500 3800 50  0001 C CNN
+	1    7500 3800
 	1    0    0    -1
 $EndComp
@@
 L Device:C C79
 U 1 1 5D83A113
-P 7750 3800
-F 0 "C79" H 7865 3846 50  0000 L CNN
-F 1 "2.2n" H 7865 3755 50  0000 L CNN
-F 2 "Capacitor_SMD:C_0805_2012Metric_Pad1.15x1.40mm_HandSolder" H 7788 3650 50  0001 C CNN
-F 3 "~" H 7750 3800 50  0001 C CNN
-	1    7750 3800
+P 7750 4200
+F 0 "C79" H 7865 4246 50  0000 L CNN
+F 1 "2.2n" H 7865 4155 50  0000 L CNN
+F 2 "Capacitor_SMD:C_0805_2012Metric_Pad1.15x1.40mm_HandSolder" H 7788 4050 50  0001 C CNN
+F 3 "~" H 7750 4200 50  0001 C CNN
+	1    7750 4200
 	1    0    0    -1
 $EndComp
@@
 L Device:C C80
 U 1 1 5D83A639
-P 8150 3800
-F 0 "C80" H 8265 3846 50  0000 L CNN
-F 1 "2.2n" H 8265 3755 50  0000 L CNN
-F 2 "Capacitor_SMD:C_0805_2012Metric_Pad1.15x1.40mm_HandSolder" H 8188 3650 50  0001 C CNN
-F 3 "~" H 8150 3800 50  0001 C CNN
-	1    8150 3800
+P 8150 4200
+F 0 "C80" H 8265 4246 50  0000 L CNN
+F 1 "2.2n" H 8265 4155 50  0000 L CNN
+F 2 "Capacitor_SMD:C_0805_2012Metric_Pad1.15x1.40mm_HandSolder" H 8188 4050 50  0001 C CNN
+F 3 "~" H 8150 4200 50  0001 C CNN
+	1    8150 4200
 	1    0    0    -1
 $EndComp
@@
 L Device:C C78
 U 1 1 5D83B385
-P 7100 4150
-F 0 "C78" H 7215 4196 50  0000 L CNN
-F 1 "0.1u" H 7215 4105 50  0000 L CNN
-F 2 "Capacitor_SMD:C_0805_2012Metric_Pad1.15x1.40mm_HandSolder" H 7138 4000 50  0001 C CNN
-F 3 "~" H 7100 4150 50  0001 C CNN
-	1    7100 4150
-	1    0    0    -1
-$EndComp
-Wire Wire Line
-	7100 4000 7100 3100
+P 7100 3800
+F 0 "C78" H 7215 3846 50  0000 L CNN
+F 1 "0.1u" H 7215 3755 50  0000 L CNN
+F 2 "Capacitor_SMD:C_0805_2012Metric_Pad1.15x1.40mm_HandSolder" H 7138 3650 50  0001 C CNN
+F 3 "~" H 7100 3800 50  0001 C CNN
+	1    7100 3800
+	1    0    0    -1
+$EndComp
+Wire Wire Line
+	7100 3650 7100 3100
 Wire Wire Line
 	5550 3100 7100 3100
@@
 	7100 3100 7500 3100
 Wire Wire Line
-	7500 4000 7500 3100
+	7500 3650 7500 3100
 Connection ~ 7500 3100
 Wire Wire Line
 	7500 3100 7550 3100
-$Comp
-L Device:CP1 C77
-U 1 1 5D8414C9
-P 6750 4300
-F 0 "C77" H 6550 4400 50  0000 C CNN
-F 1 "10u" H 6550 4200 50  0000 C CNN
-F 2 "Capacitor_SMD:C_0805_2012Metric_Pad1.15x1.40mm_HandSolder" H 6750 4300 50  0001 C CNN
-F 3 "~" H 6750 4300 50  0001 C CNN
-	1    6750 4300
-	1    0    0    -1
-$EndComp
 Wire Wire Line
 	7100 4900 7100 4550
@@
 $EndComp
 Wire Wire Line
-	7100 4300 7100 4550
+	7100 3950 7100 4550
 Connection ~ 7100 4550
 Wire Wire Line
 	7100 4550 7500 4550
 Wire Wire Line
-	7500 4300 7500 4550
+	7500 3950 7500 4550
 Connection ~ 7500 4550
 Wire Wire Line
@@
 	6500 4900 7100 4900
 Connection ~ 5450 4800
-Wire Wire Line
-	6550 4150 6750 4150
-Connection ~ 6750 4150
-Wire Wire Line
-	6750 4150 6850 4150
-Wire Wire Line
-	6750 4450 6550 4450
 Connection ~ 6550 4450
 Wire Wire Line
@@
 Wire Wire Line
 	6250 4450 6400 4450
+Wire Wire Line
+	6750 4450 6550 4450
+Wire Wire Line
+	6750 4150 6850 4150
+Connection ~ 6750 4150
+Wire Wire Line
+	6550 4150 6750 4150
+$Comp
+L Device:C C73
+U 1 1 5D86553E
+P 6550 4300
+F 0 "C73" H 6550 4200 50  0000 C CNN
+F 1 "0.1u" H 6550 4400 50  0000 C CNN
+F 2 "Capacitor_SMD:C_0805_2012Metric_Pad1.15x1.40mm_HandSolder" H 6588 4150 50  0001 C CNN
+F 3 "~" H 6550 4300 50  0001 C CNN
+	1    6550 4300
+	-1   0    0    1
+$EndComp
+$Comp
+L Device:CP1 C77
+U 1 1 5D8414C9
+P 6750 4300
+F 0 "C77" H 6850 4400 50  0000 C CNN
+F 1 "10u" H 6850 4200 50  0000 C CNN
+F 2 "Capacitor_SMD:C_0805_2012Metric_Pad1.15x1.40mm_HandSolder" H 6750 4300 50  0001 C CNN
+F 3 "~" H 6750 4300 50  0001 C CNN
+	1    6750 4300
+	1    0    0    -1
+$EndComp
 $EndSCHEMATC

Commit message: Updated component footprints. The PCB is now an unholy mess.
Parts:
- C69, C70, C71, C72, C73, C74, C75, C76, C77, C78, C79, C80: footprint Capacitor_SMD:C_0805_2012Metric_Pad1.15x1.40mm_HandSolder -> Capacitor_SMD:C_1206_3216Metric_Pad1.42x1.75mm_HandSolder
- R30, R31: footprint Resistor_SMD:R_0805_2012Metric_Pad1.15x1.40mm_HandSolder -> Resistor_SMD:R_1206_3216Metric_Pad1.42x1.75mm_HandSolder
Changed lines of the file:
@@
 F 0 "C69" V 4898 3000 50  0000 C CNN
 F 1 "0.1u" V 4989 3000 50  0000 C CNN
-F 2 "Capacitor_SMD:C_0805_2012Metric_Pad1.15x1.40mm_HandSolder" H 5188 2850 50  0001 C CNN
+F 2 "Capacitor_SMD:C_1206_3216Metric_Pad1.42x1.75mm_HandSolder" H 5188 2850 50  0001 C CNN
 F 3 "~" H 5150 3000 50  0001 C CNN
 	1    5150 3000
@@
 F 0 "C71" H 6265 3846 50  0000 L CNN
 F 1 "2.2u" H 6265 3755 50  0000 L CNN
-F 2 "Capacitor_SMD:C_0805_2012Metric_Pad1.15x1.40mm_HandSolder" H 6188 3650 50  0001 C CNN
+F 2 "Capacitor_SMD:C_1206_3216Metric_Pad1.42x1.75mm_HandSolder" H 6188 3650 50  0001 C CNN
 F 3 "~" H 6150 3800 50  0001 C CNN
 	1    6150 3800
@@
 F 0 "C70" V 5548 4650 50  0000 C CNN
 F 1 "2.2u" V 5639 4650 50  0000 C CNN
-F 2 "Capacitor_SMD:C_0805_2012Metric_Pad1.15x1.40mm_HandSolder" H 5838 4500 50  0001 C CNN
+F 2 "Capacitor_SMD:C_1206_3216Metric_Pad1.42x1.75mm_HandSolder" H 5838 4500 50  0001 C CNN
 F 3 "~" H 5800 4650 50  0001 C CNN
 	1    5800 4650
@@
 F 0 "R30" V 6350 3300 50  0000 C CNN
 F 1 "470" V 6450 3300 50  0000 C CNN
-F 2 "Resistor_SMD:R_0805_2012Metric_Pad1.15x1.40mm_HandSolder" V 6380 3300 50  0001 C CNN
+F 2 "Resistor_SMD:R_1206_3216Metric_Pad1.42x1.75mm_HandSolder" V 6380 3300 50  0001 C CNN
 F 3 "~" H 6450 3300 50  0001 C CNN
 	1    6450 3300
@@
 F 0 "R31" V 6350 3500 50  0000 C CNN
 F 1 "470" V 6450 3500 50  0000 C CNN
-F 2 "Resistor_SMD:R_0805_2012Metric_Pad1.15x1.40mm_HandSolder" V 6380 3500 50  0001 C CNN
+F 2 "Resistor_SMD:R_1206_3216Metric_Pad1.42x1.75mm_HandSolder" V 6380 3500 50  0001 C CNN
 F 3 "~" H 6450 3500 50  0001 C CNN
 	1    6450 3500
@@
 F 0 "C72" H 6150 4200 50  0000 C CNN
 F 1 "0.1u" H 6250 4400 50  0000 C CNN
-F 2 "Capacitor_SMD:C_0805_2012Metric_Pad1.15x1.40mm_HandSolder" H 6288 4150 50  0001 C CNN
+F 2 "Capacitor_SMD:C_1206_3216Metric_Pad1.42x1.75mm_HandSolder" H 6288 4150 50  0001 C CNN
 F 3 "~" H 6250 4300 50  0001 C CNN
 	1    6250 4300
@@
 F 0 "C75" H 7615 3846 50  0000 L CNN
 F 1 "10u" H 7615 3755 50  0000 L CNN
-F 2 "Capacitor_SMD:C_0805_2012Metric_Pad1.15x1.40mm_HandSolder" H 7500 3800 50  0001 C CNN
+F 2 "Capacitor_SMD:C_1206_3216Metric_Pad1.42x1.75mm_HandSolder" H 7500 3800 50  0001 C CNN
 F 3 "~" H 7500 3800 50  0001 C CNN
 	1    7500 3800
@@
 F 0 "C76" H 6150 4400 50  0000 C CNN
 F 1 "10u" H 6050 4200 50  0000 C CNN
-F 2 "Capacitor_SMD:C_0805_2012Metric_Pad1.15x1.40mm_HandSolder" H 6050 4300 50  0001 C CNN
+F 2 "Capacitor_SMD:C_1206_3216Metric_Pad1.42x1.75mm_HandSolder" H 6050 4300 50  0001 C CNN
 F 3 "~" H 6050 4300 50  0001 C CNN
 	1    6050 4300
@@
 F 0 "C79" H 7865 4246 50  0000 L CNN
 F 1 "2.2n" H 7865 4155 50  0000 L CNN
-F 2 "Capacitor_SMD:C_0805_2012Metric_Pad1.15x1.40mm_HandSolder" H 7788 4050 50  0001 C CNN
+F 2 "Capacitor_SMD:C_1206_3216Metric_Pad1.42x1.75mm_HandSolder" H 7788 4050 50  0001 C CNN
 F 3 "~" H 7750 4200 50  0001 C CNN
 	1    7750 4200
@@
 F 0 "C80" H 8265 4246 50  0000 L CNN
 F 1 "2.2n" H 8265 4155 50  0000 L CNN
-F 2 "Capacitor_SMD:C_0805_2012Metric_Pad1.15x1.40mm_HandSolder" H 8188 4050 50  0001 C CNN
+F 2 "Capacitor_SMD:C_1206_3216Metric_Pad1.42x1.75mm_HandSolder" H 8188 4050 50  0001 C CNN
 F 3 "~" H 8150 4200 50  0001 C CNN
 	1    8150 4200
@@
 F 0 "C78" H 7215 3846 50  0000 L CNN
 F 1 "0.1u" H 7215 3755 50  0000 L CNN
-F 2 "Capacitor_SMD:C_0805_2012Metric_Pad1.15x1.40mm_HandSolder" H 7138 3650 50  0001 C CNN
+F 2 "Capacitor_SMD:C_1206_3216Metric_Pad1.42x1.75mm_HandSolder" H 7138 3650 50  0001 C CNN
 F 3 "~" H 7100 3800 50  0001 C CNN
 	1    7100 3800
@@
 F 0 "C74" V 4898 2600 50  0000 C CNN
 F 1 "10u" V 4989 2600 50  0000 C CNN
-F 2 "Capacitor_SMD:C_0805_2012Metric_Pad1.15x1.40mm_HandSolder" H 5150 2600 50  0001 C CNN
+F 2 "Capacitor_SMD:C_1206_3216Metric_Pad1.42x1.75mm_HandSolder" H 5150 2600 50  0001 C CNN
 F 3 "~" H 5150 2600 50  0001 C CNN
 	1    5150 2600
@@
 F 0 "C73" H 6550 4200 50  0000 C CNN
 F 1 "0.1u" H 6550 4400 50  0000 C CNN
-F 2 "Capacitor_SMD:C_0805_2012Metric_Pad1.15x1.40mm_HandSolder" H 6588 4150 50  0001 C CNN
+F 2 "Capacitor_SMD:C_1206_3216Metric_Pad1.42x1.75mm_HandSolder" H 6588 4150 50  0001 C CNN
 F 3 "~" H 6550 4300 50  0001 C CNN
 	1    6550 4300
@@
 F 0 "C77" H 6850 4400 50  0000 C CNN
 F 1 "10u" H 6850 4200 50  0000 C CNN
-F 2 "Capacitor_SMD:C_0805_2012Metric_Pad1.15x1.40mm_HandSolder" H 6750 4300 50  0001 C CNN
+F 2 "Capacitor_SMD:C_1206_3216Metric_Pad1.42x1.75mm_HandSolder" H 6750 4300 50  0001 C CNN
 F 3 "~" H 6750 4300 50  0001 C CNN
 	1    6750 4300
