File: AudioDac.sch (KiCad schematic (older format))
At the start: 15 parts, among them U8 PCM5102

Commit message: Revert "Added in a bunch of footprints to the netlist; only missing buttons and some resistors, now."
This reverts commit 26f31b12234d03a706d1f0abb84aa744ef749ada.
Parts:
- C74, C75, C76, C77: footprint Capacitor_THT:CP_Radial_D10.0mm_P5.00mm -> Capacitor_SMD:C_1206_3216Metric_Pad1.42x1.75mm_HandSolder
Changed lines of the file:
@@
 F 0 "C75" H 7615 3846 50  0000 L CNN
 F 1 "10u" H 7615 3755 50  0000 L CNN
-F 2 "Capacitor_THT:CP_Radial_D10.0mm_P5.00mm" H 7500 3800 50  0001 C CNN
+F 2 "Capacitor_SMD:C_1206_3216Metric_Pad1.42x1.75mm_HandSolder" H 7500 3800 50  0001 C CNN
 F 3 "~" H 7500 3800 50  0001 C CNN
 	1    7500 3800
@@
 F 0 "C76" H 6150 4450 50  0000 C CNN
 F 1 "10u" H 6050 4250 50  0000 C CNN
-F 2 "Capacitor_THT:CP_Radial_D10.0mm_P5.00mm" H 6050 4350 50  0001 C CNN
+F 2 "Capacitor_SMD:C_1206_3216Metric_Pad1.42x1.75mm_HandSolder" H 6050 4350 50  0001 C CNN
 F 3 "~" H 6050 4350 50  0001 C CNN
 	1    6050 4350
@@
 F 0 "C74" V 4898 2600 50  0000 C CNN
 F 1 "10u" V 4989 2600 50  0000 C CNN
-F 2 "Capacitor_THT:CP_Radial_D10.0mm_P5.00mm" H 5150 2600 50  0001 C CNN
+F 2 "Capacitor_SMD:C_1206_3216Metric_Pad1.42x1.75mm_HandSolder" H 5150 2600 50  0001 C CNN
 F 3 "~" H 5150 2600 50  0001 C CNN
 	1    5150 2600
@@
 F 0 "C77" H 6850 4450 50  0000 C CNN
 F 1 "10u" H 6850 4250 50  0000 C CNN
-F 2 "Capacitor_THT:CP_Radial_D10.0mm_P5.00mm" H 6750 4350 50  0001 C CNN
+F 2 "Capacitor_SMD:C_1206_3216Metric_Pad1.42x1.75mm_HandSolder" H 6750 4350 50  0001 C CNN
 F 3 "~" H 6750 4350 50  0001 C CNN
 	1    6750 4350
