File: AudioDac.sch (KiCad schematic (older format))
At the start: 15 parts, among them U8 PCM5102

Commit message: Wire up 1V PSU. Use smaller footprints for small caps.
Parts:
- C69, C72, C73, C78: value 0.1u -> 100n; footprint Capacitor_SMD:C_1206_3216Metric_Pad1.42x1.75mm_HandSolder -> Capacitor_SMD:C_0805_2012Metric_Pad1.15x1.40mm_HandSolder
- C79, C80: footprint Capacitor_SMD:C_1206_3216Metric_Pad1.42x1.75mm_HandSolder -> Capacitor_SMD:C_0805_2012Metric_Pad1.15x1.40mm_HandSolder
Connections:
- net labels added: +3.3VA
Changed lines of the file:
@@
 P 5150 3000
 F 0 "C69" V 4898 3000 50  0000 C CNN
-F 1 "0.1u" V 4989 3000 50  0000 C CNN
-F 2 "Capacitor_SMD:C_1206_3216Metric_Pad1.42x1.75mm_HandSolder" H 5188 2850 50  0001 C CNN
+F 1 "100n" V 4989 3000 50  0000 C CNN
+F 2 "Capacitor_SMD:C_0805_2012Metric_Pad1.15x1.40mm_HandSolder" H 5188 2850 50  0001 C CNN
 F 3 "~" H 5150 3000 50  0001 C CNN
 	1    5150 3000
@@
 	5550 3150 5550 3100
 $Comp
-L power:+3.3V #PWR0145
+L power:+3.3VA #PWR0145
 U 1 1 5D871C47
 P 7550 2950
 F 0 "#PWR0145" H 7550 2800 50  0001 C CNN
-F 1 "+3.3V" H 7565 3123 50  0000 C CNN
+F 1 "+3.3VA" H 7565 3123 50  0000 C CNN
 F 2 "" H 7550 2950 50  0001 C CNN
 F 3 "" H 7550 2950 50  0001 C CNN
@@
 F 0 "C79" H 7865 4246 50  0000 L CNN
 F 1 "2.2n" H 7865 4155 50  0000 L CNN
-F 2 "Capacitor_SMD:C_1206_3216Metric_Pad1.42x1.75mm_HandSolder" H 7788 4050 50  0001 C CNN
+F 2 "Capacitor_SMD:C_0805_2012Metric_Pad1.15x1.40mm_HandSolder" H 7788 4050 50  0001 C CNN
 F 3 "~" H 7750 4200 50  0001 C CNN
 	1    7750 4200
@@
 F 0 "C80" H 8265 4246 50  0000 L CNN
 F 1 "2.2n" H 8265 4155 50  0000 L CNN
-F 2 "Capacitor_SMD:C_1206_3216Metric_Pad1.42x1.75mm_HandSolder" H 8188 4050 50  0001 C CNN
+F 2 "Capacitor_SMD:C_0805_2012Metric_Pad1.15x1.40mm_HandSolder" H 8188 4050 50  0001 C CNN
 F 3 "~" H 8150 4200 50  0001 C CNN
 	1    8150 4200
@@
 P 7100 3800
 F 0 "C78" H 7215 3846 50  0000 L CNN
-F 1 "0.1u" H 7215 3755 50  0000 L CNN
-F 2 "Capacitor_SMD:C_1206_3216Metric_Pad1.42x1.75mm_HandSolder" H 7138 3650 50  0001 C CNN
+F 1 "100n" H 7215 3755 50  0000 L CNN
+F 2 "Capacitor_SMD:C_0805_2012Metric_Pad1.15x1.40mm_HandSolder" H 7138 3650 50  0001 C CNN
 F 3 "~" H 7100 3800 50  0001 C CNN
 	1    7100 3800
@@
 P 6250 4350
 F 0 "C72" H 6150 4250 50  0000 C CNN
-F 1 "0.1u" H 6250 4450 50  0000 C CNN
-F 2 "Capacitor_SMD:C_1206_3216Metric_Pad1.42x1.75mm_HandSolder" H 6288 4200 50  0001 C CNN
+F 1 "100n" H 6250 4450 50  0000 C CNN
+F 2 "Capacitor_SMD:C_0805_2012Metric_Pad1.15x1.40mm_HandSolder" H 6288 4200 50  0001 C CNN
 F 3 "~" H 6250 4350 50  0001 C CNN
 	1    6250 4350
@@
 P 6550 4350
 F 0 "C73" H 6550 4250 50  0000 C CNN
-F 1 "0.1u" H 6550 4450 50  0000 C CNN
-F 2 "Capacitor_SMD:C_1206_3216Metric_Pad1.42x1.75mm_HandSolder" H 6588 4200 50  0001 C CNN
+F 1 "100n" H 6550 4450 50  0000 C CNN
+F 2 "Capacitor_SMD:C_0805_2012Metric_Pad1.15x1.40mm_HandSolder" H 6588 4200 50  0001 C CNN
 F 3 "~" H 6550 4350 50  0001 C CNN
 	1    6550 4350

Commit message: Added in a bunch of footprints to the netlist; only missing buttons and some resistors, now.
Parts:
- C74, C75, C76, C77: footprint Capacitor_SMD:C_1206_3216Metric_Pad1.42x1.75mm_HandSolder -> Capacitor_THT:CP_Radial_D10.0mm_P5.00mm
Changed lines of the file:
@@
 F 0 "C75" H 7615 3846 50  0000 L CNN
 F 1 "10u" H 7615 3755 50  0000 L CNN
-F 2 "Capacitor_SMD:C_1206_3216Metric_Pad1.42x1.75mm_HandSolder" H 7500 3800 50  0001 C CNN
+F 2 "Capacitor_THT:CP_Radial_D10.0mm_P5.00mm" H 7500 3800 50  0001 C CNN
 F 3 "~" H 7500 3800 50  0001 C CNN
 	1    7500 3800
@@
 F 0 "C76" H 6150 4450 50  0000 C CNN
 F 1 "10u" H 6050 4250 50  0000 C CNN
-F 2 "Capacitor_SMD:C_1206_3216Metric_Pad1.42x1.75mm_HandSolder" H 6050 4350 50  0001 C CNN
+F 2 "Capacitor_THT:CP_Radial_D10.0mm_P5.00mm" H 6050 4350 50  0001 C CNN
 F 3 "~" H 6050 4350 50  0001 C CNN
 	1    6050 4350
@@
 F 0 "C74" V 4898 2600 50  0000 C CNN
 F 1 "10u" V 4989 2600 50  0000 C CNN
-F 2 "Capacitor_SMD:C_1206_3216Metric_Pad1.42x1.75mm_HandSolder" H 5150 2600 50  0001 C CNN
+F 2 "Capacitor_THT:CP_Radial_D10.0mm_P5.00mm" H 5150 2600 50  0001 C CNN
 F 3 "~" H 5150 2600 50  0001 C CNN
 	1    5150 2600
@@
 F 0 "C77" H 6850 4450 50  0000 C CNN
 F 1 "10u" H 6850 4250 50  0000 C CNN
-F 2 "Capacitor_SMD:C_1206_3216Metric_Pad1.42x1.75mm_HandSolder" H 6750 4350 50  0001 C CNN
+F 2 "Capacitor_THT:CP_Radial_D10.0mm_P5.00mm" H 6750 4350 50  0001 C CNN
 F 3 "~" H 6750 4350 50  0001 C CNN
 	1    6750 4350

Commit message: Merge in USB footprint changes. Add new footprints for polarised caps and fix layout to match
Parts:
- C74, C75, C76, C77: footprint Capacitor_THT:CP_Radial_D10.0mm_P5.00mm -> Capacitor_THT:CP_Radial_D4.0mm_P1.50mm
Changed lines of the file:
@@
 F 0 "C75" H 7615 3846 50  0000 L CNN
 F 1 "10u" H 7615 3755 50  0000 L CNN
-F 2 "Capacitor_THT:CP_Radial_D10.0mm_P5.00mm" H 7500 3800 50  0001 C CNN
+F 2 "Capacitor_THT:CP_Radial_D4.0mm_P1.50mm" H 7500 3800 50  0001 C CNN
 F 3 "~" H 7500 3800 50  0001 C CNN
 	1    7500 3800
@@
 F 0 "C76" H 6150 4450 50  0000 C CNN
 F 1 "10u" H 6050 4250 50  0000 C CNN
-F 2 "Capacitor_THT:CP_Radial_D10.0mm_P5.00mm" H 6050 4350 50  0001 C CNN
+F 2 "Capacitor_THT:CP_Radial_D4.0mm_P1.50mm" H 6050 4350 50  0001 C CNN
 F 3 "~" H 6050 4350 50  0001 C CNN
 	1    6050 4350
@@
 F 0 "C74" V 4898 2600 50  0000 C CNN
 F 1 "10u" V 4989 2600 50  0000 C CNN
-F 2 "Capacitor_THT:CP_Radial_D10.0mm_P5.00mm" H 5150 2600 50  0001 C CNN
+F 2 "Capacitor_THT:CP_Radial_D4.0mm_P1.50mm" H 5150 2600 50  0001 C CNN
 F 3 "~" H 5150 2600 50  0001 C CNN
 	1    5150 2600
@@
 F 0 "C77" H 6850 4450 50  0000 C CNN
 F 1 "10u" H 6850 4250 50  0000 C CNN
-F 2 "Capacitor_THT:CP_Radial_D10.0mm_P5.00mm" H 6750 4350 50  0001 C CNN
+F 2 "Capacitor_THT:CP_Radial_D4.0mm_P1.50mm" H 6750 4350 50  0001 C CNN
 F 3 "~" H 6750 4350 50  0001 C CNN
 	1    6750 4350
