File: MCUDecouplers.sch (KiCad schematic (older format))
At the start: 8 parts

Commit message: Revert "Added in a bunch of footprints to the netlist; only missing buttons and some resistors, now."
This reverts commit 26f31b12234d03a706d1f0abb84aa744ef749ada.
Parts:
- C83, C9: footprint Capacitor_THT:CP_Radial_D10.0mm_P5.00mm -> Capacitor_SMD:C_1206_3216Metric_Pad1.42x1.75mm_HandSolder
Changed lines of the file:
@@
 F 0 "C9" H 1800 1850 50  0000 L CNN
 F 1 "10u" H 1800 1650 50  0000 L CNN
-F 2 "Capacitor_THT:CP_Radial_D10.0mm_P5.00mm" H 1750 1750 50  0001 C CNN
+F 2 "Capacitor_SMD:C_1206_3216Metric_Pad1.42x1.75mm_HandSolder" H 1750 1750 50  0001 C CNN
 F 3 "~" H 1750 1750 50  0001 C CNN
 	1    1750 1750
@@
 F 0 "C83" H 3450 1850 50  0000 L CNN
 F 1 "10u" H 3450 1650 50  0000 L CNN
-F 2 "Capacitor_THT:CP_Radial_D10.0mm_P5.00mm" H 3400 1750 50  0001 C CNN
+F 2 "Capacitor_SMD:C_1206_3216Metric_Pad1.42x1.75mm_HandSolder" H 3400 1750 50  0001 C CNN
 F 3 "~" H 3400 1750 50  0001 C CNN
 	1    3400 1750
