File: MCUDecouplers.sch (KiCad schematic (older format))
At the start: 8 parts

Commit message: add placeholder footprints, clean up ratsnest a bit
Parts:
- gave numbers to parts that had none: 8
Changed lines of the file:
@@
 AR Path="/5D8AD186" Ref="C?"  Part="1"
 AR Path="/5D8502F2/5D8AD186" Ref="C?"  Part="1"
-F 0 "C?" H 1150 1850 50  0000 L CNN
+AR Path="/5D8502F2/5D8A47A1/5D8AD186" Ref="C7"  Part="1"
+F 0 "C7" H 1150 1850 50  0000 L CNN
 F 1 "100n" H 1150 1650 50  0000 L CNN
 F 2 "Capacitor_SMD:C_0805_2012Metric_Pad1.15x1.40mm_HandSolder" H 1138 1600 50  0001 C CNN
@@
 AR Path="/5D8AD18C" Ref="C?"  Part="1"
 AR Path="/5D8502F2/5D8AD18C" Ref="C?"  Part="1"
-F 0 "C?" H 1450 1850 50  0000 L CNN
+AR Path="/5D8502F2/5D8A47A1/5D8AD18C" Ref="C8"  Part="1"
+F 0 "C8" H 1450 1850 50  0000 L CNN
 F 1 "100n" H 1450 1650 50  0000 L CNN
 F 2 "Capacitor_SMD:C_0805_2012Metric_Pad1.15x1.40mm_HandSolder" H 1438 1600 50  0001 C CNN
@@
 AR Path="/5D8AD192" Ref="C?"  Part="1"
 AR Path="/5D8502F2/5D8AD192" Ref="C?"  Part="1"
-F 0 "C?" H 1800 1850 50  0000 L CNN
+AR Path="/5D8502F2/5D8A47A1/5D8AD192" Ref="C9"  Part="1"
+F 0 "C9" H 1800 1850 50  0000 L CNN
 F 1 "10u" H 1800 1650 50  0000 L CNN
 F 2 "Capacitor_SMD:C_0805_2012Metric_Pad1.15x1.40mm_HandSolder" H 1750 1750 50  0001 C CNN
@@
 AR Path="/5D8AD1A1" Ref="C?"  Part="1"
 AR Path="/5D8502F2/5D8AD1A1" Ref="C?"  Part="1"
-F 0 "C?" H 2250 1850 50  0000 L CNN
+AR Path="/5D8502F2/5D8A47A1/5D8AD1A1" Ref="C10"  Part="1"
+F 0 "C10" H 2250 1850 50  0000 L CNN
 F 1 "100n" H 2250 1650 50  0000 L CNN
 F 2 "Capacitor_SMD:C_0805_2012Metric_Pad1.15x1.40mm_HandSolder" H 2238 1600 50  0001 C CNN
@@
 AR Path="/5D8AD1A7" Ref="C?"  Part="1"
 AR Path="/5D8502F2/5D8AD1A7" Ref="C?"  Part="1"
-F 0 "C?" H 2550 1850 50  0000 L CNN
+AR Path="/5D8502F2/5D8A47A1/5D8AD1A7" Ref="C11"  Part="1"
+F 0 "C11" H 2550 1850 50  0000 L CNN
 F 1 "100n" H 2550 1650 50  0000 L CNN
 F 2 "Capacitor_SMD:C_0805_2012Metric_Pad1.15x1.40mm_HandSolder" H 2538 1600 50  0001 C CNN
@@
 AR Path="/5D8AD1B4" Ref="C?"  Part="1"
 AR Path="/5D8502F2/5D8AD1B4" Ref="C?"  Part="1"
-F 0 "C?" H 3450 1850 50  0000 L CNN
+AR Path="/5D8502F2/5D8A47A1/5D8AD1B4" Ref="C83"  Part="1"
+F 0 "C83" H 3450 1850 50  0000 L CNN
 F 1 "10u" H 3450 1650 50  0000 L CNN
 F 2 "Capacitor_SMD:C_0805_2012Metric_Pad1.15x1.40mm_HandSolder" H 3400 1750 50  0001 C CNN
@@
 AR Path="/5D8AD1BA" Ref="C?"  Part="1"
 AR Path="/5D8502F2/5D8AD1BA" Ref="C?"  Part="1"
-F 0 "C?" H 2850 1850 50  0000 L CNN
+AR Path="/5D8502F2/5D8A47A1/5D8AD1BA" Ref="C81"  Part="1"
+F 0 "C81" H 2850 1850 50  0000 L CNN
 F 1 "100n" H 2850 1650 50  0000 L CNN
 F 2 "Capacitor_SMD:C_0805_2012Metric_Pad1.15x1.40mm_HandSolder" H 2838 1600 50  0001 C CNN
@@
 AR Path="/5D8AD1C3" Ref="#PWR?"  Part="1"
 AR Path="/5D8502F2/5D8AD1C3" Ref="#PWR?"  Part="1"
-F 0 "#PWR?" H 3400 1900 50  0001 C CNN
+AR Path="/5D8502F2/5D8A47A1/5D8AD1C3" Ref="#PWR0101"  Part="1"
+F 0 "#PWR0101" H 3400 1900 50  0001 C CNN
 F 1 "GND" H 3405 1977 50  0000 C CNN
 F 2 "" H 3400 2150 50  0001 C CNN
@@
 AR Path="/5D8AD1CB" Ref="C?"  Part="1"
 AR Path="/5D8502F2/5D8AD1CB" Ref="C?"  Part="1"
-F 0 "C?" H 3150 1850 50  0000 L CNN
+AR Path="/5D8502F2/5D8A47A1/5D8AD1CB" Ref="C82"  Part="1"
+F 0 "C82" H 3150 1850 50  0000 L CNN
 F 1 "100n" H 3150 1650 50  0000 L CNN
 F 2 "Capacitor_SMD:C_0805_2012Metric_Pad1.15x1.40mm_HandSolder" H 3138 1600 50  0001 C CNN
@@
 AR Path="/5D8AD1D8" Ref="#PWR?"  Part="1"
 AR Path="/5D8502F2/5D8AD1D8" Ref="#PWR?"  Part="1"
-F 0 "#PWR?" H 1750 1850 50  0001 C CNN
+AR Path="/5D8502F2/5D8A47A1/5D8AD1D8" Ref="#PWR0102"  Part="1"
+F 0 "#PWR0102" H 1750 1850 50  0001 C CNN
 F 1 "GND" H 1755 1927 50  0000 C CNN
 F 2 "" H 1750 2100 50  0001 C CNN
@@
 AR Path="/5D8AD1DF" Ref="#PWR?"  Part="1"
 AR Path="/5D8502F2/5D8AD1DF" Ref="#PWR?"  Part="1"
-F 0 "#PWR?" H 1100 1200 50  0001 C CNN
+AR Path="/5D8502F2/5D8A47A1/5D8AD1DF" Ref="#PWR0103"  Part="1"
+F 0 "#PWR0103" H 1100 1200 50  0001 C CNN
 F 1 "+3.3VA" H 1115 1523 50  0000 C CNN
 F 2 "" H 1100 1350 50  0001 C CNN
@@
 AR Path="/5D8AD1E5" Ref="#PWR?"  Part="1"
 AR Path="/5D8502F2/5D8AD1E5" Ref="#PWR?"  Part="1"
-F 0 "#PWR?" H 2200 1200 50  0001 C CNN
+AR Path="/5D8502F2/5D8A47A1/5D8AD1E5" Ref="#PWR0104"  Part="1"
+F 0 "#PWR0104" H 2200 1200 50  0001 C CNN
 F 1 "+3.3V" H 2215 1523 50  0000 C CNN
 F 2 "" H 2200 1350 50  0001 C CNN

Commit message: Updated component footprints. The PCB is now an unholy mess.
Parts:
- C10, C11, C7, C8, C81, C82, C83, C9: footprint Capacitor_SMD:C_0805_2012Metric_Pad1.15x1.40mm_HandSolder -> Capacitor_SMD:C_1206_3216Metric_Pad1.42x1.75mm_HandSolder
Changed lines of the file:
@@
 F 0 "C7" H 1150 1850 50  0000 L CNN
 F 1 "100n" H 1150 1650 50  0000 L CNN
-F 2 "Capacitor_SMD:C_0805_2012Metric_Pad1.15x1.40mm_HandSolder" H 1138 1600 50  0001 C CNN
+F 2 "Capacitor_SMD:C_1206_3216Metric_Pad1.42x1.75mm_HandSolder" H 1138 1600 50  0001 C CNN
 F 3 "~" H 1100 1750 50  0001 C CNN
 	1    1100 1750
@@
 F 0 "C8" H 1450 1850 50  0000 L CNN
 F 1 "100n" H 1450 1650 50  0000 L CNN
-F 2 "Capacitor_SMD:C_0805_2012Metric_Pad1.15x1.40mm_HandSolder" H 1438 1600 50  0001 C CNN
+F 2 "Capacitor_SMD:C_1206_3216Metric_Pad1.42x1.75mm_HandSolder" H 1438 1600 50  0001 C CNN
 F 3 "~" H 1400 1750 50  0001 C CNN
 	1    1400 1750
@@
 F 0 "C9" H 1800 1850 50  0000 L CNN
 F 1 "10u" H 1800 1650 50  0000 L CNN
-F 2 "Capacitor_SMD:C_0805_2012Metric_Pad1.15x1.40mm_HandSolder" H 1750 1750 50  0001 C CNN
+F 2 "Capacitor_SMD:C_1206_3216Metric_Pad1.42x1.75mm_HandSolder" H 1750 1750 50  0001 C CNN
 F 3 "~" H 1750 1750 50  0001 C CNN
 	1    1750 1750
@@
 F 0 "C10" H 2250 1850 50  0000 L CNN
 F 1 "100n" H 2250 1650 50  0000 L CNN
-F 2 "Capacitor_SMD:C_0805_2012Metric_Pad1.15x1.40mm_HandSolder" H 2238 1600 50  0001 C CNN
+F 2 "Capacitor_SMD:C_1206_3216Metric_Pad1.42x1.75mm_HandSolder" H 2238 1600 50  0001 C CNN
 F 3 "~" H 2200 1750 50  0001 C CNN
 	1    2200 1750
@@
 F 0 "C11" H 2550 1850 50  0000 L CNN
 F 1 "100n" H 2550 1650 50  0000 L CNN
-F 2 "Capacitor_SMD:C_0805_2012Metric_Pad1.15x1.40mm_HandSolder" H 2538 1600 50  0001 C CNN
+F 2 "Capacitor_SMD:C_1206_3216Metric_Pad1.42x1.75mm_HandSolder" H 2538 1600 50  0001 C CNN
 F 3 "~" H 2500 1750 50  0001 C CNN
 	1    2500 1750
@@
 F 0 "C83" H 3450 1850 50  0000 L CNN
 F 1 "10u" H 3450 1650 50  0000 L CNN
-F 2 "Capacitor_SMD:C_0805_2012Metric_Pad1.15x1.40mm_HandSolder" H 3400 1750 50  0001 C CNN
+F 2 "Capacitor_SMD:C_1206_3216Metric_Pad1.42x1.75mm_HandSolder" H 3400 1750 50  0001 C CNN
 F 3 "~" H 3400 1750 50  0001 C CNN
 	1    3400 1750
@@
 F 0 "C81" H 2850 1850 50  0000 L CNN
 F 1 "100n" H 2850 1650 50  0000 L CNN
-F 2 "Capacitor_SMD:C_0805_2012Metric_Pad1.15x1.40mm_HandSolder" H 2838 1600 50  0001 C CNN
+F 2 "Capacitor_SMD:C_1206_3216Metric_Pad1.42x1.75mm_HandSolder" H 2838 1600 50  0001 C CNN
 F 3 "~" H 2800 1750 50  0001 C CNN
 	1    2800 1750
@@
 F 0 "C82" H 3150 1850 50  0000 L CNN
 F 1 "100n" H 3150 1650 50  0000 L CNN
-F 2 "Capacitor_SMD:C_0805_2012Metric_Pad1.15x1.40mm_HandSolder" H 3138 1600 50  0001 C CNN
+F 2 "Capacitor_SMD:C_1206_3216Metric_Pad1.42x1.75mm_HandSolder" H 3138 1600 50  0001 C CNN
 F 3 "~" H 3100 1750 50  0001 C CNN
 	1    3100 1750

Commit message: Wire up 1V PSU. Use smaller footprints for small caps.
Parts:
- C10, C11, C7, C8, C81, C82: footprint Capacitor_SMD:C_1206_3216Metric_Pad1.42x1.75mm_HandSolder -> Capacitor_SMD:C_0805_2012Metric_Pad1.15x1.40mm_HandSolder
Changed lines of the file:
@@
 F 0 "C7" H 1150 1850 50  0000 L CNN
 F 1 "100n" H 1150 1650 50  0000 L CNN
-F 2 "Capacitor_SMD:C_1206_3216Metric_Pad1.42x1.75mm_HandSolder" H 1138 1600 50  0001 C CNN
+F 2 "Capacitor_SMD:C_0805_2012Metric_Pad1.15x1.40mm_HandSolder" H 1138 1600 50  0001 C CNN
 F 3 "~" H 1100 1750 50  0001 C CNN
 	1    1100 1750
@@
 F 0 "C8" H 1450 1850 50  0000 L CNN
 F 1 "100n" H 1450 1650 50  0000 L CNN
-F 2 "Capacitor_SMD:C_1206_3216Metric_Pad1.42x1.75mm_HandSolder" H 1438 1600 50  0001 C CNN
+F 2 "Capacitor_SMD:C_0805_2012Metric_Pad1.15x1.40mm_HandSolder" H 1438 1600 50  0001 C CNN
 F 3 "~" H 1400 1750 50  0001 C CNN
 	1    1400 1750
@@
 F 0 "C10" H 2250 1850 50  0000 L CNN
 F 1 "100n" H 2250 1650 50  0000 L CNN
-F 2 "Capacitor_SMD:C_1206_3216Metric_Pad1.42x1.75mm_HandSolder" H 2238 1600 50  0001 C CNN
+F 2 "Capacitor_SMD:C_0805_2012Metric_Pad1.15x1.40mm_HandSolder" H 2238 1600 50  0001 C CNN
 F 3 "~" H 2200 1750 50  0001 C CNN
 	1    2200 1750
@@
 F 0 "C11" H 2550 1850 50  0000 L CNN
 F 1 "100n" H 2550 1650 50  0000 L CNN
-F 2 "Capacitor_SMD:C_1206_3216Metric_Pad1.42x1.75mm_HandSolder" H 2538 1600 50  0001 C CNN
+F 2 "Capacitor_SMD:C_0805_2012Metric_Pad1.15x1.40mm_HandSolder" H 2538 1600 50  0001 C CNN
 F 3 "~" H 2500 1750 50  0001 C CNN
 	1    2500 1750
@@
 F 0 "C81" H 2850 1850 50  0000 L CNN
 F 1 "100n" H 2850 1650 50  0000 L CNN
-F 2 "Capacitor_SMD:C_1206_3216Metric_Pad1.42x1.75mm_HandSolder" H 2838 1600 50  0001 C CNN
+F 2 "Capacitor_SMD:C_0805_2012Metric_Pad1.15x1.40mm_HandSolder" H 2838 1600 50  0001 C CNN
 F 3 "~" H 2800 1750 50  0001 C CNN
 	1    2800 1750
@@
 F 0 "C82" H 3150 1850 50  0000 L CNN
 F 1 "100n" H 3150 1650 50  0000 L CNN
-F 2 "Capacitor_SMD:C_1206_3216Metric_Pad1.42x1.75mm_HandSolder" H 3138 1600 50  0001 C CNN
+F 2 "Capacitor_SMD:C_0805_2012Metric_Pad1.15x1.40mm_HandSolder" H 3138 1600 50  0001 C CNN
 F 3 "~" H 3100 1750 50  0001 C CNN
 	1    3100 1750

Commit message: Added in a bunch of footprints to the netlist; only missing buttons and some resistors, now.
Parts:
- C83, C9: footprint Capacitor_SMD:C_1206_3216Metric_Pad1.42x1.75mm_HandSolder -> Capacitor_THT:CP_Radial_D10.0mm_P5.00mm
Changed lines of the file:
@@
 F 0 "C9" H 1800 1850 50  0000 L CNN
 F 1 "10u" H 1800 1650 50  0000 L CNN
-F 2 "Capacitor_SMD:C_1206_3216Metric_Pad1.42x1.75mm_HandSolder" H 1750 1750 50  0001 C CNN
+F 2 "Capacitor_THT:CP_Radial_D10.0mm_P5.00mm" H 1750 1750 50  0001 C CNN
 F 3 "~" H 1750 1750 50  0001 C CNN
 	1    1750 1750
@@
 F 0 "C83" H 3450 1850 50  0000 L CNN
 F 1 "10u" H 3450 1650 50  0000 L CNN
-F 2 "Capacitor_SMD:C_1206_3216Metric_Pad1.42x1.75mm_HandSolder" H 3400 1750 50  0001 C CNN
+F 2 "Capacitor_THT:CP_Radial_D10.0mm_P5.00mm" H 3400 1750 50  0001 C CNN
 F 3 "~" H 3400 1750 50  0001 C CNN
 	1    3400 1750

Commit message: Merge in USB footprint changes. Add new footprints for polarised caps and fix layout to match
Parts:
- C83, C9: footprint Capacitor_THT:CP_Radial_D10.0mm_P5.00mm -> Capacitor_THT:CP_Radial_D4.0mm_P1.50mm
Changed lines of the file:
@@
 F 0 "C9" H 1800 1850 50  0000 L CNN
 F 1 "10u" H 1800 1650 50  0000 L CNN
-F 2 "Capacitor_THT:CP_Radial_D10.0mm_P5.00mm" H 1750 1750 50  0001 C CNN
+F 2 "Capacitor_THT:CP_Radial_D4.0mm_P1.50mm" H 1750 1750 50  0001 C CNN
 F 3 "~" H 1750 1750 50  0001 C CNN
 	1    1750 1750
@@
 F 0 "C83" H 3450 1850 50  0000 L CNN
 F 1 "10u" H 3450 1650 50  0000 L CNN
-F 2 "Capacitor_THT:CP_Radial_D10.0mm_P5.00mm" H 3400 1750 50  0001 C CNN
+F 2 "Capacitor_THT:CP_Radial_D4.0mm_P1.50mm" H 3400 1750 50  0001 C CNN
 F 3 "~" H 3400 1750 50  0001 C CNN
 	1    3400 1750
